Commit message: Fix livox frame

File: box_model/box_model/urdf/livox/livox.urdf.xacro (robot description, xacro)
@@ -35,9 +35,15 @@
     </collision>
   </link>
-  <link name="${lidar_frame}"/>
+<!--  <link name="${lidar_frame}"/>-->
+<!--  <joint name="livox_base_to_pandar" type="fixed">-->
+<!--    &lt;!&ndash; See page 12 of User Manual &ndash;&gt;-->
+<!--    &lt;!&ndash; note that the X axis points left. See manual page 11 &ndash;&gt;-->
+<!--    <origin xyz="0.0 0.0 46.4e-3" rpy="0.0 0.0 ${pi/2}"/>-->
+<!--    <parent link="livox_base"/>-->
+<!--    <child link="${lidar_frame}" />-->
+<!--  </joint>-->
+    <link name="${lidar_frame}"/>
   <joint name="livox_base_to_pandar" type="fixed">
-    <!-- See page 12 of User Manual -->
-    <!-- note that the X axis points left. See manual page 11 -->
-    <origin xyz="0.0 0.0 46.4e-3" rpy="0.0 0.0 ${pi/2}"/>
+    <origin xyz="0.0 0.0 0.0" rpy="${pi/2} 0.0 ${pi}"/>
     <parent link="livox_base"/>
     <child link="${lidar_frame}" />
