Commit message: rename eveything to box

File: box_model/box_model/urdf/box/box.urdf (robot description, URDF)
Before this commit: robot phasma, 12 links, 11 joints
Links:
- removed link body

File: box_model/box_model/urdf/box/box.urdf.xacro (robot description, xacro)
@@ -12,5 +12,5 @@
 limitations under the License.
 -->
-<robot name="phasma" xmlns:xacro="http://www.ros.org/wiki/xacro">
+<robot name="box" xmlns:xacro="http://www.ros.org/wiki/xacro">
   <xacro:include filename="$(find box_model)/urdf/alphasense/alphasense.urdf.xacro" />
   <xacro:include filename="$(find box_model)/urdf/hesai/hesai.urdf.xacro" />

Commit message: put sensors next to each other

File: box_model/box_model/urdf/box/box.urdf (robot description, URDF)
Before this commit: robot box, 11 links, 11 joints
Links:
- added link body; visual box size=0.25 0.5 0.01

File: box_model/box_model/urdf/box/box.urdf.xacro (robot description, xacro)
@@ -18,10 +18,11 @@
   <xacro:property name="alphasense_calibration" value="$(find box_model)/urdf/box/calibrations/20220322_calibration.yaml" />
   <xacro:alphasense parent="tip" calib_file="${alphasense_calibration}">
-    <origin xyz="-65.253e-3 0.0 179.0e-3" rpy="0 0 0" />
+    <origin xyz="0 0.20 0" rpy="0 0 0" />
   </xacro:alphasense>
   <link name="body">
     <visual>
       <geometry>
-        <mesh filename="package://box_model/urdf/box/meshes/phasma_body.dae" />
+        <box size="0.25 0.75 0.01"/>
+        <!-- <mesh filename="package://box_model/urdf/box/meshes/phasma_body.dae" /> -->
       </geometry>
     </visual>
@@ -41,5 +42,5 @@
   </joint>
   <xacro:hesai_device parent="tip" lidar_frame="PandarXT-32">
-    <origin xyz="-60.0e-3 0.0 95.0e-3" rpy="0 0 0"/>
+    <origin xyz="0 -0.20 0" rpy="0 0 0"/>
   </xacro:hesai_device>
 </robot>

Commit message: modeling

File: box_model/box_model/urdf/box/box.urdf (robot description, URDF)
Before this commit: robot box, 12 links, 11 joints
Links:
- link body: geometry visual box size=0.25 0.75 0.01
Joints:
- joint tip_to_alphasense: origin xyz=-65.253e-3 0.0 179.0e-3 rpy=0 0 0 -> xyz=0 0.20 0 rpy=0 0 0
- joint tip_to_hesai: origin xyz=-60.0e-3 0.0 95.0e-3 rpy=0 0 0 -> xyz=0 -0.20 0 rpy=0 0 0

File: box_model/box_model/urdf/box/box.urdf.xacro (robot description, xacro)
@@ -15,14 +15,10 @@
   <xacro:include filename="$(find box_model)/urdf/alphasense/alphasense.urdf.xacro" />
   <xacro:include filename="$(find box_model)/urdf/hesai/hesai.urdf.xacro" />
+  <xacro:include filename="$(find box_model)/urdf/livox/livox.urdf.xacro" />
   <link name="tip" />
-  <xacro:property name="alphasense_calibration" value="$(find box_model)/urdf/box/calibrations/20220322_calibration.yaml" />
-  <xacro:alphasense parent="tip" calib_file="${alphasense_calibration}">
-    <origin xyz="0 0.20 0" rpy="0 0 0" />
-  </xacro:alphasense>
-  <link name="body">
+    <link name="body">
     <visual>
       <geometry>
         <box size="0.25 0.75 0.01"/>
-        <!-- <mesh filename="package://box_model/urdf/box/meshes/phasma_body.dae" /> -->
       </geometry>
     </visual>
@@ -33,6 +29,10 @@
     <child link="body" />
   </joint>
-  <!-- This is the frame in which the ground truth is generated -->
+    <!-- This is the frame in which the ground truth is generated -->
   <link name="base"/>
+  <xacro:property name="alphasense_calibration" value="$(find box_model)/urdf/box/calibrations/20220322_calibration.yaml" />
+  <xacro:alphasense parent="tip" calib_file="${alphasense_calibration}">
+   <origin xyz="0 0 0" rpy="0 0 0" />
+  </xacro:alphasense>
   <!-- The base frame is coincident with the alphasense IMU but with the usual robot convention -->
   <joint name="alphasense_imu_to_base" type="fixed">
@@ -44,3 +44,6 @@
     <origin xyz="0 -0.20 0" rpy="0 0 0"/>
   </xacro:hesai_device>
+  <xacro:livox_device parent="tip" lidar_frame="mid360">
+    <origin xyz="0 0.20 0" rpy="1.57 0 1.57" />
+  </xacro:livox_device>
 </robot>

Commit message: Template for box urdf

File: box_model/box_model/urdf/box/box.urdf (robot description, URDF)
Before this commit: robot box, 12 links, 11 joints
Links:
- removed link body
- removed link tip
- added link box_back; visual box size=0.25 0.75 0.01
- added link gps; visual box size=0.2 0.2 0.2
- added link livox_base, mass 0.807; collision cylinder length=76.0e-3 radius=51.500e-3; visual mesh filename=package://box_model/urdf/livox/meshes/mid-360-asm.dae scale=0.001 0.001 0.001
- added link mid360
Joints:
- removed joint tip_to_alphasense
- removed joint tip_to_body
- removed joint tip_to_hesai
- added joint box_back_to_alphasense: type fixed, parent box_back, child alphasense_mount, origin xyz=0 0 0 rpy=0 0 0
- added joint box_back_to_gps: type fixed, parent box_back, child gps, origin xyz=0.0 0.0 0.0 rpy=0.0 0.0 0.0
- added joint box_back_to_hesai: type fixed, parent box_back, child hesai_base, origin xyz=0 -0.20 0 rpy=0 0 0
- added joint box_back_to_livox: type fixed, parent box_back, child livox_base, origin xyz=0 0.20 0 rpy=1.57 0 1.57
- added joint livox_base_to_pandar: type fixed, parent livox_base, child mid360, origin xyz=0.0 0.0 46.4e-3 rpy=0.0 0.0 1.5707963267948966

File: box_model/box_model/urdf/box/box.urdf.xacro (robot description, xacro)
@@ -13,37 +13,128 @@
 -->
 <robot name="box" xmlns:xacro="http://www.ros.org/wiki/xacro">
+  <!-- Loading the xacro files of sensors -->
   <xacro:include filename="$(find box_model)/urdf/alphasense/alphasense.urdf.xacro" />
   <xacro:include filename="$(find box_model)/urdf/hesai/hesai.urdf.xacro" />
   <xacro:include filename="$(find box_model)/urdf/livox/livox.urdf.xacro" />
-  <link name="tip" />
-    <link name="body">
+  <!-- Box -->
+  <link name="box">
     <visual>
       <geometry>
-        <box size="0.25 0.75 0.01"/>
+        <box size="0.8 0.2 0.2"/>
       </geometry>
+      <material name="gray_transparent">
+       <color rgba="0.3 0.3 0.4 0.3"/>
+      </material>
     </visual>
   </link>
-  <joint name="tip_to_body" type="fixed">
+  <!-- Box base -->
+  <joint name="box_to_box_base" type="fixed">
+      <origin xyz="0.0 0.0 -0.1" rpy="0.0 0.0 0.0" />
+      <parent link="box" />
+      <child link="box_base" />
+  </joint>
+  <link name="box_base">
+  </link>
+  <!-- Box back -->
+  <joint name="box_to_box_back" type="fixed">
+      <origin xyz="-0.4 0.0 -0.1" rpy="0.0 0.0 0.0" />
+      <parent link="box" />
+      <child link="box_back" />
+  </joint>
+  <link name="box_back">
+  </link>
+  <!-- GPS -->
+  <joint name="box_back_to_gps" type="fixed">
+      <origin xyz="-0.1 0.0 0.1" rpy="0.0 0.0 0.0" />
+      <parent link="box_back" />
+      <child link="gps" />
+  </joint>
+  <link name="gps">
+      <visual>
+        <geometry>
+          <box size="0.05 0.05 0.05"/>
+        </geometry>
+        <material name="gray_solid">
+          <color rgba="0.3 0.3 0.4 1.0"/>
+        </material>
+      </visual>
+  </link>
+  <!-- NUC -->
+  <joint name="box_back_to_nuc" type="fixed">
+      <origin xyz="0.4 0.0 0.2" rpy="0.0 0.0 0.0" />
+      <parent link="box_back" />
+      <child link="nuc" />
+  </joint>
+  <link name="nuc">
+      <visual>
+        <geometry>
+          <box size="0.05 0.05 0.05"/>
+        </geometry>
+        <material name="gray_solid">
+        </material>
+      </visual>
+    </link>
+  <!-- Jetson -->
+  <joint name="box_back_to_jetson" type="fixed">
+    <origin xyz="0.5 0.0 0.2" rpy="0.0 0.0 0.0" />
+    <parent link="box_back" />
+    <child link="jetson" />
+  </joint>
+  <link name="jetson">
+      <visual>
+        <geometry>
+          <box size="0.05 0.05 0.05"/>
+        </geometry>
+        <material name="gray_solid">
+        </material>
+      </visual>
+  </link>
+  <!-- Reflector -->
+  <joint name="box_back_to_reflector" type="fixed">
+    <origin xyz="0.6 0.0 0.2" rpy="0.0 0.0 0.0" />
+    <parent link="box_back" />
+    <child link="reflector" />
+  </joint>
+  <link name="reflector">
+    <visual>
+      <geometry>
+        <box size="0.05 0.05 0.05"/>
+      </geometry>
+      <material name="orange">
+          <color rgba="0.9 0.7 0.1 1.0"/>
+        </material>
+    </visual>
+  </link>
+  <!-- Alphasense -->
+  <xacro:property name="alphasense_calibration" value="$(find box_model)/urdf/box/calibrations/20220322_calibration.yaml" />
+  <xacro:alphasense parent="box_back" calib_file="${alphasense_calibration}">
+   <origin xyz="0.8 0 0.1" rpy="0 0 0" />
+  </xacro:alphasense>
+  !-- This is the frame in which the ground truth is generated, conincides with the alphasense IMU -->
+  <link name="base"/>
+  <joint name="alphasense_imu_to_base" type="fixed">
     <origin xyz="0.0 0.0 0.0" rpy="0.0 0.0 0.0" />
-    <parent link="tip" />
-    <child link="body" />
-  </joint>
-    <!-- This is the frame in which the ground truth is generated -->
-  <link name="base"/>
-  <xacro:property name="alphasense_calibration" value="$(find box_model)/urdf/box/calibrations/20220322_calibration.yaml" />
-  <xacro:alphasense parent="tip" calib_file="${alphasense_calibration}">
-   <origin xyz="0 0 0" rpy="0 0 0" />
-  </xacro:alphasense>
-  <!-- The base frame is coincident with the alphasense IMU but with the usual robot convention -->
-  <joint name="alphasense_imu_to_base" type="fixed">
-    <origin xyz="0.0 0.0 0.0" rpy="${-pi} 0.0 0.0" />
     <parent link="alphasense_imu"/>
     <child link="base"/>
   </joint>
-  <xacro:hesai_device parent="tip" lidar_frame="PandarXT-32">
-    <origin xyz="0 -0.20 0" rpy="0 0 0"/>
+  <!-- Livox -->
+  <joint name="box_back_to_livox_link" type="fixed">
+      <origin xyz="0.8 0.0 0.2" rpy="0.0 0.0 0.0" />
+      <parent link="box_back" />
+      <child link="livox_link" />
+  </joint>
+  <link name="livox_link"/>
+  <xacro:livox_device parent="livox_link" lidar_frame="mid360">
+    <origin xyz="0 0 0" rpy="${pi/2} ${-pi} 0" />
+  </xacro:livox_device>
+  <!-- Hesai -->
+  <joint name="box_back_to_hesai_link" type="fixed">
+      <origin xyz="0.8 0.0 0.0" rpy="0.0 0.0 0.0" />
+      <parent link="box_back" />
+      <child link="hesai_link" />
+  </joint>
+  <link name="hesai_link"/>
+  <xacro:hesai_device parent="hesai_link" lidar_frame="PandarXT-32">
+    <origin xyz="0 0 0" rpy="0 0 0"/>
   </xacro:hesai_device>
-  <xacro:livox_device parent="tip" lidar_frame="mid360">
-    <origin xyz="0 0.20 0" rpy="1.57 0 1.57" />
-  </xacro:livox_device>
 </robot>

Commit message: Cleanup, remove box_rviz old pkg

File: box_model/box_model/urdf/box/box.urdf (robot description, URDF)
Before this commit: robot box, 14 links, 13 joints
Links:
- removed link mid360
- added link adis16475_link
- added link adis_imu_link; visual box size=0.02 0.02 0.01
- added link box; visual box size=0.8 0.2 0.2
- added link box_base
- added link hesai_link
- added link imu_sensor_frame
- added link jetson; visual box size=0.05 0.05 0.05
- added link livox_frame
- added link livox_link
- added link nuc; visual box size=0.05 0.05 0.05
- added link reflector; visual box size=0.05 0.05 0.05
- added link usb_cam; visual box size=0.05 0.05 0.05
- added link usb_cam_link
- link box_back: geometry 
- link gps: geometry visual box size=0.05 0.05 0.05
Joints:
- removed joint box_back_to_hesai
- removed joint box_back_to_livox
- added joint adis_imu: type fixed, parent adis_imu_link, child adis16475_link, origin xyz=0.0 0.0 0.0 rpy=0.0 0.0 0.0
- added joint alphasense_imu_mapping: type fixed, parent alphasense_imu, child imu_sensor_frame, origin xyz=0.0 0.0 0.0 rpy=0.0 0.0 0.0
- added joint box_back_to_adis_imu_link: type fixed, parent box_back, child adis_imu_link, origin xyz=0.8 0.0 0.3 rpy=0.0 0.0 0.0
- added joint box_back_to_hesai_link: type fixed, parent box_back, child hesai_link, origin xyz=0.8 0.0 0.0 rpy=0.0 0.0 3.141592653589793
- added joint box_back_to_jetson: type fixed, parent box_back, child jetson, origin xyz=0.5 0.0 0.2 rpy=0.0 0.0 0.0
- added joint box_back_to_livox_link: type fixed, parent box_back, child livox_link, origin xyz=0.8 0.0 0.2 rpy=1.5707963267948966 -3.141592653589793 0.0
- added joint box_back_to_nuc: type fixed, parent box_back, child nuc, origin xyz=0.4 0.0 0.2 rpy=0.0 0.0 0.0
- added joint box_back_to_reflector: type fixed, parent box_back, child reflector, origin xyz=0.6 0.0 0.2 rpy=0.0 0.0 0.0
- added joint box_back_to_usb_cam_link: type fixed, parent box_back, child usb_cam_link, origin xyz=0.8 0.0 0.25 rpy=0.0 0.0 0.0
- added joint box_to_box_back: type fixed, parent box, child box_back, origin xyz=-0.4 0.0 -0.1 rpy=0.0 0.0 0.0
- added joint box_to_box_base: type fixed, parent box, child box_base, origin xyz=0.0 0.0 -0.1 rpy=0.0 0.0 0.0
- added joint hesai_link_to_hesai: type fixed, parent hesai_link, child hesai_base, origin xyz=0 0 0 rpy=0 0 0
- added joint livox_link_to_livox: type fixed, parent livox_link, child livox_base, origin xyz=0 0 0 rpy=0 0 0
- added joint usb_cam_link_to_usb_cam: type fixed, parent usb_cam_link, child usb_cam, origin xyz=0.0 0.0 0.0 rpy=0.0 -0.7853981633974483 0.0
- joint alphasense_imu_to_base: origin xyz=0.0 0.0 0.0 rpy=-3.141592653589793 0.0 0.0 -> xyz=0.0 0.0 0.0 rpy=0.0 0.0 0.0
- joint box_back_to_alphasense: origin xyz=0 0 0 rpy=0 0 0 -> xyz=0.8 0 0.1 rpy=0 0 0
- joint box_back_to_gps: origin xyz=0.0 0.0 0.0 rpy=0.0 0.0 0.0 -> xyz=-0.1 0.0 0.1 rpy=0.0 0.0 0.0
- joint livox_base_to_pandar: child mid360 -> livox_frame; origin xyz=0.0 0.0 46.4e-3 rpy=0.0 0.0 1.5707963267948966 -> xyz=0.0 0.0 0.0 rpy=1.5707963267948966 0.0 3.141592653589793

Commit message: add stim320 urdf

File: box_model/box_model/urdf/box/box.urdf (robot description, URDF)
Before this commit: robot box, 26 links, 25 joints
Links:
- added link STIM320
- added link stim320_imu_link; visual box size=0.02 0.02 0.01
Joints:
- added joint box_back_to_stim320_imu_link: type fixed, parent box_back, child stim320_imu_link, origin xyz=0.8 0.0 0.3 rpy=0.0 0.0 0.0
- added joint stim320_imu: type fixed, parent stim320_imu_link, child STIM320, origin xyz=0.0 0.0 0.0 rpy=0.0 0.0 0.0
