Commit message: add new frames to rviz

File: box_model/box_model/urdf/box/box.urdf (robot description, URDF)
Before this commit: robot box, 28 links, 27 joints
Links:
- removed link STIM320
- removed link usb_cam
- removed link usb_cam_link
- added link stim320_imu
- added link usb_cam_left; visual box size=0.05 0.05 0.05
- added link usb_cam_left_link
- added link usb_cam_middle; visual box size=0.05 0.05 0.05
- added link usb_cam_middle_link
- added link usb_cam_right; visual box size=0.05 0.05 0.05
- added link usb_cam_right_link
Joints:
- removed joint box_back_to_usb_cam_link
- removed joint usb_cam_link_to_usb_cam
- added joint box_back_to_usb_cam_left_link: type fixed, parent box_back, child usb_cam_left_link, origin xyz=0.8 0.0 0.25 rpy=0.0 0.0 0.0
- added joint box_back_to_usb_cam_middle_link: type fixed, parent box_back, child usb_cam_middle_link, origin xyz=0.8 0.0 0.25 rpy=0.0 0.0 0.0
- added joint box_back_to_usb_cam_right_link: type fixed, parent box_back, child usb_cam_right_link, origin xyz=0.8 0.0 0.25 rpy=0.0 0.0 0.0
- added joint usb_cam_left_link_to_usb_cam_left: type fixed, parent usb_cam_left_link, child usb_cam_left, origin xyz=0.0 0.0 0.0 rpy=0.0 -0.7853981633974483 0.0
- added joint usb_cam_middle_link_to_usb_cam_middle: type fixed, parent usb_cam_middle_link, child usb_cam_middle, origin xyz=0.0 0.0 0.0 rpy=0.0 -0.7853981633974483 0.0
- added joint usb_cam_right_link_to_usb_cam_right: type fixed, parent usb_cam_right_link, child usb_cam_right, origin xyz=0.0 0.0 0.0 rpy=0.0 -0.7853981633974483 0.0
- joint stim320_imu: child STIM320 -> stim320_imu

File: box_model/box_model/urdf/box/box.urdf.xacro (robot description, xacro)
@@ -13,195 +13,136 @@
 -->
 <robot name="box" xmlns:xacro="http://www.ros.org/wiki/xacro">
-  <!-- Loading the xacro files of sensors -->
-  <xacro:include filename="$(find box_model)/urdf/alphasense/alphasense.urdf.xacro" />
-  <xacro:include filename="$(find box_model)/urdf/hesai/hesai.urdf.xacro" />
-  <xacro:include filename="$(find box_model)/urdf/livox/livox.urdf.xacro" />
-  <!-- Defining the colors -->
-  <material name="gray_transparent">
-   <color rgba="0.3 0.3 0.4 0.3"/>
-  </material>
-  <material name="gray_solid">
-    <color rgba="0.3 0.3 0.4 1.0"/>
-  </material>
-  <material name="orange">
-          <color rgba="0.9 0.7 0.1 1.0"/>
-  </material>
-  <!-- Box -->
-  <link name="box">
+  <!-- Origin -->
+  <link name="origin"/>
+  <!-- Box base -->
+  <link name="box_base"/>
+  <joint name="origin_to_box_base" type="fixed">
+    <origin xyz="0.0 0.0 0.0" rpy="0.0 0.0 0.0" />
+    <parent link="origin" />
+    <child link="box_base" />
+  </joint>
+  <!-- Model base -->
+  <link name="model_base">
     <visual>
       <geometry>
-        <box size="0.8 0.2 0.2"/>
+        <mesh filename="package://box_model/urdf/box/mesh/box_model1.dae" />
       </geometry>
-      <material name="gray_transparent"/>
     </visual>
   </link>
-  <!-- Box base -->
-  <link name="box_base"/>
-  <joint name="box_to_box_base" type="fixed">
-      <origin xyz="0.0 0.0 -0.1" rpy="0.0 0.0 0.0" />
-      <parent link="box" />
-      <child link="box_base" />
+  <joint name="box_base_to_model_base" type="fixed">
+    <origin xyz="0.0 0.0 0.0" rpy="${pi} 0.0 ${pi/2}" />
+    <parent link="box_base" />
+    <child link="model_base" />
   </joint>
-  <!-- Box back -->
-  <link name="box_back"/>
-  <joint name="box_to_box_back" type="fixed">
-      <origin xyz="-0.4 0.0 -0.1" rpy="0.0 0.0 0.0" />
-      <parent link="box" />
-      <child link="box_back" />
+  <!-- Cameras front (coincide with front hdr cam) -->
+  <link name="cameras_front" />
+  <joint name="box_base_to_cameras_front" type="fixed">
+    <origin xyz="0.45 0.0 0.09" rpy="0.0 0.0 0.0" />
+    <parent link="box_base" />
+    <child link="cameras_front" />
   </joint>
-  <!-- GPS -->
-  <link name="gps">
-      <visual>
-        <geometry>
-          <box size="0.05 0.05 0.05"/>
-        </geometry>
-        <material name="gray_solid"/>
-      </visual>
-  </link>
-  <joint name="box_back_to_gps" type="fixed">
-      <origin xyz="-0.1 0.0 0.1" rpy="0.0 0.0 0.0" />
-      <parent link="box_back" />
-      <child link="gps" />
+  <!-- HDR camera front -->
+  <link name="hdr_front" />
+  <joint name="cameras_front_to_hdr_front" type="fixed">
+    <origin xyz="0.0 0.0 0.0" rpy="${-pi/2} 0.0 ${-pi/2}" />
+    <parent link="cameras_front" />
+    <child link="hdr_front" />
   </joint>
-  <!-- NUC -->
-  <link name="nuc">
-    <visual>
-      <geometry>
-        <box size="0.05 0.05 0.05"/>
-      </geometry>
-      <material name="gray_solid"/>
-    </visual>
-  </link>
-  <joint name="box_back_to_nuc" type="fixed">
-      <origin xyz="0.4 0.0 0.2" rpy="0.0 0.0 0.0" />
-      <parent link="box_back" />
-      <child link="nuc" />
+  <!-- Alphasense front left -->
+  <link name="alphasense_front_left" />
+  <joint name="hdr_front_to_alphasense_front_left" type="fixed">
+    <origin xyz="-0.055 -0.04 0.0" rpy="0.0 0.0 0.0" />
+    <parent link="hdr_front" />
+    <child link="alphasense_front_left" />
   </joint>
-  <!-- Jetson -->
-  <link name="jetson">
-      <visual>
-        <geometry>
-          <box size="0.05 0.05 0.05"/>
-        </geometry>
-        <material name="gray_solid"/>
-      </visual>
-  </link>
-  <joint name="box_back_to_jetson" type="fixed">
-    <origin xyz="0.5 0.0 0.2" rpy="0.0 0.0 0.0" />
-    <parent link="box_back" />
-    <child link="jetson" />
+  <!-- Alphasense front middle -->
+  <link name="alphasense_front_middle" />
+  <joint name="alphasense_front_left_to_alphasense_front_middle" type="fixed">
+    <origin xyz="0.054 0.0 0.0" rpy="0.0 0.0 0.0" />
+    <parent link="alphasense_front_left" />
+    <child link="alphasense_front_middle" />
   </joint>
-  <!-- Reflector -->
-  <link name="reflector">
-    <visual>
-      <geometry>
-        <box size="0.05 0.05 0.05"/>
-      </geometry>
-      <material name="orange"/>
-    </visual>
-  </link>
-  <joint name="box_back_to_reflector" type="fixed">
-    <origin xyz="0.6 0.0 0.2" rpy="0.0 0.0 0.0" />
-    <parent link="box_back" />
-    <child link="reflector" />
+  <!-- Alphasense front right -->
+  <link name="alphasense_front_right" />
+  <joint name="alphasense_front_middle_to_alphasense_front_right" type="fixed">
+    <origin xyz="0.054 0.0 0.0" rpy="0.0 0.0 0.0" />
+    <parent link="alphasense_front_middle" />
+    <child link="alphasense_front_right" />
   </joint>
-  <!-- Alphasense -->
-  <xacro:property name="alphasense_calibration" value="$(find box_model)/urdf/box/calibrations/20220322_calibration.yaml" />
-  <xacro:alphasense parent="box_back" calib_file="${alphasense_calibration}">
-   <origin xyz="0.8 0 0.1" rpy="0 0 0" />
-  </xacro:alphasense>
-  <!-- This is the frame in which the ground truth is generated, conincides with the alphasense IMU -->
-  <link name="base"/>
-  <link name="imu_sensor_frame"/>
-  <joint name="alphasense_imu_mapping" type="fixed">
-    <origin xyz="0.0 0.0 0.0" rpy="0.0 0.0 0.0" />
-    <parent link="alphasense_imu"/>
-    <child link="imu_sensor_frame"/>
+  <!-- Zed right -->
+  <link name="zed_right" />
+  <joint name="alphasense_front_right_to_zed_right" type="fixed">
+    <origin xyz="0.005 0.08 0.0" rpy="0.0 0.0 0.0" />
+    <parent link="alphasense_front_right" />
+    <child link="zed_right" />
   </joint>
-  <joint name="alphasense_imu_to_base" type="fixed">
-    <origin xyz="0.0 0.0 0.0" rpy="0.0 0.0 0.0" />
-    <parent link="alphasense_imu"/>
-    <child link="base"/>
+  <!-- Zed left -->
+  <link name="zed_left" />
+  <joint name="zed_right_to_zed_left" type="fixed">
+    <origin xyz="-0.12 0.0 0.0" rpy="0.0 0.0 0.0" />
+    <parent link="zed_right" />
+    <child link="zed_left" />
   </joint>
-  <!-- Livox -->
-  <link name="livox_link"/>
-  <joint name="box_back_to_livox_link" type="fixed">
-      <origin xyz="0.8 0.0 0.2" rpy="${pi/2} ${-pi} 0.0" />
-      <parent link="box_back" />
-      <child link="livox_link" />
+  <!-- Cameras right (coincide with right hdr cam) -->
+  <link name="cameras_right" />
+  <joint name="box_base_to_cameras_right" type="fixed">
+    <origin xyz="0.37 -0.10 0.09" rpy="0.0 0.0 0.0" />
+    <parent link="box_base" />
+    <child link="cameras_right" />
   </joint>
-  <xacro:livox_device parent="livox_link" lidar_frame="livox_frame">
-    <origin xyz="0 0 0" rpy="0 0 0" />
-  </xacro:livox_device>
-  <!-- Hesai -->
-  <link name="hesai_link"/>
-  <joint name="box_back_to_hesai_link" type="fixed">
-      <origin xyz="0.8 0.0 0.0" rpy="0.0 0.0 ${pi}" />
-      <parent link="box_back" />
-      <child link="hesai_link" />
+  <!-- HDR camera right -->
+  <link name="hdr_right" />
+  <joint name="cameras_right_to_hdr_right" type="fixed">
+    <origin xyz="0.0 0.0 0.0" rpy="${pi/2} ${pi} 0.0" />
+    <parent link="cameras_right" />
+    <child link="hdr_right" />
   </joint>
-  <xacro:hesai_device parent="hesai_link" lidar_frame="PandarXT-32">
-    <origin xyz="0 0 0" rpy="0 0 0"/>
-  </xacro:hesai_device>
-  <!-- USB Cam -->
-  <link name="usb_cam_link"/>
-  <joint name="box_back_to_usb_cam_link" type="fixed">
-      <origin xyz="0.8 0.0 0.25" rpy="0.0 0.0 0.0" />
-      <parent link="box_back" />
-      <child link="usb_cam_link" />
+  <link name="alphasense_right" />
+  <joint name="hdr_right_to_alphasense_right" type="fixed">
+    <origin xyz="0.0 -0.04 0.0" rpy="0.0 0.0 0.0" />
+    <parent link="hdr_right" />
+    <child link="alphasense_right" />
   </joint>
-  <link name="usb_cam">
-      <visual>
-        <geometry>
-          <box size="0.05 0.05 0.05"/>
-        </geometry>
-        <material name="gray_solid"/>
-      </visual>
-  </link>
-  <joint name="usb_cam_link_to_usb_cam" type="fixed">
-      <origin xyz="0.0 0.0 0.0" rpy="0.0 ${-pi/4} 0.0" />
-      <parent link="usb_cam_link" />
-      <child link="usb_cam" />
+  <!-- Cameras left (coincide with left hdr cam) -->
+  <link name="cameras_left" />
+  <joint name="box_base_to_cameras_left" type="fixed">
+    <origin xyz="0.37 0.10 0.09" rpy="0.0 0.0 0.0" />
+    <parent link="box_base" />
+    <child link="cameras_left" />
   </joint>
-    <!-- IMU STIM320 -->
-  <link name="stim320_imu_link">
-      <visual>
-        <geometry>
-          <box size="0.02 0.02 0.01"/>
-        </geometry>
-        <material name="gray_solid"/>
-      </visual>
-  </link>
-  <joint name="box_back_to_stim320_imu_link" type="fixed">
-    <origin xyz="0.8 0.0 0.3" rpy="0.0 0.0 0.0" />
-    <parent link="box_back" />
-    <child link="stim320_imu_link" />
+  <!-- HDR camera left -->
+  <link name="hdr_left" />
+  <joint name="cameras_left_to_hdr_left" type="fixed">
+    <origin xyz="0.0 0.0 0.0" rpy="-${pi/2} 0.0 0.0" />
+    <parent link="cameras_left" />
+    <child link="hdr_left" />
   </joint>
-  <link name="STIM320"/>
-  <joint name="stim320_imu" type="fixed">
-      <origin xyz="0.0 0.0 0.0" rpy="0.0 0.0 0.0" />
-      <parent link="stim320_imu_link" />
-      <child link="STIM320" />
+  <!-- Alphasense left -->
+  <link name="alphasense_left" />
+  <joint name="hdr_left_to_alphasense_left" type="fixed">
+    <origin xyz="0.0 -0.04 0.0" rpy="0.0 0.0 0.0" />
+    <parent link="hdr_left" />
+    <child link="alphasense_left" />
   </joint>
-  <!-- Adis IMU -->
-<!--  TODO: not calibrated-->
-  <link name="adis_imu_link">
-      <visual>
-        <geometry>
-          <box size="0.02 0.02 0.01"/>
-        </geometry>
-        <material name="gray_solid"/>
-      </visual>
-  </link>
-  <joint name="box_back_to_adis_imu_link" type="fixed">
-    <origin xyz="0.8 0.0 0.3" rpy="0.0 0.0 0.0" />
-    <parent link="box_back" />
-    <child link="adis_imu_link" />
+  <!-- Lidars (coincide with hesai) -->
+  <link name="lidars" />
+  <joint name="box_base_to_lidars" type="fixed">
+    <origin xyz="0.37 0.0 0.2" rpy="0.0 0.0 0.0" />
+    <parent link="box_base" />
+    <child link="lidars" />
   </joint>
-  <link name="adis16475_link"/>
-  <joint name="adis_imu" type="fixed">
-      <origin xyz="0.0 0.0 0.0" rpy="0.0 0.0 0.0" />
-      <parent link="adis_imu_link" />
-      <child link="adis16475_link" />
+  <!-- HDR camera left -->
+  <link name="hesai" />
+  <joint name="lidars_to_hesai" type="fixed">
+    <origin xyz="0.0 0.0 0.0" rpy="0.0 0.0 ${pi/2}" />
+    <parent link="lidars" />
+    <child link="hesai" />
+  </joint>
+  <!-- Alphasense left -->
+  <link name="livox" />
+  <joint name="hesai_to_livox" type="fixed">
+    <origin xyz="0.0 0.0 0.10" rpy="${pi} 0.0 ${-pi/2}" />
+    <parent link="hesai" />
+    <child link="livox" />
   </joint>
 </robot>

Commit message: update model

File: box_model/box_model/urdf/box/box.urdf (robot description, URDF)
Before this commit: robot box, 19 links, 18 joints
Links:
- removed link origin
- added link leica_base
- added link leica_base_model; visual cylinder length=0.2 radius=0.08
- added link leica_pos
- added link leica_world
- added link prism
Joints:
- removed joint origin_to_box_base
- added joint leica_base_to_leica_base_model: type fixed, parent leica_base, child leica_base_model, origin xyz=0.0 0.0 0.0 rpy=0.0 0.0 0.0
- added joint leica_pos_to_prism: type fixed, parent leica_pos, child prism, origin xyz=0.15 0.0 -0.3 rpy=0.0 0.0 0.0
- added joint leica_world_to_leica_base: type fixed, parent leica_world, child leica_base, origin xyz=1.0 1.0 1.0 rpy=0.0 0.0 0.0
- added joint leica_world_to_leica_pos: type fixed, parent leica_world, child leica_pos, origin xyz=0.0 0.0 0.0 rpy=0.0 0.0 0.0
- added joint prism_to_box_base: type fixed, parent prism, child box_base, origin xyz=0.0 0.0 0.0 rpy=0.0 0.0 0.0

Commit message: new stuff

File: box_model/box_model/urdf/box/box.urdf (robot description, URDF)
Before this commit: robot box, 23 links, 22 joints
Links:
- added link imu_adis16475
- added link imu_alphasense
- added link imu_stim320
Joints:
- added joint alphasense_front_left_to_imu_adis16475: type fixed, parent alphasense_front_left, child imu_adis16475, origin xyz= 0.054                   0.03                   -0.03 rpy= 1.57079632679                   0.0                   0.0
- added joint alphasense_front_left_to_imu_alphasense: type fixed, parent alphasense_front_left, child imu_alphasense, origin xyz= 0.054                   0.0                   -0.06 rpy= 1.57079632679                   -1.57079632679                   0.0
- added joint alphasense_front_left_to_imu_stim320: type fixed, parent alphasense_front_left, child imu_stim320, origin xyz= 0.054                   0.07                   -0.06 rpy= 1.57079632679                   -1.57079632679                   0.0
- joint leica_pos_to_prism: origin xyz=0.15 0.0 -0.3 rpy=0.0 0.0 0.0 -> xyz=0.0 0.0 0.0 rpy=0.0 0.0 0.0
- joint leica_world_to_leica_pos: origin xyz=0.0 0.0 0.0 rpy=0.0 0.0 0.0 -> xyz=0.15 0.0 -0.3 rpy=0.0 0.0 0.0
- joint prism_to_box_base: origin xyz=0.0 0.0 0.0 rpy=0.0 0.0 0.0 -> xyz=-0.075 0.0 -0.15 rpy=0.0 0.0 0.0

Commit message: Fixing urdf tree and linking zed2i to our tf

File: box_model/box_model/urdf/box/box.urdf (robot description, URDF)
Before this commit: robot box, 26 links, 25 joints
Links:
- removed link cameras_front
- removed link cameras_left
- removed link cameras_right
- removed link lidars
- removed link zed_left
- removed link zed_right
- added link alphasense_base
- added link hdr_base
- added link zed_base
Joints:
- removed joint alphasense_front_left_to_alphasense_front_middle
- removed joint alphasense_front_left_to_imu_adis16475
- removed joint alphasense_front_left_to_imu_alphasense
- removed joint alphasense_front_left_to_imu_stim320
- removed joint alphasense_front_middle_to_alphasense_front_right
- removed joint alphasense_front_right_to_zed_right
- removed joint box_base_to_cameras_front
- removed joint box_base_to_cameras_left
- removed joint box_base_to_cameras_right
- removed joint box_base_to_lidars
- removed joint cameras_front_to_hdr_front
- removed joint cameras_left_to_hdr_left
- removed joint cameras_right_to_hdr_right
- removed joint hdr_front_to_alphasense_front_left
- removed joint hdr_left_to_alphasense_left
- removed joint hdr_right_to_alphasense_right
- removed joint hesai_to_livox
- removed joint lidars_to_hesai
- removed joint zed_right_to_zed_left
- added joint alphasense_base_to_alphasense_front_left: type fixed, parent alphasense_base, child alphasense_front_left, origin xyz= 0.0                   0.0                   0.0 rpy= 0.0                   -0.0                   0.0
- added joint alphasense_base_to_alphasense_front_middle: type fixed, parent alphasense_base, child alphasense_front_middle, origin xyz= -0.054698757442450376                   -0.00020882496281570827                   -1.3877157931421699e-05 rpy= -3.136983778289491                   -0.005097155708924058                   -0.0012557767788089916
- added joint alphasense_base_to_alphasense_front_right: type fixed, parent alphasense_base, child alphasense_front_right, origin xyz= -0.11019818815545741                   1.0443869016379444e-05                   0.00025540782272211936 rpy= -0.0029393004042356442                   0.004871180163295483                   0.0006816981213750387
- added joint alphasense_base_to_alphasense_left: type fixed, parent alphasense_base, child alphasense_left, origin xyz= 0.047741167988699394                   -0.010988463753934308                   -0.06505666385033826 rpy= 1.5179219498551384                   -1.3779789320747404                   1.4581154559729528
- added joint alphasense_base_to_alphasense_right: type fixed, parent alphasense_base, child alphasense_right, origin xyz= -0.1567271351088724                   -0.011454790409696271                   -0.06597305132157129 rpy= -1.5458536755417267                   1.3955245673292458                   1.4168617596472088
- added joint box_base_to_alphasense_base: type fixed, parent box_base, child alphasense_base, origin xyz= 0.0                   0.0                   0.0 rpy= 0.0                   -0.0                   0.0
- added joint box_base_to_hdr_base: type fixed, parent box_base, child hdr_base, origin xyz= 0.0                   0.0                   0.0 rpy= 0.0                   0.0                   0.0
- added joint box_base_to_hesai: type fixed, parent box_base, child hesai, origin xyz= 0.0                   0.0                   0.0 rpy= 0.0                   0.0                   0.0
- added joint box_base_to_imu_adis16475: type fixed, parent box_base, child imu_adis16475, origin xyz= 0.0                   0.0                   0.0 rpy= 0.0                   0.0                   0.0
- added joint box_base_to_imu_alphasense: type fixed, parent box_base, child imu_alphasense, origin xyz= 0.0                   0.0                   0.0 rpy= 0.0                   0.0                   0.0
- added joint box_base_to_imu_stim320: type fixed, parent box_base, child imu_stim320, origin xyz= 0.0                   0.0                   0.0 rpy= 0.0                   -0.0                   0.0
- added joint box_base_to_livox: type fixed, parent box_base, child livox, origin xyz= 0.0                   0.0                   0.0 rpy= 0.0                   0.0                   0.0
- added joint box_base_to_zed_base: type fixed, parent box_base, child zed_base, origin xyz= 0.004928341904269176                   -0.07386742204771816                   0.022120515689282243 rpy= -3.1392184529965577                   -0.0006804673548911917                   0.0011198404612205875
- added joint hdr_base_to_hdr_front: type fixed, parent hdr_base, child hdr_front, origin xyz= 0.0                   0.0                   0.0 rpy= 0.0                   0.0                   0.0
- added joint hdr_base_to_hdr_left: type fixed, parent hdr_base, child hdr_left, origin xyz= 0.0                   0.0                   0.0 rpy= 0.0                   0.0                   0.0
- added joint hdr_base_to_hdr_right: type fixed, parent hdr_base, child hdr_right, origin xyz= 0.0                   0.0                   0.0 rpy= 0.0                   0.0                   0.0
- joint prism_to_box_base: origin xyz=-0.075 0.0 -0.15 rpy=0.0 0.0 0.0 -> xyz= -0.075                   0.0                   -0.15 rpy= 0.0                   0.0                   0.0

File: box_model/box_model/urdf/cameras/cameras.urdf.xacro (robot description, xacro)
@@ -108,5 +108,5 @@
                   ${calib['hdr_base_to_hdr_left']['pitch']}
                   ${calib['hdr_base_to_hdr_left']['yaw']}" />
-    <parent link="cameras_left" />
+    <parent link="hdr_base" />
     <child link="hdr_left" />
   </joint>

Commit message: renamed cameras

File: box_model/box_model/urdf/box/box.urdf (robot description, URDF)
Before this commit: robot box, 23 links, 22 joints
Joints:
- joint box_base_to_alphasense_base: origin xyz= 0.0                   0.0                   0.0 rpy= 0.0                   -0.0                   0.0 -> xyz= 0.054                   0.07                   -0.06 rpy= 0.0                   -1.5707963267948966                   0.0
- joint box_base_to_zed_base: origin xyz= 0.004928341904269176                   -0.07386742204771816                   0.022120515689282243 rpy= -3.1392184529965577                   -0.0006804673548911917                   0.0011198404612205875 -> xyz= 0.08212051568928225                   0.04907165809573082                   0.14386742204771819 rpy= 1.5701158575221625                   -0.00237420004356465                   1.5719177828250257

Commit message: Lets see

File: box_model/box_model/urdf/box/box.urdf (robot description, URDF)
Before this commit: robot box, 23 links, 22 joints
Links:
- removed link hesai
- added link hesaiXT32
Joints:
- joint box_base_to_hesai: child hesai -> hesaiXT32

File: box_model/box_model/urdf/lidars/lidars.urdf.xacro (robot description, xacro)
@@ -1,6 +1,6 @@
 <?xml version="1.0" ?>
 <robot name="lidars" xmlns:xacro="http://www.ros.org/wiki/xacro">
-  <!-- Hesai -->
-  <link name="hesai" />
+  <!-- hesaiXT32 -->
+  <link name="hesaiXT32" />
   <joint name="box_base_to_hesai" type="fixed">
     <origin xyz=" ${calib['box_base_to_hesai']['x']}
@@ -11,5 +11,5 @@
                   ${calib['box_base_to_hesai']['yaw']}" />
     <parent link="box_base" />
-    <child link="hesai" />
+    <child link="hesaiXT32" />
   </joint>
   <!-- Livox -->
