Commit message: zed2i visualization in RVIZ, camera rotations, other visualization changes

File: box_model/box_model/urdf/box/box.urdf (robot description, URDF)
Before this commit: robot box, 23 links, 22 joints
Links:
- removed link model_base
- added link box_base_model; visual mesh filename=package://box_model/urdf/box/mesh/box_assembly_incl_livox_m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
- added link hesaiXT32_model; visual mesh filename=package://box_model/urdf/box/mesh/hesai_lidar.dae
- added link livox_model; visual mesh filename=package://box_model/urdf/box/mesh/livox_mid360_lidar.dae
- added link prism_model; visual mesh filename=package://box_model/urdf/box/mesh/leica_small_prism.dae
Joints:
- removed joint box_base_to_model_base
- added joint box_base_to_box_base_model: type fixed, parent box_base, child box_base_model, origin xyz=0.0 0.0 0.0 rpy=0.0 0.0 0.0
- added joint hesaiXT32_to_hesaiXT32_model: type fixed, parent hesaiXT32, child hesaiXT32_model, origin xyz=0.0 0.0 0.0 rpy=0.0 0.0 0.0
- added joint livox_to_livox_model: type fixed, parent livox, child livox_model, origin xyz=0.0 0.0 0.0 rpy=0.0 0.0 0.0
- added joint prism_to_prism_model: type fixed, parent box_base, child prism_model, origin xyz=0.0 0.0 0.0 rpy=0.0 0.0 0.0
- joint alphasense_base_to_alphasense_front_left: origin xyz= 0.0                   0.0                   0.0 rpy= 0.0                   -0.0                   0.0 -> xyz= 0.0                   0.0                   0.0 rpy= 0.0                   0.0                   0.0
- joint alphasense_base_to_alphasense_front_middle: origin xyz= -0.054698757442450376                   -0.00020882496281570827                   -1.3877157931421699e-05 rpy= -3.136983778289491                   -0.005097155708924058                   -0.0012557767788089916 -> xyz= 0.055                   -0.0                   -0.0 rpy= 0.0                   0.0                   0.0
- joint alphasense_base_to_alphasense_front_right: origin xyz= -0.11019818815545741                   1.0443869016379444e-05                   0.00025540782272211936 rpy= -0.0029393004042356442                   0.004871180163295483                   0.0006816981213750387 -> xyz= 0.11                   -0.0                   -0.0 rpy= 0.0                   0.0                   0.0
- joint alphasense_base_to_alphasense_left: origin xyz= 0.047741167988699394                   -0.010988463753934308                   -0.06505666385033826 rpy= 1.5179219498551384                   -1.3779789320747404                   1.4581154559729528 -> xyz= -0.045                   0.011                   -0.065 rpy= 1.396                   -1.396                   -1.571
- joint alphasense_base_to_alphasense_right: origin xyz= -0.1567271351088724                   -0.011454790409696271                   -0.06597305132157129 rpy= -1.5458536755417267                   1.3955245673292458                   1.4168617596472088 -> xyz= 0.155                   0.011                   -0.065 rpy= -1.396                   -1.396                   -1.571
- joint box_base_to_alphasense_base: origin xyz= 0.054                   0.07                   -0.06 rpy= 0.0                   -1.5707963267948966                   0.0 -> xyz= 0.072                   0.033                   0.089 rpy= -1.745                   0.0                   -1.571
- joint box_base_to_hdr_base: origin xyz= 0.0                   0.0                   0.0 rpy= 0.0                   0.0                   0.0 -> xyz= 0.059                   -0.022                   0.054 rpy= -1.571                   0.0                   -1.571
- joint box_base_to_hesai: origin xyz= 0.0                   0.0                   0.0 rpy= 0.0                   0.0                   0.0 -> xyz= 0.013                   -0.022                   0.169 rpy= 0.0                   0.0                   1.571
- joint box_base_to_imu_adis16475: origin xyz= 0.0                   0.0                   0.0 rpy= 0.0                   0.0                   0.0 -> xyz= 0.032                   -0.056                   0.002 rpy= 0.0                   0.0                   1.571
- joint box_base_to_imu_stim320: origin xyz= 0.0                   0.0                   0.0 rpy= 0.0                   -0.0                   0.0 -> xyz= 0.0                   0.0                   0.0 rpy= 0.0                   0.0                   0.0
- joint box_base_to_livox: origin xyz= 0.0                   0.0                   0.0 rpy= 0.0                   0.0                   0.0 -> xyz= 0.013                   -0.022                   0.264 rpy= 3.142                   0.0                   0.0
- joint box_base_to_zed_base: origin xyz= 0.08212051568928225                   0.04907165809573082                   0.14386742204771819 rpy= 1.5701158575221625                   -0.00237420004356465                   1.5719177828250257 -> xyz= 0.075                   -0.022                   0.028 rpy= 3.142                   0.175                   0.0
- joint hdr_base_to_hdr_left: origin xyz= 0.0                   0.0                   0.0 rpy= 0.0                   0.0                   0.0 -> xyz= -0.087                   0.0                   -0.055 rpy= 3.142                   -1.396                   3.142
- joint hdr_base_to_hdr_right: origin xyz= 0.0                   0.0                   0.0 rpy= 0.0                   0.0                   0.0 -> xyz= 0.087                   0.0                   -0.055 rpy= 3.142                   1.396                   3.142
- joint prism_to_box_base: origin xyz= -0.075                   0.0                   -0.15 rpy= 0.0                   0.0                   0.0 -> xyz= -0.013                   0.022                   -0.34 rpy= 0.0                   0.0                   0.0

File: box_model/box_model/urdf/box/box.urdf.xacro (robot description, xacro)
@@ -75,5 +75,5 @@
   <joint name="prism_to_prism_model" type="fixed">
     <origin xyz="0.0 0.0 0.0" rpy="0.0 0.0 0.0" />
-    <parent link="box_base" />
+    <parent link="prism" />
     <child link="prism_model" />
   </joint>
