Commit message: fix

File: box_model/box_model/urdf/box/box.urdf.xacro (robot description, xacro)
@@ -33,5 +33,5 @@
   <joint name="box_base_to_box_base_model" type="fixed">
     <origin xyz="-0.02 0.0 0.0" rpy="0.0 0.0 0.0" />
-    <parent link="box_base" />
+    <parent link="stim320_imu" />
     <child link="box_base_model" />
   </joint>

Commit message: Adding colors

File: box_model/box_model/urdf/box/box.urdf.xacro (robot description, xacro)
@@ -17,4 +17,14 @@
   <xacro:include filename="$(find box_model)/urdf/hesai/hesai.urdf.xacro" />
   <xacro:include filename="$(find box_model)/urdf/livox/livox.urdf.xacro" />
+  <!-- Defining the colors -->
+  <material name="gray_transparent">
+   <color rgba="0.3 0.3 0.4 0.3"/>
+  </material>
+  <material name="gray_solid">
+    <color rgba="0.3 0.3 0.4 1.0"/>
+  </material>
+  <material name="orange">
+          <color rgba="0.9 0.7 0.1 1.0"/>
+  </material>
   <!-- Box -->
   <link name="box">
@@ -23,7 +33,5 @@
         <box size="0.8 0.2 0.2"/>
       </geometry>
-      <material name="gray_transparent">
-       <color rgba="0.3 0.3 0.4 0.3"/>
-      </material>
+      <material name="gray_transparent"/>
     </visual>
   </link>
@@ -55,7 +63,5 @@
           <box size="0.05 0.05 0.05"/>
         </geometry>
-        <material name="gray_solid">
-          <color rgba="0.3 0.3 0.4 1.0"/>
-        </material>
+        <material name="gray_solid"/>
       </visual>
   </link>
@@ -71,6 +77,5 @@
           <box size="0.05 0.05 0.05"/>
         </geometry>
-        <material name="gray_solid">
-        </material>
+        <material name="gray_solid"/>
       </visual>
     </link>
@@ -86,6 +91,5 @@
           <box size="0.05 0.05 0.05"/>
         </geometry>
-        <material name="gray_solid">
-        </material>
+        <material name="gray_solid"/>
       </visual>
   </link>
@@ -101,7 +105,5 @@
         <box size="0.05 0.05 0.05"/>
       </geometry>
-      <material name="orange">
-          <color rgba="0.9 0.7 0.1 1.0"/>
-        </material>
+      <material name="orange"/>
     </visual>
   </link>
@@ -138,3 +140,23 @@
     <origin xyz="0 0 0" rpy="0 0 0"/>
   </xacro:hesai_device>
+  <!-- USB Cam -->
+  <joint name="box_back_to_usb_cam_link" type="fixed">
+      <origin xyz="0.8 0.0 0.25" rpy="0.0 0.0 0.0" />
+      <parent link="box_back" />
+      <child link="usb_cam_link" />
+  </joint>
+  <link name="usb_cam_link"/>
+  <joint name="usb_cam_link_to_usb_cam" type="fixed">
+      <origin xyz="0.0 0.0 0.0" rpy="0.0 ${-pi/4} 0.0" />
+      <parent link="usb_cam_link" />
+      <child link="usb_cam" />
+  </joint>
+  <link name="usb_cam">
+      <visual>
+        <geometry>
+          <box size="0.05 0.05 0.05"/>
+        </geometry>
+        <material name="gray_solid"/>
+      </visual>
+  </link>
 </robot>

Commit message: Cleanup and add alphasense imu

File: box_model/box_model/urdf/box/box.urdf.xacro (robot description, xacro)
@@ -37,4 +37,5 @@
   </link>
   <!-- Box base -->
+  <link name="box_base"/>
   <joint name="box_to_box_base" type="fixed">
       <origin xyz="0.0 0.0 -0.1" rpy="0.0 0.0 0.0" />
@@ -42,7 +43,6 @@
       <child link="box_base" />
   </joint>
-  <link name="box_base">
-  </link>
   <!-- Box back -->
+  <link name="box_back"/>
   <joint name="box_to_box_back" type="fixed">
       <origin xyz="-0.4 0.0 -0.1" rpy="0.0 0.0 0.0" />
@@ -50,12 +50,5 @@
       <child link="box_back" />
   </joint>
-  <link name="box_back">
-  </link>
   <!-- GPS -->
-  <joint name="box_back_to_gps" type="fixed">
-      <origin xyz="-0.1 0.0 0.1" rpy="0.0 0.0 0.0" />
-      <parent link="box_back" />
-      <child link="gps" />
-  </joint>
   <link name="gps">
       <visual>
@@ -66,5 +59,18 @@
       </visual>
   </link>
+  <joint name="box_back_to_gps" type="fixed">
+      <origin xyz="-0.1 0.0 0.1" rpy="0.0 0.0 0.0" />
+      <parent link="box_back" />
+      <child link="gps" />
+  </joint>
   <!-- NUC -->
+  <link name="nuc">
+    <visual>
+      <geometry>
+        <box size="0.05 0.05 0.05"/>
+      </geometry>
+      <material name="gray_solid"/>
+    </visual>
+  </link>
   <joint name="box_back_to_nuc" type="fixed">
       <origin xyz="0.4 0.0 0.2" rpy="0.0 0.0 0.0" />
@@ -72,18 +78,5 @@
       <child link="nuc" />
   </joint>
-  <link name="nuc">
-      <visual>
-        <geometry>
-          <box size="0.05 0.05 0.05"/>
-        </geometry>
-        <material name="gray_solid"/>
-      </visual>
-    </link>
   <!-- Jetson -->
-  <joint name="box_back_to_jetson" type="fixed">
-    <origin xyz="0.5 0.0 0.2" rpy="0.0 0.0 0.0" />
-    <parent link="box_back" />
-    <child link="jetson" />
-  </joint>
   <link name="jetson">
       <visual>
@@ -94,10 +87,10 @@
       </visual>
   </link>
+  <joint name="box_back_to_jetson" type="fixed">
+    <origin xyz="0.5 0.0 0.2" rpy="0.0 0.0 0.0" />
+    <parent link="box_back" />
+    <child link="jetson" />
+  </joint>
   <!-- Reflector -->
-  <joint name="box_back_to_reflector" type="fixed">
-    <origin xyz="0.6 0.0 0.2" rpy="0.0 0.0 0.0" />
-    <parent link="box_back" />
-    <child link="reflector" />
-  </joint>
   <link name="reflector">
     <visual>
@@ -108,4 +101,9 @@
     </visual>
   </link>
+  <joint name="box_back_to_reflector" type="fixed">
+    <origin xyz="0.6 0.0 0.2" rpy="0.0 0.0 0.0" />
+    <parent link="box_back" />
+    <child link="reflector" />
+  </joint>
   <!-- Alphasense -->
   <xacro:property name="alphasense_calibration" value="$(find box_model)/urdf/box/calibrations/20220322_calibration.yaml" />
@@ -113,6 +111,12 @@
    <origin xyz="0.8 0 0.1" rpy="0 0 0" />
   </xacro:alphasense>
-  !-- This is the frame in which the ground truth is generated, conincides with the alphasense IMU -->
+  <!-- This is the frame in which the ground truth is generated, conincides with the alphasense IMU -->
   <link name="base"/>
+  <link name="imu_sensor_frame"/>
+  <joint name="alphasense_imu_mapping" type="fixed">
+    <origin xyz="0.0 0.0 0.0" rpy="0.0 0.0 0.0" />
+    <parent link="alphasense_imu"/>
+    <child link="imu_sensor_frame"/>
+  </joint>
   <joint name="alphasense_imu_to_base" type="fixed">
     <origin xyz="0.0 0.0 0.0" rpy="0.0 0.0 0.0" />
@@ -121,4 +125,5 @@
   </joint>
   <!-- Livox -->
+  <link name="livox_link"/>
   <joint name="box_back_to_livox_link" type="fixed">
       <origin xyz="0.8 0.0 0.2" rpy="0.0 0.0 0.0" />
@@ -126,9 +131,9 @@
       <child link="livox_link" />
   </joint>
-  <link name="livox_link"/>
-  <xacro:livox_device parent="livox_link" lidar_frame="mid360">
+  <xacro:livox_device parent="livox_link" lidar_frame="livox_frame">
     <origin xyz="0 0 0" rpy="${pi/2} ${-pi} 0" />
   </xacro:livox_device>
   <!-- Hesai -->
+  <link name="hesai_link"/>
   <joint name="box_back_to_hesai_link" type="fixed">
       <origin xyz="0.8 0.0 0.0" rpy="0.0 0.0 0.0" />
@@ -136,19 +141,13 @@
       <child link="hesai_link" />
   </joint>
-  <link name="hesai_link"/>
   <xacro:hesai_device parent="hesai_link" lidar_frame="PandarXT-32">
     <origin xyz="0 0 0" rpy="0 0 0"/>
   </xacro:hesai_device>
   <!-- USB Cam -->
+  <link name="usb_cam_link"/>
   <joint name="box_back_to_usb_cam_link" type="fixed">
       <origin xyz="0.8 0.0 0.25" rpy="0.0 0.0 0.0" />
       <parent link="box_back" />
       <child link="usb_cam_link" />
-  </joint>
-  <link name="usb_cam_link"/>
-  <joint name="usb_cam_link_to_usb_cam" type="fixed">
-      <origin xyz="0.0 0.0 0.0" rpy="0.0 ${-pi/4} 0.0" />
-      <parent link="usb_cam_link" />
-      <child link="usb_cam" />
   </joint>
   <link name="usb_cam">
@@ -160,3 +159,8 @@
       </visual>
   </link>
+  <joint name="usb_cam_link_to_usb_cam" type="fixed">
+      <origin xyz="0.0 0.0 0.0" rpy="0.0 ${-pi/4} 0.0" />
+      <parent link="usb_cam_link" />
+      <child link="usb_cam" />
+  </joint>
 </robot>

Commit message: Fix hesai frame

File: box_model/box_model/urdf/box/box.urdf.xacro (robot description, xacro)
@@ -127,15 +127,15 @@
   <link name="livox_link"/>
   <joint name="box_back_to_livox_link" type="fixed">
-      <origin xyz="0.8 0.0 0.2" rpy="0.0 0.0 0.0" />
+      <origin xyz="0.8 0.0 0.2" rpy="${pi/2} ${-pi} 0.0" />
       <parent link="box_back" />
       <child link="livox_link" />
   </joint>
   <xacro:livox_device parent="livox_link" lidar_frame="livox_frame">
-    <origin xyz="0 0 0" rpy="${pi/2} ${-pi} 0" />
+    <origin xyz="0 0 0" rpy="0 0 0" />
   </xacro:livox_device>
   <!-- Hesai -->
   <link name="hesai_link"/>
   <joint name="box_back_to_hesai_link" type="fixed">
-      <origin xyz="0.8 0.0 0.0" rpy="0.0 0.0 0.0" />
+      <origin xyz="0.8 0.0 0.0" rpy="0.0 0.0 ${pi}" />
       <parent link="box_back" />
       <child link="hesai_link" />

Commit message: Add adis imu frame

File: box_model/box_model/urdf/box/box.urdf.xacro (robot description, xacro)
@@ -164,3 +164,24 @@
       <child link="usb_cam" />
   </joint>
+  <!-- Adis IMU -->
+<!--  TODO: not calibrated-->
+  <link name="adis_imu_link">
+      <visual>
+        <geometry>
+          <box size="0.02 0.02 0.01"/>
+        </geometry>
+        <material name="gray_solid"/>
+      </visual>
+  </link>
+  <joint name="box_back_to_adis_imu_link" type="fixed">
+    <origin xyz="0.8 0.0 0.3" rpy="0.0 0.0 0.0" />
+    <parent link="box_back" />
+    <child link="adis_imu_link" />
+  </joint>
+  <link name="adis16475_link"/>
+  <joint name="adis_imu" type="fixed">
+      <origin xyz="0.0 0.0 0.0" rpy="0.0 0.0 0.0" />
+      <parent link="adis_imu_link" />
+      <child link="adis16475_link" />
+  </joint>
 </robot>

Commit message: add namespace and tf tree

File: box_model/box_model/urdf/box/box.urdf.xacro (robot description, xacro)
@@ -164,4 +164,24 @@
       <child link="usb_cam" />
   </joint>
+    <!-- IMU STIM320 -->
+  <link name="stim320_imu_link">
+      <visual>
+        <geometry>
+          <box size="0.02 0.02 0.01"/>
+        </geometry>
+        <material name="gray_solid"/>
+      </visual>
+  </link>
+  <joint name="box_back_to_stim320_imu_link" type="fixed">
+    <origin xyz="0.8 0.0 0.3" rpy="0.0 0.0 0.0" />
+    <parent link="box_back" />
+    <child link="stim320_imu_link" />
+  </joint>
+  <link name="STIM320"/>
+  <joint name="stim320_imu" type="fixed">
+      <origin xyz="0.0 0.0 0.0" rpy="0.0 0.0 0.0" />
+      <parent link="stim320_imu_link" />
+      <child link="STIM320" />
+  </joint>
   <!-- Adis IMU -->
 <!--  TODO: not calibrated-->

Commit message: new urdf, with data read by yaml file

File: box_model/box_model/urdf/box/box.urdf.xacro (robot description, xacro)
@@ -13,4 +13,8 @@
 -->
 <robot name="box" xmlns:xacro="http://www.ros.org/wiki/xacro">
+<!-- YAML file containing the default values from CAD -->
+<xacro:property name="default_calib" value="$(find box_model)/urdf/box/calibrations/default_calibration.yaml" />
+<!-- load the YAML calibration file into a property -->
+<xacro:property name="calib" value="${xacro.load_yaml(default_calib)}"/>
   <!-- Origin -->
   <link name="origin"/>
@@ -38,5 +42,10 @@
   <link name="cameras_front" />
   <joint name="box_base_to_cameras_front" type="fixed">
-    <origin xyz="0.45 0.0 0.09" rpy="0.0 0.0 0.0" />
+    <origin xyz=" ${calib['box_base_to_cameras_front']['x']}
+                  ${calib['box_base_to_cameras_front']['y']}
+                  ${calib['box_base_to_cameras_front']['z']}"
+            rpy=" ${calib['box_base_to_cameras_front']['roll']}
+                  ${calib['box_base_to_cameras_front']['pitch']}
+                  ${calib['box_base_to_cameras_front']['yaw']}" />
     <parent link="box_base" />
     <child link="cameras_front" />
@@ -45,5 +54,10 @@
   <link name="hdr_front" />
   <joint name="cameras_front_to_hdr_front" type="fixed">
-    <origin xyz="0.0 0.0 0.0" rpy="${-pi/2} 0.0 ${-pi/2}" />
+    <origin xyz=" ${calib['cameras_front_to_hdr_front']['x']}
+                  ${calib['cameras_front_to_hdr_front']['y']}
+                  ${calib['cameras_front_to_hdr_front']['z']}"
+            rpy=" ${calib['cameras_front_to_hdr_front']['roll']}
+                  ${calib['cameras_front_to_hdr_front']['pitch']}
+                  ${calib['cameras_front_to_hdr_front']['yaw']}" />
     <parent link="cameras_front" />
     <child link="hdr_front" />
@@ -52,5 +66,10 @@
   <link name="alphasense_front_left" />
   <joint name="hdr_front_to_alphasense_front_left" type="fixed">
-    <origin xyz="-0.055 -0.04 0.0" rpy="0.0 0.0 0.0" />
+    <origin xyz=" ${calib['hdr_front_to_alphasense_front_left']['x']}
+                  ${calib['hdr_front_to_alphasense_front_left']['y']}
+                  ${calib['hdr_front_to_alphasense_front_left']['z']}"
+            rpy=" ${calib['hdr_front_to_alphasense_front_left']['roll']}
+                  ${calib['hdr_front_to_alphasense_front_left']['pitch']}
+                  ${calib['hdr_front_to_alphasense_front_left']['yaw']}" />
     <parent link="hdr_front" />
     <child link="alphasense_front_left" />
@@ -59,5 +78,10 @@
   <link name="alphasense_front_middle" />
   <joint name="alphasense_front_left_to_alphasense_front_middle" type="fixed">
-    <origin xyz="0.054 0.0 0.0" rpy="0.0 0.0 0.0" />
+    <origin xyz=" ${calib['alphasense_front_left_to_alphasense_front_middle']['x']}
+                  ${calib['alphasense_front_left_to_alphasense_front_middle']['y']}
+                  ${calib['alphasense_front_left_to_alphasense_front_middle']['z']}"
+            rpy=" ${calib['alphasense_front_left_to_alphasense_front_middle']['roll']}
+                  ${calib['alphasense_front_left_to_alphasense_front_middle']['pitch']}
+                  ${calib['alphasense_front_left_to_alphasense_front_middle']['yaw']}" />
     <parent link="alphasense_front_left" />
     <child link="alphasense_front_middle" />
@@ -66,5 +90,10 @@
   <link name="alphasense_front_right" />
   <joint name="alphasense_front_middle_to_alphasense_front_right" type="fixed">
-    <origin xyz="0.054 0.0 0.0" rpy="0.0 0.0 0.0" />
+    <origin xyz=" ${calib['alphasense_front_middle_to_alphasense_front_right']['x']}
+                  ${calib['alphasense_front_middle_to_alphasense_front_right']['y']}
+                  ${calib['alphasense_front_middle_to_alphasense_front_right']['z']}"
+            rpy=" ${calib['alphasense_front_middle_to_alphasense_front_right']['roll']}
+                  ${calib['alphasense_front_middle_to_alphasense_front_right']['pitch']}
+                  ${calib['alphasense_front_middle_to_alphasense_front_right']['yaw']}" />
     <parent link="alphasense_front_middle" />
     <child link="alphasense_front_right" />
@@ -73,5 +102,10 @@
   <link name="zed_right" />
   <joint name="alphasense_front_right_to_zed_right" type="fixed">
-    <origin xyz="0.005 0.08 0.0" rpy="0.0 0.0 0.0" />
+    <origin xyz=" ${calib['alphasense_front_right_to_zed_right']['x']}
+                  ${calib['alphasense_front_right_to_zed_right']['y']}
+                  ${calib['alphasense_front_right_to_zed_right']['z']}"
+            rpy=" ${calib['alphasense_front_right_to_zed_right']['roll']}
+                  ${calib['alphasense_front_right_to_zed_right']['pitch']}
+                  ${calib['alphasense_front_right_to_zed_right']['yaw']}" />
     <parent link="alphasense_front_right" />
     <child link="zed_right" />
@@ -80,5 +114,10 @@
   <link name="zed_left" />
   <joint name="zed_right_to_zed_left" type="fixed">
-    <origin xyz="-0.12 0.0 0.0" rpy="0.0 0.0 0.0" />
+    <origin xyz=" ${calib['zed_right_to_zed_left']['x']}
+                  ${calib['zed_right_to_zed_left']['y']}
+                  ${calib['zed_right_to_zed_left']['z']}"
+            rpy=" ${calib['zed_right_to_zed_left']['roll']}
+                  ${calib['zed_right_to_zed_left']['pitch']}
+                  ${calib['zed_right_to_zed_left']['yaw']}" />
     <parent link="zed_right" />
     <child link="zed_left" />
@@ -87,5 +126,10 @@
   <link name="cameras_right" />
   <joint name="box_base_to_cameras_right" type="fixed">
-    <origin xyz="0.37 -0.10 0.09" rpy="0.0 0.0 0.0" />
+    <origin xyz=" ${calib['box_base_to_cameras_right']['x']}
+                  ${calib['box_base_to_cameras_right']['y']}
+                  ${calib['box_base_to_cameras_right']['z']}"
+            rpy=" ${calib['box_base_to_cameras_right']['roll']}
+                  ${calib['box_base_to_cameras_right']['pitch']}
+                  ${calib['box_base_to_cameras_right']['yaw']}" />
     <parent link="box_base" />
     <child link="cameras_right" />
@@ -94,5 +138,10 @@
   <link name="hdr_right" />
   <joint name="cameras_right_to_hdr_right" type="fixed">
-    <origin xyz="0.0 0.0 0.0" rpy="${pi/2} ${pi} 0.0" />
+    <origin xyz=" ${calib['cameras_right_to_hdr_right']['x']}
+                  ${calib['cameras_right_to_hdr_right']['y']}
+                  ${calib['cameras_right_to_hdr_right']['z']}"
+            rpy=" ${calib['cameras_right_to_hdr_right']['roll']}
+                  ${calib['cameras_right_to_hdr_right']['pitch']}
+                  ${calib['cameras_right_to_hdr_right']['yaw']}" />
     <parent link="cameras_right" />
     <child link="hdr_right" />
@@ -100,5 +149,10 @@
   <link name="alphasense_right" />
   <joint name="hdr_right_to_alphasense_right" type="fixed">
-    <origin xyz="0.0 -0.04 0.0" rpy="0.0 0.0 0.0" />
+    <origin xyz=" ${calib['hdr_right_to_alphasense_right']['x']}
+                  ${calib['hdr_right_to_alphasense_right']['y']}
+                  ${calib['hdr_right_to_alphasense_right']['z']}"
+            rpy=" ${calib['hdr_right_to_alphasense_right']['roll']}
+                  ${calib['hdr_right_to_alphasense_right']['pitch']}
+                  ${calib['hdr_right_to_alphasense_right']['yaw']}" />
     <parent link="hdr_right" />
     <child link="alphasense_right" />
@@ -107,5 +161,10 @@
   <link name="cameras_left" />
   <joint name="box_base_to_cameras_left" type="fixed">
-    <origin xyz="0.37 0.10 0.09" rpy="0.0 0.0 0.0" />
+    <origin xyz=" ${calib['box_base_to_cameras_left']['x']}
+                  ${calib['box_base_to_cameras_left']['y']}
+                  ${calib['box_base_to_cameras_left']['z']}"
+            rpy=" ${calib['box_base_to_cameras_left']['roll']}
+                  ${calib['box_base_to_cameras_left']['pitch']}
+                  ${calib['box_base_to_cameras_left']['yaw']}" />
     <parent link="box_base" />
     <child link="cameras_left" />
@@ -114,5 +173,10 @@
   <link name="hdr_left" />
   <joint name="cameras_left_to_hdr_left" type="fixed">
-    <origin xyz="0.0 0.0 0.0" rpy="-${pi/2} 0.0 0.0" />
+    <origin xyz=" ${calib['cameras_left_to_hdr_left']['x']}
+                  ${calib['cameras_left_to_hdr_left']['y']}
+                  ${calib['cameras_left_to_hdr_left']['z']}"
+            rpy=" ${calib['cameras_left_to_hdr_left']['roll']}
+                  ${calib['cameras_left_to_hdr_left']['pitch']}
+                  ${calib['cameras_left_to_hdr_left']['yaw']}" />
     <parent link="cameras_left" />
     <child link="hdr_left" />
@@ -121,5 +185,10 @@
   <link name="alphasense_left" />
   <joint name="hdr_left_to_alphasense_left" type="fixed">
-    <origin xyz="0.0 -0.04 0.0" rpy="0.0 0.0 0.0" />
+    <origin xyz=" ${calib['hdr_left_to_alphasense_left']['x']}
+                  ${calib['hdr_left_to_alphasense_left']['y']}
+                  ${calib['hdr_left_to_alphasense_left']['z']}"
+            rpy=" ${calib['hdr_left_to_alphasense_left']['roll']}
+                  ${calib['hdr_left_to_alphasense_left']['pitch']}
+                  ${calib['hdr_left_to_alphasense_left']['yaw']}" />
     <parent link="hdr_left" />
     <child link="alphasense_left" />
@@ -128,5 +197,10 @@
   <link name="lidars" />
   <joint name="box_base_to_lidars" type="fixed">
-    <origin xyz="0.37 0.0 0.2" rpy="0.0 0.0 0.0" />
+    <origin xyz=" ${calib['box_base_to_lidars']['x']}
+                  ${calib['box_base_to_lidars']['y']}
+                  ${calib['box_base_to_lidars']['z']}"
+            rpy=" ${calib['box_base_to_lidars']['roll']}
+                  ${calib['box_base_to_lidars']['pitch']}
+                  ${calib['box_base_to_lidars']['yaw']}" />
     <parent link="box_base" />
     <child link="lidars" />
@@ -135,5 +209,10 @@
   <link name="hesai" />
   <joint name="lidars_to_hesai" type="fixed">
-    <origin xyz="0.0 0.0 0.0" rpy="0.0 0.0 ${pi/2}" />
+    <origin xyz=" ${calib['lidars_to_hesai']['x']}
+                  ${calib['lidars_to_hesai']['y']}
+                  ${calib['lidars_to_hesai']['z']}"
+            rpy=" ${calib['lidars_to_hesai']['roll']}
+                  ${calib['lidars_to_hesai']['pitch']}
+                  ${calib['lidars_to_hesai']['yaw']}" />
     <parent link="lidars" />
     <child link="hesai" />
@@ -142,5 +221,10 @@
   <link name="livox" />
   <joint name="hesai_to_livox" type="fixed">
-    <origin xyz="0.0 0.0 0.10" rpy="${pi} 0.0 ${-pi/2}" />
+    <origin xyz=" ${calib['hesai_to_livox']['x']}
+                  ${calib['hesai_to_livox']['y']}
+                  ${calib['hesai_to_livox']['z']}"
+            rpy=" ${calib['hesai_to_livox']['roll']}
+                  ${calib['hesai_to_livox']['pitch']}
+                  ${calib['hesai_to_livox']['yaw']}" />
     <parent link="hesai" />
     <child link="livox" />
