Commit message: put lidar and camera urdf in seperate files

File: box_model/box_model/urdf/box/box.urdf.xacro (robot description, xacro)
@@ -1,15 +1,3 @@
 <?xml version="1.0" ?>
-<!--
-Copyright 2022 University of Oxford, Hilti Corporation
-Licensed under the Apache License, Version 2.0 (the "License");
-you may not use this file except in compliance with the License.
-You may obtain a copy of the License at
-    http://www.apache.org/licenses/LICENSE-2.0
-Unless required by applicable law or agreed to in writing, software
-distributed under the License is distributed on an "AS IS" BASIS,
-WITHOUT WARRANTIES OR CONDITIONS OF ANY KIND, either express or implied.
-See the License for the specific language governing permissions and
-limitations under the License.
--->
 <robot name="box" xmlns:xacro="http://www.ros.org/wiki/xacro">
 <!-- YAML file containing the default values from CAD -->
@@ -39,194 +27,5 @@
     <child link="model_base" />
   </joint>
-  <!-- Cameras front (coincide with front hdr cam) -->
-  <link name="cameras_front" />
-  <joint name="box_base_to_cameras_front" type="fixed">
-    <origin xyz=" ${calib['box_base_to_cameras_front']['x']}
-                  ${calib['box_base_to_cameras_front']['y']}
-                  ${calib['box_base_to_cameras_front']['z']}"
-            rpy=" ${calib['box_base_to_cameras_front']['roll']}
-                  ${calib['box_base_to_cameras_front']['pitch']}
-                  ${calib['box_base_to_cameras_front']['yaw']}" />
-    <parent link="box_base" />
-    <child link="cameras_front" />
-  </joint>
-  <!-- HDR camera front -->
-  <link name="hdr_front" />
-  <joint name="cameras_front_to_hdr_front" type="fixed">
-    <origin xyz=" ${calib['cameras_front_to_hdr_front']['x']}
-                  ${calib['cameras_front_to_hdr_front']['y']}
-                  ${calib['cameras_front_to_hdr_front']['z']}"
-            rpy=" ${calib['cameras_front_to_hdr_front']['roll']}
-                  ${calib['cameras_front_to_hdr_front']['pitch']}
-                  ${calib['cameras_front_to_hdr_front']['yaw']}" />
-    <parent link="cameras_front" />
-    <child link="hdr_front" />
-  </joint>
-  <!-- Alphasense front left -->
-  <link name="alphasense_front_left" />
-  <joint name="hdr_front_to_alphasense_front_left" type="fixed">
-    <origin xyz=" ${calib['hdr_front_to_alphasense_front_left']['x']}
-                  ${calib['hdr_front_to_alphasense_front_left']['y']}
-                  ${calib['hdr_front_to_alphasense_front_left']['z']}"
-            rpy=" ${calib['hdr_front_to_alphasense_front_left']['roll']}
-                  ${calib['hdr_front_to_alphasense_front_left']['pitch']}
-                  ${calib['hdr_front_to_alphasense_front_left']['yaw']}" />
-    <parent link="hdr_front" />
-    <child link="alphasense_front_left" />
-  </joint>
-  <!-- Alphasense front middle -->
-  <link name="alphasense_front_middle" />
-  <joint name="alphasense_front_left_to_alphasense_front_middle" type="fixed">
-    <origin xyz=" ${calib['alphasense_front_left_to_alphasense_front_middle']['x']}
-                  ${calib['alphasense_front_left_to_alphasense_front_middle']['y']}
-                  ${calib['alphasense_front_left_to_alphasense_front_middle']['z']}"
-            rpy=" ${calib['alphasense_front_left_to_alphasense_front_middle']['roll']}
-                  ${calib['alphasense_front_left_to_alphasense_front_middle']['pitch']}
-                  ${calib['alphasense_front_left_to_alphasense_front_middle']['yaw']}" />
-    <parent link="alphasense_front_left" />
-    <child link="alphasense_front_middle" />
-  </joint>
-  <!-- Alphasense front right -->
-  <link name="alphasense_front_right" />
-  <joint name="alphasense_front_middle_to_alphasense_front_right" type="fixed">
-    <origin xyz=" ${calib['alphasense_front_middle_to_alphasense_front_right']['x']}
-                  ${calib['alphasense_front_middle_to_alphasense_front_right']['y']}
-                  ${calib['alphasense_front_middle_to_alphasense_front_right']['z']}"
-            rpy=" ${calib['alphasense_front_middle_to_alphasense_front_right']['roll']}
-                  ${calib['alphasense_front_middle_to_alphasense_front_right']['pitch']}
-                  ${calib['alphasense_front_middle_to_alphasense_front_right']['yaw']}" />
-    <parent link="alphasense_front_middle" />
-    <child link="alphasense_front_right" />
-  </joint>
-  <!-- Zed right -->
-  <link name="zed_right" />
-  <joint name="alphasense_front_right_to_zed_right" type="fixed">
-    <origin xyz=" ${calib['alphasense_front_right_to_zed_right']['x']}
-                  ${calib['alphasense_front_right_to_zed_right']['y']}
-                  ${calib['alphasense_front_right_to_zed_right']['z']}"
-            rpy=" ${calib['alphasense_front_right_to_zed_right']['roll']}
-                  ${calib['alphasense_front_right_to_zed_right']['pitch']}
-                  ${calib['alphasense_front_right_to_zed_right']['yaw']}" />
-    <parent link="alphasense_front_right" />
-    <child link="zed_right" />
-  </joint>
-  <!-- Zed left -->
-  <link name="zed_left" />
-  <joint name="zed_right_to_zed_left" type="fixed">
-    <origin xyz=" ${calib['zed_right_to_zed_left']['x']}
-                  ${calib['zed_right_to_zed_left']['y']}
-                  ${calib['zed_right_to_zed_left']['z']}"
-            rpy=" ${calib['zed_right_to_zed_left']['roll']}
-                  ${calib['zed_right_to_zed_left']['pitch']}
-                  ${calib['zed_right_to_zed_left']['yaw']}" />
-    <parent link="zed_right" />
-    <child link="zed_left" />
-  </joint>
-  <!-- Cameras right (coincide with right hdr cam) -->
-  <link name="cameras_right" />
-  <joint name="box_base_to_cameras_right" type="fixed">
-    <origin xyz=" ${calib['box_base_to_cameras_right']['x']}
-                  ${calib['box_base_to_cameras_right']['y']}
-                  ${calib['box_base_to_cameras_right']['z']}"
-            rpy=" ${calib['box_base_to_cameras_right']['roll']}
-                  ${calib['box_base_to_cameras_right']['pitch']}
-                  ${calib['box_base_to_cameras_right']['yaw']}" />
-    <parent link="box_base" />
-    <child link="cameras_right" />
-  </joint>
-  <!-- HDR camera right -->
-  <link name="hdr_right" />
-  <joint name="cameras_right_to_hdr_right" type="fixed">
-    <origin xyz=" ${calib['cameras_right_to_hdr_right']['x']}
-                  ${calib['cameras_right_to_hdr_right']['y']}
-                  ${calib['cameras_right_to_hdr_right']['z']}"
-            rpy=" ${calib['cameras_right_to_hdr_right']['roll']}
-                  ${calib['cameras_right_to_hdr_right']['pitch']}
-                  ${calib['cameras_right_to_hdr_right']['yaw']}" />
-    <parent link="cameras_right" />
-    <child link="hdr_right" />
-  </joint>
-  <link name="alphasense_right" />
-  <joint name="hdr_right_to_alphasense_right" type="fixed">
-    <origin xyz=" ${calib['hdr_right_to_alphasense_right']['x']}
-                  ${calib['hdr_right_to_alphasense_right']['y']}
-                  ${calib['hdr_right_to_alphasense_right']['z']}"
-            rpy=" ${calib['hdr_right_to_alphasense_right']['roll']}
-                  ${calib['hdr_right_to_alphasense_right']['pitch']}
-                  ${calib['hdr_right_to_alphasense_right']['yaw']}" />
-    <parent link="hdr_right" />
-    <child link="alphasense_right" />
-  </joint>
-  <!-- Cameras left (coincide with left hdr cam) -->
-  <link name="cameras_left" />
-  <joint name="box_base_to_cameras_left" type="fixed">
-    <origin xyz=" ${calib['box_base_to_cameras_left']['x']}
-                  ${calib['box_base_to_cameras_left']['y']}
-                  ${calib['box_base_to_cameras_left']['z']}"
-            rpy=" ${calib['box_base_to_cameras_left']['roll']}
-                  ${calib['box_base_to_cameras_left']['pitch']}
-                  ${calib['box_base_to_cameras_left']['yaw']}" />
-    <parent link="box_base" />
-    <child link="cameras_left" />
-  </joint>
-  <!-- HDR camera left -->
-  <link name="hdr_left" />
-  <joint name="cameras_left_to_hdr_left" type="fixed">
-    <origin xyz=" ${calib['cameras_left_to_hdr_left']['x']}
-                  ${calib['cameras_left_to_hdr_left']['y']}
-                  ${calib['cameras_left_to_hdr_left']['z']}"
-            rpy=" ${calib['cameras_left_to_hdr_left']['roll']}
-                  ${calib['cameras_left_to_hdr_left']['pitch']}
-                  ${calib['cameras_left_to_hdr_left']['yaw']}" />
-    <parent link="cameras_left" />
-    <child link="hdr_left" />
-  </joint>
-  <!-- Alphasense left -->
-  <link name="alphasense_left" />
-  <joint name="hdr_left_to_alphasense_left" type="fixed">
-    <origin xyz=" ${calib['hdr_left_to_alphasense_left']['x']}
-                  ${calib['hdr_left_to_alphasense_left']['y']}
-                  ${calib['hdr_left_to_alphasense_left']['z']}"
-            rpy=" ${calib['hdr_left_to_alphasense_left']['roll']}
-                  ${calib['hdr_left_to_alphasense_left']['pitch']}
-                  ${calib['hdr_left_to_alphasense_left']['yaw']}" />
-    <parent link="hdr_left" />
-    <child link="alphasense_left" />
-  </joint>
-  <!-- Lidars (coincide with hesai) -->
-  <link name="lidars" />
-  <joint name="box_base_to_lidars" type="fixed">
-    <origin xyz=" ${calib['box_base_to_lidars']['x']}
-                  ${calib['box_base_to_lidars']['y']}
-                  ${calib['box_base_to_lidars']['z']}"
-            rpy=" ${calib['box_base_to_lidars']['roll']}
-                  ${calib['box_base_to_lidars']['pitch']}
-                  ${calib['box_base_to_lidars']['yaw']}" />
-    <parent link="box_base" />
-    <child link="lidars" />
-  </joint>
-  <!-- HDR camera left -->
-  <link name="hesai" />
-  <joint name="lidars_to_hesai" type="fixed">
-    <origin xyz=" ${calib['lidars_to_hesai']['x']}
-                  ${calib['lidars_to_hesai']['y']}
-                  ${calib['lidars_to_hesai']['z']}"
-            rpy=" ${calib['lidars_to_hesai']['roll']}
-                  ${calib['lidars_to_hesai']['pitch']}
-                  ${calib['lidars_to_hesai']['yaw']}" />
-    <parent link="lidars" />
-    <child link="hesai" />
-  </joint>
-  <!-- Alphasense left -->
-  <link name="livox" />
-  <joint name="hesai_to_livox" type="fixed">
-    <origin xyz=" ${calib['hesai_to_livox']['x']}
-                  ${calib['hesai_to_livox']['y']}
-                  ${calib['hesai_to_livox']['z']}"
-            rpy=" ${calib['hesai_to_livox']['roll']}
-                  ${calib['hesai_to_livox']['pitch']}
-                  ${calib['hesai_to_livox']['yaw']}" />
-    <parent link="hesai" />
-    <child link="livox" />
-  </joint>
+  <xacro:include filename="$(find box_model)/urdf/cameras/cameras.urdf.xacro" />
+  <xacro:include filename="$(find box_model)/urdf/lidars/lidars.urdf.xacro" />
 </robot>

Commit message: add position by totalstation

File: box_model/box_model/urdf/box/box.urdf.xacro (robot description, xacro)
@@ -6,10 +6,24 @@
 <xacro:property name="calib" value="${xacro.load_yaml(default_calib)}"/>
   <!-- Origin -->
-  <link name="origin"/>
+  <link name="leica_world"/>
+  <!-- Measured prism position -->
+  <link name="leica_pos"/>
+  <joint name="leica_world_to_leica_pos" type="fixed">
+    <origin xyz="0.0 0.0 0.0" rpy="0.0 0.0 0.0" />
+    <parent link="leica_world" />
+    <child link="leica_pos" />
+  </joint>
+  <!-- Prism -->
+  <link name="prism"/>
+  <joint name="leica_pos_to_prism" type="fixed">
+    <origin xyz="0.15 0.0 -0.3" rpy="0.0 0.0 0.0" />
+    <parent link="leica_pos" />
+    <child link="prism" />
+  </joint>
   <!-- Box base -->
   <link name="box_base"/>
-  <joint name="origin_to_box_base" type="fixed">
+  <joint name="prism_to_box_base" type="fixed">
     <origin xyz="0.0 0.0 0.0" rpy="0.0 0.0 0.0" />
-    <parent link="origin" />
+    <parent link="prism" />
     <child link="box_base" />
   </joint>

Commit message: works

File: box_model/box_model/urdf/box/box.urdf.xacro (robot description, xacro)
@@ -7,4 +7,17 @@
   <!-- Origin -->
   <link name="leica_world"/>
+  <!-- Totalstation base position -->
+  <link name="leica_base"/>
+  <joint name="leica_world_to_leica_base" type="fixed">
+    <origin xyz="0.1 0.1 0.1" rpy="0.0 0.0 0.0" />
+    <parent link="leica_world" />
+    <child link="leica_base" />
+  </joint>
+  <link name="leica_base_model"/>
+  <joint name="leica_base_to_leica_base_model" type="fixed">
+    <origin xyz="0.0 0.0 0.0" rpy="0.0 0.0 0.0" />
+    <parent link="leica_base" />
+    <child link="leica_base_model" />
+  </joint>
   <!-- Measured prism position -->
   <link name="leica_pos"/>

Commit message: totalstation model

File: box_model/box_model/urdf/box/box.urdf.xacro (robot description, xacro)
@@ -10,9 +10,16 @@
   <link name="leica_base"/>
   <joint name="leica_world_to_leica_base" type="fixed">
-    <origin xyz="0.1 0.1 0.1" rpy="0.0 0.0 0.0" />
+    <origin xyz="1.0 1.0 1.0" rpy="0.0 0.0 0.0" />
     <parent link="leica_world" />
     <child link="leica_base" />
   </joint>
-  <link name="leica_base_model"/>
+  <!-- Totalstation model -->
+  <link name="leica_base_model">
+    <visual>
+      <geometry>
+        <cylinder length="0.2" radius="0.08"/>
+      </geometry>
+    </visual>
+  </link>
   <joint name="leica_base_to_leica_base_model" type="fixed">
     <origin xyz="0.0 0.0 0.0" rpy="0.0 0.0 0.0" />

Commit message: position imus and prism

File: box_model/box_model/urdf/box/box.urdf.xacro (robot description, xacro)
@@ -27,8 +27,8 @@
     <child link="leica_base_model" />
   </joint>
-  <!-- Measured prism position -->
+  <!-- Measured prism position, changes when totalstation is tracking -->
   <link name="leica_pos"/>
   <joint name="leica_world_to_leica_pos" type="fixed">
-    <origin xyz="0.0 0.0 0.0" rpy="0.0 0.0 0.0" />
+    <origin xyz="0.15 0.0 -0.3" rpy="0.0 0.0 0.0" />
     <parent link="leica_world" />
     <child link="leica_pos" />
@@ -37,5 +37,5 @@
   <link name="prism"/>
   <joint name="leica_pos_to_prism" type="fixed">
-    <origin xyz="0.15 0.0 -0.3" rpy="0.0 0.0 0.0" />
+    <origin xyz="0.0 0.0 0.0" rpy="0.0 0.0 0.0" />
     <parent link="leica_pos" />
     <child link="prism" />
@@ -44,5 +44,5 @@
   <link name="box_base"/>
   <joint name="prism_to_box_base" type="fixed">
-    <origin xyz="0.0 0.0 0.0" rpy="0.0 0.0 0.0" />
+    <origin xyz="-0.075 0.0 -0.15" rpy="0.0 0.0 0.0" />
     <parent link="prism" />
     <child link="box_base" />

Commit message: calib_importer.py script works from command line.

File: box_model/box_model/urdf/box/box.urdf.xacro (robot description, xacro)
@@ -2,7 +2,7 @@
 <robot name="box" xmlns:xacro="http://www.ros.org/wiki/xacro">
 <!-- YAML file containing the default values from CAD -->
-<xacro:property name="default_calib" value="$(find box_model)/urdf/box/calibrations/default_calibration.yaml" />
+<xacro:property name="calib_file" value="$(find box_model)/urdf/box/calibrations/calibration.yaml" />
 <!-- load the YAML calibration file into a property -->
-<xacro:property name="calib" value="${xacro.load_yaml(default_calib)}"/>
+<xacro:property name="calib" value="${xacro.load_yaml(calib_file)}"/>
   <!-- Origin -->
   <link name="leica_world"/>

Commit message: Replaced default calibration data with new field names

File: box_model/box_model/urdf/box/box.urdf.xacro (robot description, xacro)
@@ -44,5 +44,10 @@
   <link name="box_base"/>
   <joint name="prism_to_box_base" type="fixed">
-    <origin xyz="-0.075 0.0 -0.15" rpy="0.0 0.0 0.0" />
+    <origin xyz=" ${calib['prism_to_box_base']['x']}
+                  ${calib['prism_to_box_base']['y']}
+                  ${calib['prism_to_box_base']['z']}"
+            rpy=" ${calib['prism_to_box_base']['roll']}
+                  ${calib['prism_to_box_base']['pitch']}
+                  ${calib['prism_to_box_base']['yaw']}" />
     <parent link="prism" />
     <child link="box_base" />

File: box_model/box_model/urdf/cameras/cameras.urdf.xacro (robot description, xacro)
@@ -124,5 +124,5 @@
   </joint>
   <!-- ////////// ZED2i ////////// -->
-  <!-- ZED Base (coincides with Zed2i right cam) -->
+  <!-- ZED Base -->
   <link name="zed_base" />
   <joint name="box_base_to_zed_base" type="fixed">
@@ -136,27 +136,4 @@
     <child link="zed_base" />
   </joint>
-  <!-- Zed right (should be identity)-->
-  <link name="zed_right" />
-  <joint name="zed_base_to_zed_right" type="fixed">
-    <origin xyz=" ${calib['zed_base_to_zed_right']['x']}
-                  ${calib['zed_base_to_zed_right']['y']}
-                  ${calib['zed_base_to_zed_right']['z']}"
-            rpy=" ${calib['zed_base_to_zed_right']['roll']}
-                  ${calib['zed_base_to_zed_right']['pitch']}
-                  ${calib['zed_base_to_zed_right']['yaw']}" />
-    <parent link="zed_base" />
-    <child link="zed_right" />
-  </joint>
-  <!-- Zed left (parent is zed_right not zed_base because we use the zed2i calib data) -->
-  <link name="zed_left" />
-  <joint name="zed_right_to_zed_left" type="fixed">
-    <origin xyz=" ${calib['zed_right_to_zed_left']['x']}
-                  ${calib['zed_right_to_zed_left']['y']}
-                  ${calib['zed_right_to_zed_left']['z']}"
-            rpy=" ${calib['zed_right_to_zed_left']['roll']}
-                  ${calib['zed_right_to_zed_left']['pitch']}
-                  ${calib['zed_right_to_zed_left']['yaw']}" />
-    <parent link="zed_right" />
-    <child link="zed_left" />
-  </joint>
+  <!-- Zed right and left from from Zed2i TF Publisher -->
 </robot>

Commit message: Adding new meshes to box model

File: box_model/box_model/urdf/box/box.urdf.xacro (robot description, xacro)
@@ -54,15 +54,27 @@
   </joint>
   <!-- Model base -->
-  <link name="model_base">
+  <link name="box_base_model">
     <visual>
       <geometry>
-        <mesh filename="package://box_model/urdf/box/mesh/box_model1.dae" />
+        <mesh filename="package://box_model/urdf/box/mesh/box_assembly_incl_livox_mount.dae" />
       </geometry>
     </visual>
   </link>
-  <joint name="box_base_to_model_base" type="fixed">
-    <origin xyz="0.0 0.0 0.0" rpy="${pi} 0.0 ${pi/2}" />
+  <joint name="box_base_to_box_base_model" type="fixed">
+    <origin xyz="0.0 0.0 0.0" rpy="0.0 0.0 0.0" />
     <parent link="box_base" />
-    <child link="model_base" />
+    <child link="box_base_model" />
+  </joint>
+  <link name="prism_model">
+    <visual>
+      <geometry>
+        <mesh filename="package://box_model/urdf/box/mesh/leica_small_prism.dae" />
+      </geometry>
+    </visual>
+  </link>
+  <joint name="prism_to_prism_model" type="fixed">
+    <origin xyz="0.0 0.0 0.0" rpy="0.0 0.0 0.0" />
+    <parent link="box_base" />
+    <child link="prism_model" />
   </joint>
   <xacro:include filename="$(find box_model)/urdf/cameras/cameras.urdf.xacro" />

File: box_model/box_model/urdf/lidars/lidars.urdf.xacro (robot description, xacro)
@@ -13,4 +13,16 @@
     <child link="hesaiXT32" />
   </joint>
+  <link name="hesaiXT32_model">
+    <visual>
+      <geometry>
+        <mesh filename="package://box_model/urdf/box/mesh/hesai_lidar.dae" />
+      </geometry>
+    </visual>
+  </link>
+  <joint name="hesaiXT32_to_hesaiXT32_model" type="fixed">
+    <origin xyz="0.0 0.0 0.0" rpy="0.0 0.0 0.0" />
+    <parent link="hesaiXT32" />
+    <child link="hesaiXT32_model" />
+  </joint>
   <!-- Livox -->
   <link name="livox" />
@@ -25,3 +37,15 @@
     <child link="livox" />
   </joint>
+  <link name="livox_model">
+    <visual>
+      <geometry>
+        <mesh filename="package://box_model/urdf/box/mesh/livox_mid360_lidar.dae" />
+      </geometry>
+    </visual>
+  </link>
+  <joint name="livox_to_livox_model" type="fixed">
+    <origin xyz="0.0 0.0 0.0" rpy="0.0 0.0 0.0" />
+    <parent link="livox" />
+    <child link="livox_model" />
+  </joint>
 </robot>

Commit message: Fix lidar imu xacro and add CPT7 and Basilisk frames to URDF

File: box_model/box_model/urdf/box/box.urdf.xacro (robot description, xacro)
@@ -78,4 +78,18 @@
     <child link="prism_model" />
   </joint>
+  <link name="cpt7_imu"/>
+  <!-- CPT7 Coordinate System -->
+  <joint name="base_to_cpt7_imu_frame" type="fixed">
+    <origin xyz="-0.294 -0.058 0.164" rpy="3.142 0.0 0.0" />
+    <parent link="box_base" />
+    <child link="cpt7_imu" />
+  </joint>
+  <link name="State"/>
+  <!-- Basilisk IMU Frame -->
+  <joint name="base_to_basilisk_imu_frame" type="fixed">
+    <origin xyz="-0.293 0.034 0.155" rpy="1.571 0.0 0.0" />
+    <parent link="box_base" />
+    <child link="State" />
+  </joint>
   <xacro:include filename="$(find box_model)/urdf/cameras/cameras.urdf.xacro" />
   <xacro:include filename="$(find box_model)/urdf/lidars/lidars.urdf.xacro" />

File: box_model/box_model/urdf/lidars/lidars.urdf.xacro (robot description, xacro)
@@ -49,5 +49,5 @@
     <child link="livox_model" />
   </joint>
-  <link name="livox_frame">
+  <link name="livox_frame"/>
   <!-- From page 15 https://terra-1-g.djicdn.com/851d20f7b9f64838a34cd02351370894/Livox/Livox_Mid-360_User_Manual_EN.pdf -->
   <joint name="livox_to_livox_imu_frame" type="fixed">

Commit message: updated calibration structure

File: box_model/box_model/urdf/box/box.urdf.xacro (robot description, xacro)
@@ -2,5 +2,5 @@
 <robot name="box" xmlns:xacro="http://www.ros.org/wiki/xacro">
 <!-- YAML file containing the default values from CAD -->
-<xacro:property name="calib_file" value="$(find box_model)/urdf/box/calibrations/calibration.yaml" />
+<xacro:property name="calib_file" value="$(find box_calibration)/calibration/tf/calibration_latest.yaml" />
 <!-- load the YAML calibration file into a property -->
 <xacro:property name="calib" value="${xacro.load_yaml(calib_file)}"/>
