Commit message: Refactor CPT7 and Basilisk definitions into calibration_latest.yaml file

File: box_model/box_model/urdf/box/box.urdf.xacro (robot description, xacro)
@@ -51,5 +51,10 @@
   <!-- CPT7 Coordinate System -->
   <joint name="base_to_cpt7_imu_frame" type="fixed">
-    <origin xyz="-0.294 -0.058 0.164" rpy="3.142 0.0 0.0" />
+    <origin xyz=" ${calib['box_base_to_cpt7_imu_frame']['x']}
+                  ${calib['box_base_to_cpt7_imu_frame']['y']}
+                  ${calib['box_base_to_cpt7_imu_frame']['z']}"
+            rpy=" ${calib['box_base_to_cpt7_imu_frame']['roll']}
+                  ${calib['box_base_to_cpt7_imu_frame']['pitch']}
+                  ${calib['box_base_to_cpt7_imu_frame']['yaw']}" />
     <parent link="box_base" />
     <child link="cpt7_imu" />
@@ -78,5 +83,10 @@
   <!-- Basilisk IMU Frame -->
   <joint name="base_to_basilisk_imu_frame" type="fixed">
-    <origin xyz="-0.293 0.034 0.155" rpy="1.571 0.0 0.0" />
+    <origin xyz=" ${calib['box_base_to_basilisk_imu_frame']['x']}
+                  ${calib['box_base_to_basilisk_imu_frame']['y']}
+                  ${calib['box_base_to_basilisk_imu_frame']['z']}"
+            rpy=" ${calib['box_base_to_basilisk_imu_frame']['roll']}
+                  ${calib['box_base_to_basilisk_imu_frame']['pitch']}
+                  ${calib['box_base_to_basilisk_imu_frame']['yaw']}" />
     <parent link="box_base" />
     <child link="State" />

Commit message: Add script to load assembly html and old stim320 cad, and generate new cad in cpt7

File: box_model/box_model/urdf/box/box.urdf.xacro (robot description, xacro)
@@ -2,5 +2,5 @@
 <robot name="box" xmlns:xacro="http://www.ros.org/wiki/xacro">
 <!-- YAML file containing the default values from CAD -->
-<xacro:property name="calib_file" value="$(find box_calibration)/calibration/tf/calibration_latest.yaml" />
+<xacro:property name="calib_file" value="$(find box_calibration)/calibration/tf/calibration_latest_in_cpt7.yaml" />
 <!-- load the YAML calibration file into a property -->
 <xacro:property name="calib" value="${xacro.load_yaml(calib_file)}"/>
@@ -13,13 +13,13 @@
   <!-- Box base -->
   <link name="box_base"/>
-  <joint name="prism_to_box_base" type="fixed">
-    <origin xyz=" ${calib['prism_to_box_base']['x']}
-                  ${calib['prism_to_box_base']['y']}
-                  ${calib['prism_to_box_base']['z']}"
-            rpy=" ${calib['prism_to_box_base']['roll']}
-                  ${calib['prism_to_box_base']['pitch']}
-                  ${calib['prism_to_box_base']['yaw']}" />
-    <parent link="prism" />
-    <child link="box_base" />
+  <joint name="box_base_to_prism" type="fixed">
+    <origin xyz=" ${calib['box_base_to_prism']['x']}
+                  ${calib['box_base_to_prism']['y']}
+                  ${calib['box_base_to_prism']['z']}"
+            rpy=" ${calib['box_base_to_prism']['roll']}
+                  ${calib['box_base_to_prism']['pitch']}
+                  ${calib['box_base_to_prism']['yaw']}" />
+    <parent link="box_base" />
+    <child link="prism" />
   </joint>
   <!-- Model base -->

Commit message: Move CPT and ZED base link to pinned connections

File: box_model/box_model/urdf/box/box.urdf.xacro (robot description, xacro)
@@ -51,10 +51,10 @@
   <!-- CPT7 Coordinate System -->
   <joint name="base_to_cpt7_imu_frame" type="fixed">
-    <origin xyz=" ${calib['box_base_to_cpt7_imu_frame']['x']}
-                  ${calib['box_base_to_cpt7_imu_frame']['y']}
-                  ${calib['box_base_to_cpt7_imu_frame']['z']}"
-            rpy=" ${calib['box_base_to_cpt7_imu_frame']['roll']}
-                  ${calib['box_base_to_cpt7_imu_frame']['pitch']}
-                  ${calib['box_base_to_cpt7_imu_frame']['yaw']}" />
+    <origin xyz=" ${pinned_constraints['box_base_to_cpt7_imu_frame']['x']}
+                  ${pinned_constraints['box_base_to_cpt7_imu_frame']['y']}
+                  ${pinned_constraints['box_base_to_cpt7_imu_frame']['z']}"
+            rpy=" ${pinned_constraints['box_base_to_cpt7_imu_frame']['roll']}
+                  ${pinned_constraints['box_base_to_cpt7_imu_frame']['pitch']}
+                  ${pinned_constraints['box_base_to_cpt7_imu_frame']['yaw']}" />
     <parent link="box_base" />
     <child link="cpt7_imu" />

Commit message: Use calibration_latest.yaml

File: box_model/box_model/urdf/box/box.urdf.xacro (robot description, xacro)
@@ -2,5 +2,5 @@
 <robot name="box" xmlns:xacro="http://www.ros.org/wiki/xacro">
 <!-- YAML file containing the default values from CAD -->
-<xacro:property name="calib_file" value="$(find box_calibration)/calibration/tf/calibration_latest_in_cpt7.yaml" />
+<xacro:property name="calib_file" value="$(find box_calibration)/calibration/tf/calibration_latest.yaml" />
 <!-- load the YAML calibration file into a property -->
 <xacro:property name="calib" value="${xacro.load_yaml(calib_file)}"/>

Commit message: Fix box_model to STIM_320 frame. Add new RViz config

File: box_model/box_model/urdf/box/box.urdf.xacro (robot description, xacro)
@@ -32,6 +32,6 @@
   </link>
   <joint name="box_base_to_box_base_model" type="fixed">
-    <origin xyz="0.0 0.0 0.0" rpy="0.0 0.0 0.0" />
-    <parent link="box_base" />
+    <origin xyz="-0.02 0.0 0.0" rpy="0.0 0.0 0.0" />
+    <parent link="imu_stim320" />
     <child link="box_base_model" />
   </joint>

Commit message: Update antenna names to be consistent in style

File: box_model/box_model/urdf/box/box.urdf.xacro (robot description, xacro)
@@ -66,17 +66,17 @@
     <child link="base" />
   </joint>
-  <link name="cpt7_front_antenna"/>
+  <link name="cpt7_antenna_front"/>
   <!-- CPT7 Coordinate System -->
-  <joint name="cpt7_to_front_antenna" type="fixed">
+  <joint name="cpt7_to_antenna_front" type="fixed">
     <origin xyz="0.13924890003 -0.0361 -0.1712000" rpy="0.0 0.0 0.0" />
     <parent link="cpt7_imu" />
-    <child link="cpt7_front_antenna" />
+    <child link="cpt7_antenna_front" />
   </joint>
-  <link name="cpt7_back_antenna"/>
+  <link name="cpt7_antenna_back"/>
   <!-- CPT7 Coordinate System -->
-  <joint name="cpt7_to_back_antenna" type="fixed">
+  <joint name="cpt7_to_antenna_back" type="fixed">
     <origin xyz="-0.4404038 -0.0361 -0.0267714" rpy="0.0 0.0 0.0" />
     <parent link="cpt7_imu" />
-    <child link="cpt7_back_antenna" />
+    <child link="cpt7_antenna_back" />
   </joint>
   <link name="State"/>

Commit message: Update ap20 imu frame id in urdf

File: box_model/box_model/urdf/box/box.urdf.xacro (robot description, xacro)
@@ -80,5 +80,5 @@
     <child link="cpt7_antenna_back" />
   </joint>
-  <link name="State"/>
+  <link name="ap20_imu"/>
   <!-- Basilisk IMU Frame -->
   <joint name="base_to_basilisk_imu_frame" type="fixed">
@@ -90,5 +90,5 @@
                   ${calib['box_base_to_basilisk_imu_frame']['yaw']}" />
     <parent link="box_base" />
-    <child link="State" />
+    <child link="ap20_imu" />
   </joint>
   <xacro:include filename="$(find box_model)/urdf/cameras/cameras.urdf.xacro" />

Commit message: Fix box_base and stim320

File: box_model/box_model/urdf/box/box.urdf.xacro (robot description, xacro)
@@ -33,5 +33,5 @@
   <joint name="box_base_to_box_base_model" type="fixed">
     <origin xyz="-0.02 0.0 0.0" rpy="0.0 0.0 0.0" />
-    <parent link="imu_stim320" />
+    <parent link="box_base" />
     <child link="box_base_model" />
   </joint>

Commit message: updated gps antenna location with span values

File: box_model/box_model/urdf/box/box.urdf.xacro (robot description, xacro)
@@ -69,5 +69,5 @@
   <!-- CPT7 Coordinate System -->
   <joint name="cpt7_to_antenna_front" type="fixed">
-    <origin xyz="0.13924890003 -0.0361 -0.1712000" rpy="0.0 0.0 0.0" />
+    <origin xyz="0.13924890003 -0.0361 -0.193298" rpy="0.0 0.0 0.0" />
     <parent link="cpt7_imu" />
     <child link="cpt7_antenna_front" />
@@ -76,5 +76,5 @@
   <!-- CPT7 Coordinate System -->
   <joint name="cpt7_to_antenna_back" type="fixed">
-    <origin xyz="-0.4404038 -0.0361 -0.0267714" rpy="0.0 0.0 0.0" />
+    <origin xyz="-0.4404038 -0.0361 -0.048868" rpy="0.0 0.0 0.0" />
     <parent link="cpt7_imu" />
     <child link="cpt7_antenna_back" />

Commit message: Set Anymal base as TF root

File: box_model/box_model/urdf/box/box.urdf.xacro (robot description, xacro)
@@ -57,12 +57,12 @@
                   ${pinned_constraints['box_base_to_cpt7_imu_frame']['pitch']}
                   ${pinned_constraints['box_base_to_cpt7_imu_frame']['yaw']}" />
-    <parent link="box_base" />
-    <child link="cpt7_imu" />
+    <parent link="cpt7_imu" />
+    <child link="box_base" />
   </joint>
   <link name="base"/>
   <joint name="cpt7_to_robot_base" type="fixed">
-    <origin xyz="-0.0764038 -0.0361 0.2802790" rpy="3.1415126 0.0 0.0" />
-    <parent link="cpt7_imu" />
-    <child link="base" />
+    <origin xyz="0.0764038 -0.0361 0.2802790" rpy="3.1415126 0.0 0.0" />
+    <parent link="base" />
+    <child link="cpt7_imu" />
   </joint>
   <link name="cpt7_antenna_front"/>

Commit message: fixed chrony and pi sync and box urdf

File: box_model/box_model/urdf/box/box.urdf.xacro (robot description, xacro)
@@ -57,6 +57,6 @@
                   ${pinned_constraints['box_base_to_cpt7_imu_frame']['pitch']}
                   ${pinned_constraints['box_base_to_cpt7_imu_frame']['yaw']}" />
-    <parent link="cpt7_imu" />
-    <child link="box_base" />
+    <parent link="box_base" />
+    <child link="cpt7_imu" />
   </joint>
   <link name="base"/>
@@ -64,5 +64,5 @@
     <origin xyz="0.0764038 -0.0361 0.2802790" rpy="3.1415126 0.0 0.0" />
     <parent link="base" />
-    <child link="cpt7_imu" />
+    <child link="box_base" />
   </joint>
   <link name="cpt7_antenna_front"/>

Commit message: Remove large image files

File: box_model/box_model/urdf/box/box.urdf.xacro (robot description, xacro)
@@ -2,5 +2,5 @@
 <robot name="box" xmlns:xacro="http://www.ros.org/wiki/xacro">
 <!-- YAML file containing the default values from CAD -->
-<xacro:property name="calib_file" value="$(find box_calibration)/calibration/tf/calibration_latest.yaml" />
+<xacro:property name="calib_file" value="$(find box_calibration)/calibration/tf/calibration_cad.yaml" />
 <!-- load the YAML calibration file into a property -->
 <xacro:property name="calib" value="${xacro.load_yaml(calib_file)}"/>
@@ -32,5 +32,5 @@
   </link>
   <joint name="box_base_to_box_base_model" type="fixed">
-    <origin xyz="-0.02 0.0 0.0" rpy="0.0 0.0 0.0" />
+    <origin xyz="0.0 0.0 0.0" rpy="0.0 0.0 0.0" />
     <parent link="stim320_imu" />
     <child link="box_base_model" />

Commit message: Remove reliance on pinned_constraints.yaml

File: box_model/box_model/urdf/box/box.urdf.xacro (robot description, xacro)
@@ -5,8 +5,34 @@
 <!-- load the YAML calibration file into a property -->
 <xacro:property name="calib" value="${xacro.load_yaml(calib_file)}"/>
-<!-- YAML file containing the default values from CAD -->
-<xacro:property name="pinned_constraints_file" value="$(find box_calibration)/calibration/tf/pinned_constraints.yaml" />
-<!-- load the YAML calibration file into a property -->
-<xacro:property name="pinned_constraints" value="${xacro.load_yaml(pinned_constraints_file)}"/>
+  <link name="base"/>
+  <joint name="cpt7_to_robot_base" type="fixed">
+    <origin xyz="0.0764038 -0.0361 0.2802790" rpy="3.1415126 0.0 0.0" />
+    <parent link="base" />
+    <child link="box_base" />
+  </joint>
+  <link name="cpt7_antenna_front"/>
+  <!-- CPT7 Coordinate System -->
+  <joint name="cpt7_to_antenna_front" type="fixed">
+    <origin xyz="0.13924890003 -0.0361 -0.193298" rpy="0.0 0.0 0.0" />
+    <parent link="cpt7_imu" />
+    <child link="cpt7_antenna_front" />
+  </joint>
+  <link name="cpt7_antenna_back"/>
+  <!-- CPT7 Coordinate System -->
+  <joint name="cpt7_to_antenna_back" type="fixed">
+    <origin xyz="-0.4404038 -0.0361 -0.048868" rpy="0.0 0.0 0.0" />
+    <parent link="cpt7_imu" />
+    <child link="cpt7_antenna_back" />
+  </joint>
+  <joint name="stim320_imu_to_box_base_model" type="fixed">
+    <origin xyz="0.0 0.0 0.0" rpy="0.0 0.0 0.0" />
+    <parent link="stim320_imu" />
+    <child link="box_base_model" />
+  </joint>
+  <joint name="prism_to_prism_model" type="fixed">
+    <origin xyz="0.0 0.0 0.0" rpy="0.0 0.0 0.0" />
+    <parent link="prism" />
+    <child link="prism_model" />
+  </joint>
   <!-- Prism -->
   <link name="prism"/>
@@ -31,9 +57,4 @@
     </visual>
   </link>
-  <joint name="box_base_to_box_base_model" type="fixed">
-    <origin xyz="0.0 0.0 0.0" rpy="0.0 0.0 0.0" />
-    <parent link="stim320_imu" />
-    <child link="box_base_model" />
-  </joint>
   <link name="prism_model">
     <visual>
@@ -43,40 +64,15 @@
     </visual>
   </link>
-  <joint name="prism_to_prism_model" type="fixed">
-    <origin xyz="0.0 0.0 0.0" rpy="0.0 0.0 0.0" />
-    <parent link="prism" />
-    <child link="prism_model" />
-  </joint>
   <link name="cpt7_imu"/>
   <!-- CPT7 Coordinate System -->
-  <joint name="base_to_cpt7_imu_frame" type="fixed">
-    <origin xyz=" ${pinned_constraints['box_base_to_cpt7_imu_frame']['x']}
-                  ${pinned_constraints['box_base_to_cpt7_imu_frame']['y']}
-                  ${pinned_constraints['box_base_to_cpt7_imu_frame']['z']}"
-            rpy=" ${pinned_constraints['box_base_to_cpt7_imu_frame']['roll']}
-                  ${pinned_constraints['box_base_to_cpt7_imu_frame']['pitch']}
-                  ${pinned_constraints['box_base_to_cpt7_imu_frame']['yaw']}" />
+  <joint name="box_base_to_cpt7_imu_frame" type="fixed">
+    <origin xyz=" ${calib['box_base_to_cpt7_imu_frame']['x']}
+                  ${calib['box_base_to_cpt7_imu_frame']['y']}
+                  ${calib['box_base_to_cpt7_imu_frame']['z']}"
+            rpy=" ${calib['box_base_to_cpt7_imu_frame']['roll']}
+                  ${calib['box_base_to_cpt7_imu_frame']['pitch']}
+                  ${calib['box_base_to_cpt7_imu_frame']['yaw']}" />
     <parent link="box_base" />
     <child link="cpt7_imu" />
-  </joint>
-  <link name="base"/>
-  <joint name="cpt7_to_robot_base" type="fixed">
-    <origin xyz="0.0764038 -0.0361 0.2802790" rpy="3.1415126 0.0 0.0" />
-    <parent link="base" />
-    <child link="box_base" />
-  </joint>
-  <link name="cpt7_antenna_front"/>
-  <!-- CPT7 Coordinate System -->
-  <joint name="cpt7_to_antenna_front" type="fixed">
-    <origin xyz="0.13924890003 -0.0361 -0.193298" rpy="0.0 0.0 0.0" />
-    <parent link="cpt7_imu" />
-    <child link="cpt7_antenna_front" />
-  </joint>
-  <link name="cpt7_antenna_back"/>
-  <!-- CPT7 Coordinate System -->
-  <joint name="cpt7_to_antenna_back" type="fixed">
-    <origin xyz="-0.4404038 -0.0361 -0.048868" rpy="0.0 0.0 0.0" />
-    <parent link="cpt7_imu" />
-    <child link="cpt7_antenna_back" />
   </joint>
   <link name="ap20_imu"/>

File: box_model/box_model/urdf/cameras/cameras.urdf.xacro (robot description, xacro)
@@ -59,10 +59,10 @@
     <link name="cam3_sensor_frame"/>
     <joint name="alphasense_base_to_alphasense_front_left" type="fixed">
-        <origin xyz=" ${pinned_constraints['alphasense_base_to_alphasense_front_left']['x']}
-                  ${pinned_constraints['alphasense_base_to_alphasense_front_left']['y']}
-                  ${pinned_constraints['alphasense_base_to_alphasense_front_left']['z']}"
-                rpy=" ${pinned_constraints['alphasense_base_to_alphasense_front_left']['roll']}
-                  ${pinned_constraints['alphasense_base_to_alphasense_front_left']['pitch']}
-                  ${pinned_constraints['alphasense_base_to_alphasense_front_left']['yaw']}"/>
+        <origin xyz=" ${calib['alphasense_base_to_alphasense_front_left']['x']}
+                  ${calib['alphasense_base_to_alphasense_front_left']['y']}
+                  ${calib['alphasense_base_to_alphasense_front_left']['z']}"
+                rpy=" ${calib['alphasense_base_to_alphasense_front_left']['roll']}
+                  ${calib['alphasense_base_to_alphasense_front_left']['pitch']}
+                  ${calib['alphasense_base_to_alphasense_front_left']['yaw']}"/>
         <parent link="alphasense_base"/>
         <child link="cam3_sensor_frame"/>
@@ -120,10 +120,10 @@
     <link name="hdr_front"/>
     <joint name="hdr_base_to_hdr_front" type="fixed">
-        <origin xyz=" ${pinned_constraints['hdr_base_to_hdr_front']['x']}
-                  ${pinned_constraints['hdr_base_to_hdr_front']['y']}
-                  ${pinned_constraints['hdr_base_to_hdr_front']['z']}"
-                rpy=" ${pinned_constraints['hdr_base_to_hdr_front']['roll']}
-                  ${pinned_constraints['hdr_base_to_hdr_front']['pitch']}
-                  ${pinned_constraints['hdr_base_to_hdr_front']['yaw']}"/>
+        <origin xyz=" ${calib['hdr_base_to_hdr_front']['x']}
+                  ${calib['hdr_base_to_hdr_front']['y']}
+                  ${calib['hdr_base_to_hdr_front']['z']}"
+                rpy=" ${calib['hdr_base_to_hdr_front']['roll']}
+                  ${calib['hdr_base_to_hdr_front']['pitch']}
+                  ${calib['hdr_base_to_hdr_front']['yaw']}"/>
         <parent link="hdr_base"/>
         <child link="hdr_front"/>
@@ -157,10 +157,10 @@
     <link name="zed_base_link"/>
     <joint name="box_base_to_zed_base" type="fixed">
-        <origin xyz=" ${pinned_constraints['box_base_to_zed_base']['x']}
-                  ${pinned_constraints['box_base_to_zed_base']['y']}
-                  ${pinned_constraints['box_base_to_zed_base']['z']}"
-                rpy=" ${pinned_constraints['box_base_to_zed_base']['roll']}
-                  ${pinned_constraints['box_base_to_zed_base']['pitch']}
-                  ${pinned_constraints['box_base_to_zed_base']['yaw']}"/>
+        <origin xyz=" ${calib['box_base_to_zed_base']['x']}
+                  ${calib['box_base_to_zed_base']['y']}
+                  ${calib['box_base_to_zed_base']['z']}"
+                rpy=" ${calib['box_base_to_zed_base']['roll']}
+                  ${calib['box_base_to_zed_base']['pitch']}
+                  ${calib['box_base_to_zed_base']['yaw']}"/>
         <parent link="box_base"/>
         <child link="zed_base_link"/>
@@ -174,10 +174,10 @@
     <link name="zed2i_camera_center"/>
     <joint name="zed2i_base_to_camera_center" type="fixed">
-        <origin xyz=" ${pinned_constraints['zed2i_base_to_camera_center']['x']}
-                  ${pinned_constraints['zed2i_base_to_camera_center']['y']}
-                  ${pinned_constraints['zed2i_base_to_camera_center']['z']}"
-                rpy=" ${pinned_constraints['zed2i_base_to_camera_center']['roll']}
-                  ${pinned_constraints['zed2i_base_to_camera_center']['pitch']}
-                  ${pinned_constraints['zed2i_base_to_camera_center']['yaw']}"/>
+        <origin xyz=" ${calib['zed2i_base_to_camera_center']['x']}
+                  ${calib['zed2i_base_to_camera_center']['y']}
+                  ${calib['zed2i_base_to_camera_center']['z']}"
+                rpy=" ${calib['zed2i_base_to_camera_center']['roll']}
+                  ${calib['zed2i_base_to_camera_center']['pitch']}
+                  ${calib['zed2i_base_to_camera_center']['yaw']}"/>
         <parent link="zed2i_base_link"/>
         <child link="zed2i_camera_center"/>
@@ -185,10 +185,10 @@
     <link name="zed2i_left_camera_frame"/>
     <joint name="zed_camera_center_to_zed_left" type="fixed">
-        <origin xyz=" ${pinned_constraints['zed_camera_center_to_zed_left']['x']}
-                  ${pinned_constraints['zed_camera_center_to_zed_left']['y']}
-                  ${pinned_constraints['zed_camera_center_to_zed_left']['z']}"
-                rpy=" ${pinned_constraints['zed_camera_center_to_zed_left']['roll']}
-                  ${pinned_constraints['zed_camera_center_to_zed_left']['pitch']}
-                  ${pinned_constraints['zed_camera_center_to_zed_left']['yaw']}"/>
+        <origin xyz=" ${calib['zed_camera_center_to_zed_left']['x']}
+                  ${calib['zed_camera_center_to_zed_left']['y']}
+                  ${calib['zed_camera_center_to_zed_left']['z']}"
+                rpy=" ${calib['zed_camera_center_to_zed_left']['roll']}
+                  ${calib['zed_camera_center_to_zed_left']['pitch']}
+                  ${calib['zed_camera_center_to_zed_left']['yaw']}"/>
         <parent link="zed2i_camera_center"/>
         <child link="zed2i_left_camera_frame"/>
@@ -196,10 +196,10 @@
     <link name="zed2i_left_camera_optical_frame"/>
     <joint name="zed_left_to_optical" type="fixed">
-        <origin xyz=" ${pinned_constraints['zed2i_camera_to_zed2i_optical']['x']}
-                  ${pinned_constraints['zed2i_camera_to_zed2i_optical']['y']}
-                  ${pinned_constraints['zed2i_camera_to_zed2i_optical']['z']}"
-                rpy=" ${pinned_constraints['zed2i_camera_to_zed2i_optical']['roll']}
-                  ${pinned_constraints['zed2i_camera_to_zed2i_optical']['pitch']}
-                  ${pinned_constraints['zed2i_camera_to_zed2i_optical']['yaw']}"/>
+        <origin xyz=" ${calib['zed2i_camera_to_zed2i_optical']['x']}
+                  ${calib['zed2i_camera_to_zed2i_optical']['y']}
+                  ${calib['zed2i_camera_to_zed2i_optical']['z']}"
+                rpy=" ${calib['zed2i_camera_to_zed2i_optical']['roll']}
+                  ${calib['zed2i_camera_to_zed2i_optical']['pitch']}
+                  ${calib['zed2i_camera_to_zed2i_optical']['yaw']}"/>
         <parent link="zed2i_left_camera_frame"/>
         <child link="zed2i_left_camera_optical_frame"/>
@@ -229,10 +229,10 @@
     <link name="zed2i_right_camera_frame"/>
     <joint name="zed_camera_center_to_zed_right" type="fixed">
-        <origin xyz=" ${pinned_constraints['zed2i_optical_to_zed2i_camera']['x']}
-                  ${pinned_constraints['zed2i_optical_to_zed2i_camera']['y']}
-                  ${pinned_constraints['zed2i_optical_to_zed2i_camera']['z']}"
-                rpy=" ${pinned_constraints['zed2i_optical_to_zed2i_camera']['roll']}
-                  ${pinned_constraints['zed2i_optical_to_zed2i_camera']['pitch']}
-                  ${pinned_constraints['zed2i_optical_to_zed2i_camera']['yaw']}"/>
+        <origin xyz=" ${calib['zed2i_optical_to_zed2i_camera']['x']}
+                  ${calib['zed2i_optical_to_zed2i_camera']['y']}
+                  ${calib['zed2i_optical_to_zed2i_camera']['z']}"
+                rpy=" ${calib['zed2i_optical_to_zed2i_camera']['roll']}
+                  ${calib['zed2i_optical_to_zed2i_camera']['pitch']}
+                  ${calib['zed2i_optical_to_zed2i_camera']['yaw']}"/>
         <parent link="zed2i_right_camera_optical_frame"/>
         <child link="zed2i_right_camera_frame"/>
