Commit message: Renaming box_base_to_basilisk_imu_frame into box_base_to_ap20_imu_frame

File: box_model/box_model/urdf/box/box.urdf.xacro (robot description, xacro)
@@ -76,16 +76,4 @@
     <child link="cpt7_imu" />
   </joint>
-  <link name="ap20_imu"/>
-  <!-- Basilisk IMU Frame -->
-  <joint name="base_to_basilisk_imu_frame" type="fixed">
-    <origin xyz=" ${calib['box_base_to_basilisk_imu_frame']['x']}
-                  ${calib['box_base_to_basilisk_imu_frame']['y']}
-                  ${calib['box_base_to_basilisk_imu_frame']['z']}"
-            rpy=" ${calib['box_base_to_basilisk_imu_frame']['roll']}
-                  ${calib['box_base_to_basilisk_imu_frame']['pitch']}
-                  ${calib['box_base_to_basilisk_imu_frame']['yaw']}" />
-    <parent link="box_base" />
-    <child link="ap20_imu" />
-  </joint>
   <xacro:include filename="$(find box_model)/urdf/cameras/cameras.urdf.xacro" />
   <xacro:include filename="$(find box_model)/urdf/lidars/lidars.urdf.xacro" />

File: box_model/box_model/urdf/box/box_calibrated.urdf.xacro (robot description, xacro)
@@ -98,10 +98,10 @@
     <!--  &lt;!&ndash; Basilisk IMU Frame &ndash;&gt;-->
     <!--  <joint name="base_to_basilisk_imu_frame" type="fixed">-->
-    <!--    <origin xyz=" ${calib['box_base_to_basilisk_imu_frame']['x']}-->
-    <!--                  ${calib['box_base_to_basilisk_imu_frame']['y']}-->
-    <!--                  ${calib['box_base_to_basilisk_imu_frame']['z']}"-->
-    <!--            rpy=" ${calib['box_base_to_basilisk_imu_frame']['roll']}-->
-    <!--                  ${calib['box_base_to_basilisk_imu_frame']['pitch']}-->
-    <!--                  ${calib['box_base_to_basilisk_imu_frame']['yaw']}" />-->
+    <!--    <origin xyz=" ${calib['box_base_to_ap20_imu_frame']['x']}-->
+    <!--                  ${calib['box_base_to_ap20_imu_frame']['y']}-->
+    <!--                  ${calib['box_base_to_ap20_imu_frame']['z']}"-->
+    <!--            rpy=" ${calib['box_base_to_ap20_imu_frame']['roll']}-->
+    <!--                  ${calib['box_base_to_ap20_imu_frame']['pitch']}-->
+    <!--                  ${calib['box_base_to_ap20_imu_frame']['yaw']}" />-->
     <!--    <parent link="box_base" />-->
     <!--    <child link="ap20_imu" />-->

File: box_model/box_model/urdf/imus/imus.urdf.xacro (robot description, xacro)
@@ -1,4 +1,16 @@
 <?xml version="1.0" ?>
 <robot name="imus" xmlns:xacro="http://www.ros.org/wiki/xacro">
+  <link name="ap20_imu"/>
+  <!-- Basilisk IMU Frame -->
+  <joint name="base_to_basilisk_imu_frame" type="fixed">
+    <origin xyz=" ${calib['box_base_to_ap20_imu_frame']['x']}
+                  ${calib['box_base_to_ap20_imu_frame']['y']}
+                  ${calib['box_base_to_ap20_imu_frame']['z']}"
+            rpy=" ${calib['box_base_to_ap20_imu_frame']['roll']}
+                  ${calib['box_base_to_ap20_imu_frame']['pitch']}
+                  ${calib['box_base_to_ap20_imu_frame']['yaw']}" />
+    <parent link="box_base" />
+    <child link="ap20_imu" />
+  </joint>
   <!-- IMU STIM320 -->
   <link name="stim320_imu" />

Commit message: Minor rename

File: box_model/box_model/urdf/box/box.urdf.xacro (robot description, xacro)
@@ -2,5 +2,5 @@
 <robot name="box" xmlns:xacro="http://www.ros.org/wiki/xacro">
 <!-- YAML file containing the default values from CAD -->
-<xacro:property name="calib_file" value="$(find box_calibration)/calibration/tf/calibration_cad.yaml" />
+<xacro:property name="calib_file" value="$(find box_calibration)/calibration/tf/calibration_latest.yaml" />
 <!-- load the YAML calibration file into a property -->
 <xacro:property name="calib" value="${xacro.load_yaml(calib_file)}"/>
@@ -11,25 +11,11 @@
     <child link="box_base" />
   </joint>
-  <link name="cpt7_antenna_front"/>
-  <!-- CPT7 Coordinate System -->
-  <joint name="cpt7_to_antenna_front" type="fixed">
-    <origin xyz="0.13924890003 -0.0361 -0.193298" rpy="0.0 0.0 0.0" />
-    <parent link="cpt7_imu" />
-    <child link="cpt7_antenna_front" />
-  </joint>
-  <link name="cpt7_antenna_back"/>
-  <!-- CPT7 Coordinate System -->
-  <joint name="cpt7_to_antenna_back" type="fixed">
-    <origin xyz="-0.4404038 -0.0361 -0.048868" rpy="0.0 0.0 0.0" />
-    <parent link="cpt7_imu" />
-    <child link="cpt7_antenna_back" />
-  </joint>
-  <joint name="stim320_imu_to_box_base_model" type="fixed">
-    <origin xyz="0.0 0.0 0.0" rpy="0.0 0.0 0.0" />
-    <parent link="stim320_imu" />
-    <child link="box_base_model" />
-  </joint>
   <joint name="prism_to_prism_model" type="fixed">
-    <origin xyz="0.0 0.0 0.0" rpy="0.0 0.0 0.0" />
+    <origin xyz=" ${calib['prism_to_prism_model']['x']}
+                  ${calib['prism_to_prism_model']['y']}
+                  ${calib['prism_to_prism_model']['z']}"
+            rpy=" ${calib['prism_to_prism_model']['roll']}
+                  ${calib['prism_to_prism_model']['pitch']}
+                  ${calib['prism_to_prism_model']['yaw']}" />
     <parent link="prism" />
     <child link="prism_model" />
@@ -64,16 +50,4 @@
     </visual>
   </link>
-  <link name="cpt7_imu"/>
-  <!-- CPT7 Coordinate System -->
-  <joint name="box_base_to_cpt7_imu_frame" type="fixed">
-    <origin xyz=" ${calib['box_base_to_cpt7_imu_frame']['x']}
-                  ${calib['box_base_to_cpt7_imu_frame']['y']}
-                  ${calib['box_base_to_cpt7_imu_frame']['z']}"
-            rpy=" ${calib['box_base_to_cpt7_imu_frame']['roll']}
-                  ${calib['box_base_to_cpt7_imu_frame']['pitch']}
-                  ${calib['box_base_to_cpt7_imu_frame']['yaw']}" />
-    <parent link="box_base" />
-    <child link="cpt7_imu" />
-  </joint>
   <xacro:include filename="$(find box_model)/urdf/cameras/cameras.urdf.xacro" />
   <xacro:include filename="$(find box_model)/urdf/lidars/lidars.urdf.xacro" />

File: box_model/box_model/urdf/cameras/cameras.urdf.xacro (robot description, xacro)
@@ -16,5 +16,10 @@
     <link name="alphasense_front_center"/>
     <joint name="alphasense_front_center_identity" type="fixed">
-        <origin xyz="0 0 0" rpy="0 0 0"/>
+        <origin xyz=" ${calib['alphasense_cam1_helper_joint']['x']}
+                  ${calib['alphasense_cam2_helper_joint']['y']}
+                  ${calib['alphasense_cam1_helper_joint']['z']}"
+                rpy=" ${calib['alphasense_cam1_helper_joint']['roll']}
+                  ${calib['alphasense_cam1_helper_joint']['pitch']}
+                  ${calib['alphasense_cam1_helper_joint']['yaw']}"/>
         <parent link="cam1_sensor_frame"/>
         <child link="alphasense_front_center"/>
@@ -34,5 +39,10 @@
     <link name="alphasense_front_right"/>
     <joint name="alphasense_front_right_identity" type="fixed">
-        <origin xyz="0 0 0" rpy="0 0 0"/>
+        <origin xyz=" ${calib['alphasense_cam2_helper_joint']['x']}
+                  ${calib['alphasense_cam2_helper_joint']['y']}
+                  ${calib['alphasense_cam2_helper_joint']['z']}"
+                rpy=" ${calib['alphasense_cam2_helper_joint']['roll']}
+                  ${calib['alphasense_cam2_helper_joint']['pitch']}
+                  ${calib['alphasense_cam2_helper_joint']['yaw']}"/>
         <parent link="cam2_sensor_frame"/>
         <child link="alphasense_front_right"/>
@@ -52,5 +62,10 @@
     <link name="alphasense_front_left"/>
     <joint name="alphasense_front_left_identity" type="fixed">
-        <origin xyz="0 0 0" rpy="0 0 0"/>
+        <origin xyz=" ${calib['alphasense_cam3_helper_joint']['x']}
+                  ${calib['alphasense_cam3_helper_joint']['y']}
+                  ${calib['alphasense_cam3_helper_joint']['z']}"
+                rpy=" ${calib['alphasense_cam3_helper_joint']['roll']}
+                  ${calib['alphasense_cam3_helper_joint']['pitch']}
+                  ${calib['alphasense_cam3_helper_joint']['yaw']}"/>
         <parent link="cam3_sensor_frame"/>
         <child link="alphasense_front_left"/>
@@ -70,5 +85,10 @@
     <link name="alphasense_left"/>
     <joint name="alphasense_left_identity" type="fixed">
-        <origin xyz="0 0 0" rpy="0 0 0"/>
+        <origin xyz=" ${calib['alphasense_cam4_helper_joint']['x']}
+                  ${calib['alphasense_cam4_helper_joint']['y']}
+                  ${calib['alphasense_cam4_helper_joint']['z']}"
+                rpy=" ${calib['alphasense_cam4_helper_joint']['roll']}
+                  ${calib['alphasense_cam4_helper_joint']['pitch']}
+                  ${calib['alphasense_cam4_helper_joint']['yaw']}"/>
         <parent link="cam4_sensor_frame"/>
         <child link="alphasense_left"/>
@@ -88,5 +108,10 @@
     <link name="alphasense_right"/>
     <joint name="alphasense_right_identity" type="fixed">
-        <origin xyz="0 0 0" rpy="0 0 0"/>
+        <origin xyz=" ${calib['alphasense_cam5_helper_joint']['x']}
+                  ${calib['alphasense_cam5_helper_joint']['y']}
+                  ${calib['alphasense_cam5_helper_joint']['z']}"
+                rpy=" ${calib['alphasense_cam5_helper_joint']['roll']}
+                  ${calib['alphasense_cam5_helper_joint']['pitch']}
+                  ${calib['alphasense_cam5_helper_joint']['yaw']}"/>
         <parent link="cam5_sensor_frame"/>
         <child link="alphasense_right"/>
@@ -167,6 +192,11 @@
     </joint>
     <link name="zed2i_base_link"/>
-    <joint name="zed2i_redundant_indentity" type="fixed">
-        <origin xyz="0 0 0" rpy="0 0 0"/>
+    <joint name="zed2i_base_helper_joint" type="fixed">
+        <origin xyz=" ${calib['zed2i_base_helper_joint']['x']}
+                  ${calib['zed2i_base_helper_joint']['y']}
+                  ${calib['zed2i_base_helper_joint']['z']}"
+                rpy=" ${calib['zed2i_base_helper_joint']['roll']}
+                  ${calib['zed2i_base_helper_joint']['pitch']}
+                  ${calib['zed2i_base_helper_joint']['yaw']}"/>
         <parent link="zed_base_link"/>
         <child link="zed2i_base_link"/>
@@ -196,21 +226,21 @@
     <link name="zed2i_left_camera_optical_frame"/>
     <joint name="zed_left_to_optical" type="fixed">
-        <origin xyz=" ${calib['zed2i_camera_to_zed2i_optical']['x']}
-                  ${calib['zed2i_camera_to_zed2i_optical']['y']}
-                  ${calib['zed2i_camera_to_zed2i_optical']['z']}"
-                rpy=" ${calib['zed2i_camera_to_zed2i_optical']['roll']}
-                  ${calib['zed2i_camera_to_zed2i_optical']['pitch']}
-                  ${calib['zed2i_camera_to_zed2i_optical']['yaw']}"/>
+        <origin xyz=" ${calib['zed_left_to_left_optical']['x']}
+                  ${calib['zed_left_to_left_optical']['y']}
+                  ${calib['zed_left_to_left_optical']['z']}"
+                rpy=" ${calib['zed_left_to_left_optical']['roll']}
+                  ${calib['zed_left_to_left_optical']['pitch']}
+                  ${calib['zed_left_to_left_optical']['yaw']}"/>
         <parent link="zed2i_left_camera_frame"/>
         <child link="zed2i_left_camera_optical_frame"/>
     </joint>
     <link name="zed2i_imu_link"/>
-    <joint name="zed_base_to_zed_imu_link" type="fixed">
-        <origin xyz=" ${calib['zed_left_camera_frame_to_zed_imu_link']['x']}
-                  ${calib['zed_left_camera_frame_to_zed_imu_link']['y']}
-                  ${calib['zed_left_camera_frame_to_zed_imu_link']['z']}"
-                rpy=" ${calib['zed_left_camera_frame_to_zed_imu_link']['roll']}
-                  ${calib['zed_left_camera_frame_to_zed_imu_link']['pitch']}
-                  ${calib['zed_left_camera_frame_to_zed_imu_link']['yaw']}"/>
+    <joint name="zed_left_camera_frame_to_zed_imu_joint" type="fixed">
+        <origin xyz=" ${calib['zed_left_camera_frame_to_zed_imu']['x']}
+                  ${calib['zed_left_camera_frame_to_zed_imu']['y']}
+                  ${calib['zed_left_camera_frame_to_zed_imu']['z']}"
+                rpy=" ${calib['zed_left_camera_frame_to_zed_imu']['roll']}
+                  ${calib['zed_left_camera_frame_to_zed_imu']['pitch']}
+                  ${calib['zed_left_camera_frame_to_zed_imu']['yaw']}"/>
         <parent link="zed2i_left_camera_frame"/>
         <child link="zed2i_imu_link"/>
@@ -229,10 +259,10 @@
     <link name="zed2i_right_camera_frame"/>
     <joint name="zed_camera_center_to_zed_right" type="fixed">
-        <origin xyz=" ${calib['zed2i_optical_to_zed2i_camera']['x']}
-                  ${calib['zed2i_optical_to_zed2i_camera']['y']}
-                  ${calib['zed2i_optical_to_zed2i_camera']['z']}"
-                rpy=" ${calib['zed2i_optical_to_zed2i_camera']['roll']}
-                  ${calib['zed2i_optical_to_zed2i_camera']['pitch']}
-                  ${calib['zed2i_optical_to_zed2i_camera']['yaw']}"/>
+        <origin xyz=" ${calib['zed_right_to_right_optical']['x']}
+                  ${calib['zed_right_to_right_optical']['y']}
+                  ${calib['zed_right_to_right_optical']['z']}"
+                rpy=" ${calib['zed_right_to_right_optical']['roll']}
+                  ${calib['zed_right_to_right_optical']['pitch']}
+                  ${calib['zed_right_to_right_optical']['yaw']}"/>
         <parent link="zed2i_right_camera_optical_frame"/>
         <child link="zed2i_right_camera_frame"/>

File: box_model/box_model/urdf/imus/imus.urdf.xacro (robot description, xacro)
@@ -1,7 +1,43 @@
 <?xml version="1.0" ?>
 <robot name="imus" xmlns:xacro="http://www.ros.org/wiki/xacro">
+  <link name="cpt7_imu"/>
+  <!-- CPT7 Coordinate System -->
+  <joint name="box_base_to_cpt7_imu_frame" type="fixed">
+    <origin xyz=" ${calib['box_base_to_cpt7_imu_frame']['x']}
+                  ${calib['box_base_to_cpt7_imu_frame']['y']}
+                  ${calib['box_base_to_cpt7_imu_frame']['z']}"
+            rpy=" ${calib['box_base_to_cpt7_imu_frame']['roll']}
+                  ${calib['box_base_to_cpt7_imu_frame']['pitch']}
+                  ${calib['box_base_to_cpt7_imu_frame']['yaw']}" />
+    <parent link="box_base" />
+    <child link="cpt7_imu" />
+  </joint>
+  <link name="cpt7_antenna_front"/>
+  <!-- CPT7 Coordinate System -->
+  <joint name="cpt7_to_antenna_front" type="fixed">
+    <origin xyz=" ${calib['cpt7_imu_frame_to_cpt7_antenna_front']['x']}
+                  ${calib['cpt7_imu_frame_to_cpt7_antenna_front']['y']}
+                  ${calib['cpt7_imu_frame_to_cpt7_antenna_front']['z']}"
+            rpy=" ${calib['cpt7_imu_frame_to_cpt7_antenna_front']['roll']}
+                  ${calib['cpt7_imu_frame_to_cpt7_antenna_front']['pitch']}
+                  ${calib['cpt7_imu_frame_to_cpt7_antenna_front']['yaw']}" />
+    <parent link="cpt7_imu" />
+    <child link="cpt7_antenna_front" />
+  </joint>
+  <link name="cpt7_antenna_back"/>
+  <!-- CPT7 Coordinate System -->
+  <joint name="cpt7_to_antenna_back" type="fixed">
+    <origin xyz=" ${calib['cpt7_imu_frame_to_cpt7_antenna_back']['x']}
+                  ${calib['cpt7_imu_frame_to_cpt7_antenna_back']['y']}
+                  ${calib['cpt7_imu_frame_to_cpt7_antenna_back']['z']}"
+            rpy=" ${calib['cpt7_imu_frame_to_cpt7_antenna_back']['roll']}
+                  ${calib['cpt7_imu_frame_to_cpt7_antenna_back']['pitch']}
+                  ${calib['cpt7_imu_frame_to_cpt7_antenna_back']['yaw']}" />
+    <parent link="cpt7_imu" />
+    <child link="cpt7_antenna_back" />
+  </joint>
   <link name="ap20_imu"/>
   <!-- Basilisk IMU Frame -->
-  <joint name="base_to_basilisk_imu_frame" type="fixed">
+  <joint name="box_base_to_ap20_imu_frame" type="fixed">
     <origin xyz=" ${calib['box_base_to_ap20_imu_frame']['x']}
                   ${calib['box_base_to_ap20_imu_frame']['y']}
@@ -24,4 +60,14 @@
     <parent link="box_base" />
     <child link="stim320_imu" />
+  </joint>
+  <joint name="stim320_imu_to_box_base_model" type="fixed">
+    <origin xyz=" ${calib['stim320_imu_to_box_base_model']['x']}
+                  ${calib['stim320_imu_to_box_base_model']['y']}
+                  ${calib['stim320_imu_to_box_base_model']['z']}"
+            rpy=" ${calib['stim320_imu_to_box_base_model']['roll']}
+                  ${calib['stim320_imu_to_box_base_model']['pitch']}
+                  ${calib['stim320_imu_to_box_base_model']['yaw']}" />
+    <parent link="stim320_imu" />
+    <child link="box_base_model" />
   </joint>
   <!-- IMU ADIS16475 -->

File: box_model/box_model/urdf/lidars/lidars.urdf.xacro (robot description, xacro)
@@ -3,11 +3,11 @@
   <!-- hesai_lidar -->
   <link name="hesai_lidar" />
-  <joint name="box_base_to_hesai" type="fixed">
-    <origin xyz=" ${calib['box_base_to_hesai']['x']}
-                  ${calib['box_base_to_hesai']['y']}
-                  ${calib['box_base_to_hesai']['z']}"
-            rpy=" ${calib['box_base_to_hesai']['roll']}
-                  ${calib['box_base_to_hesai']['pitch']}
-                  ${calib['box_base_to_hesai']['yaw']}" />
+  <joint name="box_base_to_hesai_lidar" type="fixed">
+    <origin xyz=" ${calib['box_base_to_hesai_lidar']['x']}
+                  ${calib['box_base_to_hesai_lidar']['y']}
+                  ${calib['box_base_to_hesai_lidar']['z']}"
+            rpy=" ${calib['box_base_to_hesai_lidar']['roll']}
+                  ${calib['box_base_to_hesai_lidar']['pitch']}
+                  ${calib['box_base_to_hesai_lidar']['yaw']}" />
     <parent link="box_base" />
     <child link="hesai_lidar" />
@@ -21,5 +21,10 @@
   </link>
   <joint name="hesai_lidar_to_hesai_model" type="fixed">
-    <origin xyz="0.0 0.0 0.0" rpy="0.0 0.0 0.0" />
+    <origin xyz=" ${calib['hesai_lidar_to_hesai_model']['x']}
+                  ${calib['hesai_lidar_to_hesai_model']['y']}
+                  ${calib['hesai_lidar_to_hesai_model']['z']}"
+            rpy=" ${calib['hesai_lidar_to_hesai_model']['roll']}
+                  ${calib['hesai_lidar_to_hesai_model']['pitch']}
+                  ${calib['hesai_lidar_to_hesai_model']['yaw']}" />
     <parent link="hesai_lidar" />
     <child link="hesai_model" />
@@ -27,11 +32,11 @@
   <!-- Livox -->
   <link name="livox_lidar" />
-  <joint name="box_base_to_livox" type="fixed">
-    <origin xyz=" ${calib['box_base_to_livox']['x']}
-                  ${calib['box_base_to_livox']['y']}
-                  ${calib['box_base_to_livox']['z']}"
-            rpy=" ${calib['box_base_to_livox']['roll']}
-                  ${calib['box_base_to_livox']['pitch']}
-                  ${calib['box_base_to_livox']['yaw']}" />
+  <joint name="box_base_to_livox_lidar" type="fixed">
+    <origin xyz=" ${calib['box_base_to_livox_lidar']['x']}
+                  ${calib['box_base_to_livox_lidar']['y']}
+                  ${calib['box_base_to_livox_lidar']['z']}"
+            rpy=" ${calib['box_base_to_livox_lidar']['roll']}
+                  ${calib['box_base_to_livox_lidar']['pitch']}
+                  ${calib['box_base_to_livox_lidar']['yaw']}" />
     <parent link="box_base" />
     <child link="livox_lidar" />
@@ -44,6 +49,11 @@
     </visual>
   </link>
-  <joint name="livox_to_livox_model" type="fixed">
-    <origin xyz="0.0 0.0 0.0" rpy="0.0 0.0 0.0" />
+  <joint name="livox_lidar_to_livox_model" type="fixed">
+    <origin xyz=" ${calib['livox_lidar_to_livox_model']['x']}
+                  ${calib['livox_lidar_to_livox_model']['y']}
+                  ${calib['livox_lidar_to_livox_model']['z']}"
+            rpy=" ${calib['livox_lidar_to_livox_model']['roll']}
+                  ${calib['livox_lidar_to_livox_model']['pitch']}
+                  ${calib['livox_lidar_to_livox_model']['yaw']}" />
     <parent link="livox_lidar" />
     <child link="livox_model" />
@@ -51,6 +61,11 @@
   <link name="livox_imu"/>
   <!-- From page 15 https://terra-1-g.djicdn.com/851d20f7b9f64838a34cd02351370894/Livox/Livox_Mid-360_User_Manual_EN.pdf -->
-  <joint name="livox_to_livox_imu_frame" type="fixed">
-    <origin xyz="0.011 0.02329 -0.04412" rpy="0.0 0.0 0.0" />
+  <joint name="livox_lidar_to_livox_imu" type="fixed">
+    <origin xyz=" ${calib['livox_lidar_to_livox_imu']['x']}
+                  ${calib['livox_lidar_to_livox_imu']['y']}
+                  ${calib['livox_lidar_to_livox_imu']['z']}"
+            rpy=" ${calib['livox_lidar_to_livox_imu']['roll']}
+                  ${calib['livox_lidar_to_livox_imu']['pitch']}
+                  ${calib['livox_lidar_to_livox_imu']['yaw']}" />
     <parent link="livox_lidar" />
     <child link="livox_imu" />
