Commit message: updated urdf without uploading large stl files

File: box_model/box_model/urdf/box/box.urdf.xacro (robot description, xacro)
@@ -25,5 +25,5 @@
   <!-- Box base -->
   <link name="box_base"/>
-  <joint name="box_base_to_prism" type="fixed">
+  <!-- <joint name="box_base_to_prism" type="fixed">
     <origin xyz=" ${calib['box_base_to_prism']['x']}
                   ${calib['box_base_to_prism']['y']}
@@ -34,4 +34,19 @@
     <parent link="box_base" />
     <child link="prism" />
+  </joint> -->
+  <joint name="box_base_to_prism" type="fixed">
+        <origin xyz="0.0 0.0 0.0" rpy="0.0 0.0 0.0"/>
+        <parent link="box_base"/>
+        <child link="prism"/>
+  </joint>
+  <joint name="box_base_to_box_base_model" type="fixed">
+        <origin xyz="0.0 0.0 0.0" rpy="0.0 0.0 0.0"/>
+        <parent link="box_base"/>
+        <child link="box_base_model"/>
+  </joint>
+  <joint name="base_to_cpt7_antenna_back_model" type="fixed">
+        <origin xyz="0.0 0.0 0.0" rpy="0.0 0.0 0.0"/>
+        <parent link="base"/>
+        <child link="cpt7_antenna_back_model"/>
   </joint>
   <!-- Model base -->
@@ -39,5 +54,12 @@
     <visual>
       <geometry>
-        <mesh filename="package://box_model/urdf/box/mesh/box_assembly_incl_livox_mount.dae" />
+        <mesh filename="package://box_model/urdf/box/mesh/2312_box_model_reduced_size.stl" scale="0.001 0.001 0.001" />
+      </geometry>
+    </visual>
+  </link>
+  <link name="cpt7_antenna_back_model">
+    <visual>
+      <geometry>
+        <mesh filename="package://box_model/urdf/box/mesh/2312_antenna_back_in_base_csys.stl" scale="0.001 0.001 0.001" />
       </geometry>
     </visual>
@@ -46,5 +68,5 @@
     <visual>
       <geometry>
-        <mesh filename="package://box_model/urdf/box/mesh/leica_small_prism.dae" />
+        <mesh filename="package://box_model/urdf/box/mesh/2312_prism_in_cpt7_csys.stl" scale="0.001 0.001 0.001" />
       </geometry>
     </visual>

File: box_model/box_model/urdf/box/box_calibrated.urdf.xacro (robot description, xacro)
@@ -32,5 +32,5 @@
     <joint name="box_base_to_box_base_model" type="fixed">
         <origin xyz="0.0 0.0 0.0" rpy="0.0 0.0 0.0"/>
-        <parent link="stim320_imu"/>
+        <parent link="box_base"/>
         <child link="box_base_model"/>
     </joint>

File: box_model/box_model/urdf/imus/imus.urdf.xacro (robot description, xacro)
@@ -61,14 +61,4 @@
     <child link="stim320_imu" />
   </joint>
-  <joint name="stim320_imu_to_box_base_model" type="fixed">
-    <origin xyz=" ${calib['stim320_imu_to_box_base_model']['x']}
-                  ${calib['stim320_imu_to_box_base_model']['y']}
-                  ${calib['stim320_imu_to_box_base_model']['z']}"
-            rpy=" ${calib['stim320_imu_to_box_base_model']['roll']}
-                  ${calib['stim320_imu_to_box_base_model']['pitch']}
-                  ${calib['stim320_imu_to_box_base_model']['yaw']}" />
-    <parent link="stim320_imu" />
-    <child link="box_base_model" />
-  </joint>
   <!-- IMU ADIS16475 -->
   <link name="adis16475_imu" />

Commit message: disabled unused links

File: box_model/box_model/urdf/box/box.urdf.xacro (robot description, xacro)
@@ -11,4 +11,5 @@
     <child link="box_base" />
   </joint>
+<!--
   <joint name="prism_to_prism_model" type="fixed">
     <origin xyz=" ${calib['prism_to_prism_model']['x']}
@@ -20,5 +21,5 @@
     <parent link="prism" />
     <child link="prism_model" />
-  </joint>
+  </joint> -->
   <!-- Prism -->
   <link name="prism"/>
@@ -45,17 +46,18 @@
         <child link="box_base_model"/>
   </joint>
-  <joint name="base_to_cpt7_antenna_back_model" type="fixed">
+  <!-- <joint name="base_to_cpt7_antenna_back_model" type="fixed">
         <origin xyz="0.0 0.0 0.0" rpy="0.0 0.0 0.0"/>
         <parent link="base"/>
         <child link="cpt7_antenna_back_model"/>
-  </joint>
+  </joint> -->
   <!-- Model base -->
   <link name="box_base_model">
     <visual>
       <geometry>
-        <mesh filename="package://box_model/urdf/box/mesh/2312_box_model_reduced_size.stl" scale="0.001 0.001 0.001" />
+        <mesh filename="package://box_model/urdf/box/mesh/box_colored.dae" scale="0.001 0.001 0.001" />
       </geometry>
     </visual>
   </link>
+<!--
   <link name="cpt7_antenna_back_model">
     <visual>
@@ -71,5 +73,5 @@
       </geometry>
     </visual>
-  </link>
+  </link> -->
   <xacro:include filename="$(find box_model)/urdf/cameras/cameras.urdf.xacro" />
   <xacro:include filename="$(find box_model)/urdf/lidars/lidars.urdf.xacro" />

File: box_model/box_model/urdf/lidars/lidars.urdf.xacro (robot description, xacro)
@@ -13,5 +13,5 @@
     <child link="hesai_lidar" />
   </joint>
-  <link name="hesai_model">
+  <!-- <link name="hesai_model">
     <visual>
       <geometry>
@@ -19,6 +19,6 @@
       </geometry>
     </visual>
-  </link>
-  <joint name="hesai_lidar_to_hesai_model" type="fixed">
+  </link> -->
+  <!-- <joint name="hesai_lidar_to_hesai_model" type="fixed">
     <origin xyz=" ${calib['hesai_lidar_to_hesai_model']['x']}
                   ${calib['hesai_lidar_to_hesai_model']['y']}
@@ -29,5 +29,5 @@
     <parent link="hesai_lidar" />
     <child link="hesai_model" />
-  </joint>
+  </joint> -->
   <!-- Livox -->
   <link name="livox_lidar" />
@@ -42,5 +42,5 @@
     <child link="livox_lidar" />
   </joint>
-  <link name="livox_model">
+  <!-- <link name="livox_model">
     <visual>
       <geometry>
@@ -48,6 +48,6 @@
       </geometry>
     </visual>
-  </link>
-  <joint name="livox_lidar_to_livox_model" type="fixed">
+  </link> -->
+  <!-- <joint name="livox_lidar_to_livox_model" type="fixed">
     <origin xyz=" ${calib['livox_lidar_to_livox_model']['x']}
                   ${calib['livox_lidar_to_livox_model']['y']}
@@ -58,5 +58,5 @@
     <parent link="livox_lidar" />
     <child link="livox_model" />
-  </joint>
+  </joint> -->
   <link name="livox_imu"/>
   <!-- From page 15 https://terra-1-g.djicdn.com/851d20f7b9f64838a34cd02351370894/Livox/Livox_Mid-360_User_Manual_EN.pdf -->

Commit message: updated urdf - to be visually correct

File: box_model/box_model/urdf/box/box.urdf.xacro (robot description, xacro)
@@ -5,7 +5,8 @@
 <!-- load the YAML calibration file into a property -->
 <xacro:property name="calib" value="${xacro.load_yaml(calib_file)}"/>
+  <!-- Wrong export origins in CAD - the coorect ones are xyz="0.0764038 -0.0361 0.2802790" -->
   <link name="base"/>
   <joint name="cpt7_to_robot_base" type="fixed">
-    <origin xyz="0.0764038 -0.0361 0.2802790" rpy="3.1415126 0.0 0.0" />
+    <origin xyz="0.0764038 -0.0461 0.2602790" rpy="3.1415126 0.0 0.0" />
     <parent link="base" />
     <child link="box_base" />
@@ -41,8 +42,21 @@
         <child link="prism"/>
   </joint>
+  <!-- Wrong export origins in CAD - the coorect ones are xyz="0 0 0" -->
   <joint name="box_base_to_box_base_model" type="fixed">
-        <origin xyz="0.0 0.0 0.0" rpy="0.0 0.0 0.0"/>
+        <origin xyz="0.004 -0.01 -0.007" rpy="0.0 0.0 0.0"/>
         <parent link="box_base"/>
         <child link="box_base_model"/>
+  </joint>
+  <!-- Wrong export origins in CAD - the coorect ones are xyz="0 0 0" -->
+  <joint name="box_base_to_prism_model" type="fixed">
+        <origin xyz="0.004 -0.01 -0.007" rpy="0.0 0.0 0.0"/>
+        <parent link="box_base"/>
+        <child link="prism_model"/>
+  </joint>
+  <!-- Wrong export origins in CAD - the coorect ones are xyz="0 0 0" -->
+  <joint name="base_to_cpt7_antenna_back_model" type="fixed">
+        <origin xyz="0 0 0.03 " rpy="0.0 0.0 0.0"/>
+        <parent link="base"/>
+        <child link="cpt7_antenna_back_model"/>
   </joint>
   <!-- <joint name="base_to_cpt7_antenna_back_model" type="fixed">
@@ -55,13 +69,12 @@
     <visual>
       <geometry>
-        <mesh filename="package://box_model/urdf/box/mesh/box_colored.dae" scale="0.001 0.001 0.001" />
+        <mesh filename="package://box_model/urdf/box/mesh/box_colored_units.dae" scale="1 1 1" />
       </geometry>
     </visual>
   </link>
-<!--
   <link name="cpt7_antenna_back_model">
     <visual>
       <geometry>
-        <mesh filename="package://box_model/urdf/box/mesh/2312_antenna_back_in_base_csys.stl" scale="0.001 0.001 0.001" />
+        <mesh filename="package://box_model/urdf/box/mesh/gps_colored_units.dae" scale="1 1 1" />
       </geometry>
     </visual>
@@ -70,8 +83,8 @@
     <visual>
       <geometry>
-        <mesh filename="package://box_model/urdf/box/mesh/2312_prism_in_cpt7_csys.stl" scale="0.001 0.001 0.001" />
+        <mesh filename="package://box_model/urdf/box/mesh/prism_colored_units.dae" scale="1 1 1" />
       </geometry>
     </visual>
-  </link> -->
+  </link>
   <xacro:include filename="$(find box_model)/urdf/cameras/cameras.urdf.xacro" />
   <xacro:include filename="$(find box_model)/urdf/lidars/lidars.urdf.xacro" />

Commit message: Undo visual fixes in URDF xacro

File: box_model/box_model/urdf/box/box.urdf.xacro (robot description, xacro)
@@ -44,5 +44,5 @@
   <!-- Wrong export origins in CAD - the coorect ones are xyz="0 0 0" -->
   <joint name="box_base_to_box_base_model" type="fixed">
-        <origin xyz="0.004 -0.01 -0.007" rpy="0.0 0.0 0.0"/>
+        <origin xyz="0.00 -0.0 -0.00" rpy="0.0 0.0 0.0"/>
         <parent link="box_base"/>
         <child link="box_base_model"/>
@@ -50,5 +50,5 @@
   <!-- Wrong export origins in CAD - the coorect ones are xyz="0 0 0" -->
   <joint name="box_base_to_prism_model" type="fixed">
-        <origin xyz="0.004 -0.01 -0.007" rpy="0.0 0.0 0.0"/>
+        <origin xyz="0.00 -0.0 -0.00" rpy="0.0 0.0 0.0"/>
         <parent link="box_base"/>
         <child link="prism_model"/>

Commit message: reverted tf_static base to box_base

File: box_model/box_model/urdf/box/box.urdf.xacro (robot description, xacro)
@@ -6,7 +6,8 @@
 <xacro:property name="calib" value="${xacro.load_yaml(calib_file)}"/>
   <!-- Wrong export origins in CAD - the coorect ones are xyz="0.0764038 -0.0361 0.2802790" -->
+  <!-- 0.0764038 -0.0461 0.2602790 manually tuned values -->
   <link name="base"/>
   <joint name="cpt7_to_robot_base" type="fixed">
-    <origin xyz="0.0764038 -0.0461 0.2602790" rpy="3.1415126 0.0 0.0" />
+    <origin xyz="0.0764038 -0.0361 0.2802790" rpy="3.1415126 0.0 0.0" />
     <parent link="base" />
     <child link="box_base" />

Commit message: added for final experiments

File: box_model/box_model/urdf/box/box.urdf.xacro (robot description, xacro)
@@ -28,5 +28,5 @@
   <!-- Box base -->
   <link name="box_base"/>
-  <!-- <joint name="box_base_to_prism" type="fixed">
+  <joint name="box_base_to_prism" type="fixed">
     <origin xyz=" ${calib['box_base_to_prism']['x']}
                   ${calib['box_base_to_prism']['y']}
@@ -37,10 +37,10 @@
     <parent link="box_base" />
     <child link="prism" />
-  </joint> -->
-  <joint name="box_base_to_prism" type="fixed">
+  </joint>
+  <!-- <joint name="box_base_to_prism" type="fixed">
         <origin xyz="0.0 0.0 0.0" rpy="0.0 0.0 0.0"/>
         <parent link="box_base"/>
         <child link="prism"/>
-  </joint>
+  </joint> -->
   <!-- Wrong export origins in CAD - the coorect ones are xyz="0 0 0" -->
   <joint name="box_base_to_box_base_model" type="fixed">

Commit message: final urdf

File: box_model/box_model/urdf/box/box.urdf.xacro (robot description, xacro)
@@ -70,5 +70,5 @@
     <visual>
       <geometry>
-        <mesh filename="package://box_model/urdf/box/mesh/box_colored_units.dae" scale="1 1 1" />
+        <mesh filename="package://box_model/urdf/box/mesh/box.dae" scale="1 1 1" />
       </geometry>
     </visual>
@@ -77,5 +77,5 @@
     <visual>
       <geometry>
-        <mesh filename="package://box_model/urdf/box/mesh/gps_colored_units.dae" scale="1 1 1" />
+        <mesh filename="package://box_model/urdf/box/mesh/gps.dae" scale="1 1 1" />
       </geometry>
     </visual>
@@ -84,5 +84,5 @@
     <visual>
       <geometry>
-        <mesh filename="package://box_model/urdf/box/mesh/prism_colored_units.dae" scale="1 1 1" />
+        <mesh filename="package://box_model/urdf/box/mesh/prism.dae" scale="1 1 1" />
       </geometry>
     </visual>

Commit message: verify TF with robot models, more cleaning and box_auto error handling

File: box_model/box_model/urdf/box/box.urdf.xacro (robot description, xacro)
@@ -56,9 +56,9 @@
   </joint>
   <!-- Wrong export origins in CAD - the coorect ones are xyz="0 0 0" -->
-  <joint name="base_to_cpt7_antenna_back_model" type="fixed">
+  <!-- <joint name="base_to_cpt7_antenna_back_model" type="fixed">
         <origin xyz="0 0 0.03 " rpy="0.0 0.0 0.0"/>
         <parent link="base"/>
         <child link="cpt7_antenna_back_model"/>
-  </joint>
+  </joint> -->
   <!-- <joint name="base_to_cpt7_antenna_back_model" type="fixed">
         <origin xyz="0.0 0.0 0.0" rpy="0.0 0.0 0.0"/>
@@ -74,5 +74,5 @@
     </visual>
   </link>
-  <link name="cpt7_antenna_back_model">
+  <!-- <link name="cpt7_antenna_back_model">
     <visual>
       <geometry>
@@ -80,5 +80,5 @@
       </geometry>
     </visual>
-  </link>
+  </link> -->
   <link name="prism_model">
     <visual>

Commit message: URDF issues tracked

File: box_model/box_model/urdf/box/box.urdf.xacro (robot description, xacro)
@@ -13,15 +13,4 @@
     <child link="box_base" />
   </joint>
-<!--
-  <joint name="prism_to_prism_model" type="fixed">
-    <origin xyz=" ${calib['prism_to_prism_model']['x']}
-                  ${calib['prism_to_prism_model']['y']}
-                  ${calib['prism_to_prism_model']['z']}"
-            rpy=" ${calib['prism_to_prism_model']['roll']}
-                  ${calib['prism_to_prism_model']['pitch']}
-                  ${calib['prism_to_prism_model']['yaw']}" />
-    <parent link="prism" />
-    <child link="prism_model" />
-  </joint> -->
   <!-- Prism -->
   <link name="prism"/>
@@ -38,12 +27,7 @@
     <child link="prism" />
   </joint>
-  <!-- <joint name="box_base_to_prism" type="fixed">
-        <origin xyz="0.0 0.0 0.0" rpy="0.0 0.0 0.0"/>
-        <parent link="box_base"/>
-        <child link="prism"/>
-  </joint> -->
   <!-- Wrong export origins in CAD - the coorect ones are xyz="0 0 0" -->
   <joint name="box_base_to_box_base_model" type="fixed">
-        <origin xyz="0.00 -0.0 -0.00" rpy="0.0 0.0 0.0"/>
+        <origin xyz="0.0 0.0 0.0" rpy="0.0 0.0 0.0"/>
         <parent link="box_base"/>
         <child link="box_base_model"/>
@@ -51,19 +35,14 @@
   <!-- Wrong export origins in CAD - the coorect ones are xyz="0 0 0" -->
   <joint name="box_base_to_prism_model" type="fixed">
-        <origin xyz="0.00 -0.0 -0.00" rpy="0.0 0.0 0.0"/>
+        <origin xyz="0.0 0.0 0.0" rpy="0.0 0.0 0.0"/>
         <parent link="box_base"/>
         <child link="prism_model"/>
   </joint>
   <!-- Wrong export origins in CAD - the coorect ones are xyz="0 0 0" -->
-  <!-- <joint name="base_to_cpt7_antenna_back_model" type="fixed">
-        <origin xyz="0 0 0.03 " rpy="0.0 0.0 0.0"/>
-        <parent link="base"/>
-        <child link="cpt7_antenna_back_model"/>
-  </joint> -->
-  <!-- <joint name="base_to_cpt7_antenna_back_model" type="fixed">
+  <joint name="base_to_cpt7_antenna_back_model" type="fixed">
         <origin xyz="0.0 0.0 0.0" rpy="0.0 0.0 0.0"/>
         <parent link="base"/>
         <child link="cpt7_antenna_back_model"/>
-  </joint> -->
+  </joint>
   <!-- Model base -->
   <link name="box_base_model">
@@ -74,5 +53,6 @@
     </visual>
   </link>
-  <!-- <link name="cpt7_antenna_back_model">
+  <!-- Back antenna -->
+  <link name="cpt7_antenna_back_model">
     <visual>
       <geometry>
@@ -80,5 +60,6 @@
       </geometry>
     </visual>
-  </link> -->
+  </link>
+  <!-- Leica Mini prism -->
   <link name="prism_model">
     <visual>
@@ -88,4 +69,5 @@
     </visual>
   </link>
+  <!-- Sensors -->
   <xacro:include filename="$(find box_model)/urdf/cameras/cameras.urdf.xacro" />
   <xacro:include filename="$(find box_model)/urdf/lidars/lidars.urdf.xacro" />
