Commit message: combined tf compatible with urdfs

File: box_model/box_model/urdf/box/box.urdf.xacro (robot description, xacro)
@@ -1,10 +1,12 @@
 <?xml version="1.0" ?>
 <robot name="box" xmlns:xacro="http://www.ros.org/wiki/xacro">
+  <!-- Declare all arguments BEFORE any usage -->
+  <xacro:arg name="enable_visualizable_model" default="false"/>
+  <xacro:property name="enable_visualizable_model_arg" value="$(arg enable_visualizable_model)" />
 <!-- YAML file containing the default values from CAD -->
 <xacro:property name="calib_file" value="$(find box_calibration)/calibration/tf/calibration_latest.yaml" />
 <!-- load the YAML calibration file into a property -->
 <xacro:property name="calib" value="${xacro.load_yaml(calib_file)}"/>
-  <!-- Wrong export origins in CAD - the coorect ones are xyz="0.0764038 -0.0361 0.2802790" -->
-  <!-- 0.0764038 -0.0461 0.2602790 manually tuned values -->
+<!-- YAML file containing the default values from CAD -->
   <link name="base"/>
   <joint name="cpt7_to_robot_base" type="fixed">
@@ -15,5 +17,4 @@
   <!-- Prism -->
   <link name="prism"/>
-  <!-- Box base -->
   <link name="box_base"/>
   <joint name="box_base_to_prism" type="fixed">
@@ -27,5 +28,5 @@
     <child link="prism" />
   </joint>
-  <!-- Wrong export origins in CAD - the coorect ones are xyz="0 0 0" -->
+  <!-- Box model -->
   <joint name="box_base_to_box_base_model" type="fixed">
         <origin xyz="0.0 0.0 0.0" rpy="0.0 0.0 0.0"/>
@@ -33,5 +34,5 @@
         <child link="box_base_model"/>
   </joint>
-  <!-- Wrong export origins in CAD - the coorect ones are xyz="0 0 0" -->
+  <!-- Prism model -->
   <joint name="box_base_to_prism_model" type="fixed">
         <origin xyz="0.0 0.0 0.0" rpy="0.0 0.0 0.0"/>
@@ -39,5 +40,5 @@
         <child link="prism_model"/>
   </joint>
-  <!-- Wrong export origins in CAD - the coorect ones are xyz="0 0 0" -->
+  <!-- Back antenna model -->
   <joint name="base_to_cpt7_antenna_back_model" type="fixed">
         <origin xyz="0.0 0.0 0.0" rpy="0.0 0.0 0.0"/>
@@ -45,5 +46,13 @@
         <child link="cpt7_antenna_back_model"/>
   </joint>
-  <!-- Model base -->
+  <!-- Back antenna mesh -->
+  <link name="cpt7_antenna_back_model">
+    <visual>
+      <geometry>
+        <mesh filename="package://box_model/urdf/box/mesh/gps.dae" scale="1 1 1" />
+      </geometry>
+    </visual>
+  </link>
+  <!-- Box Model Mesh -->
   <link name="box_base_model">
     <visual>
@@ -53,13 +62,5 @@
     </visual>
   </link>
-  <!-- Back antenna -->
-  <link name="cpt7_antenna_back_model">
-    <visual>
-      <geometry>
-        <mesh filename="package://box_model/urdf/box/mesh/gps.dae" scale="1 1 1" />
-      </geometry>
-    </visual>
-  </link>
-  <!-- Leica Mini prism -->
+  <!-- Leica Mini prism model -->
   <link name="prism_model">
     <visual>
@@ -70,6 +71,10 @@
   </link>
   <!-- Sensors -->
+  <!-- Sensor meshes are baked into the box mesh. -->
   <xacro:include filename="$(find box_model)/urdf/cameras/cameras.urdf.xacro" />
+  <xacro:viz_param_cameras enable_visualizable_model="${enable_visualizable_model_arg}"/>
   <xacro:include filename="$(find box_model)/urdf/lidars/lidars.urdf.xacro" />
+  <xacro:viz_param_lidars enable_visualizable_model="${enable_visualizable_model_arg}"/>
   <xacro:include filename="$(find box_model)/urdf/imus/imus.urdf.xacro" />
+  <xacro:viz_param_imus enable_visualizable_model="${enable_visualizable_model_arg}"/>
 </robot>

File: box_model/box_model/urdf/cameras/cameras.urdf.xacro (robot description, xacro)
@@ -1,4 +1,6 @@
 <?xml version="1.0" ?>
 <robot name="cameras" xmlns:xacro="http://www.ros.org/wiki/xacro">
+  <xacro:macro name="viz_param_cameras" params="enable_visualizable_model"/>
+  <xacro:property name="enable_visualizable_model_prop" value="$(arg enable_visualizable_model)" />
     <!-- ////////// Alphasense ////////// -->
     <!-- Alphasense base (coincides with alphasense Cam1/ front center) -->
@@ -14,4 +16,6 @@
         <child link="alphasense_base"/>
     </joint>
+    <xacro:unless value="${enable_visualizable_model_prop}">
+    <!-- We disable, as these frames are renamed in the URDF after calibration. -->
     <link name="alphasense_front_center"/>
     <joint name="alphasense_front_center_identity" type="fixed">
@@ -129,4 +133,5 @@
         <child link="cam5_sensor_frame"/>
     </joint>
+    </xacro:unless>
     <!-- ////////// HDR ////////// -->
     <!-- HDR Base (coincides with front hdr cam) -->
@@ -179,92 +184,96 @@
     </joint>
     <!-- ////////// ZED2i ////////// -->
-    <!-- ZED Base -->
-    <link name="zed_base_link"/>
-    <joint name="box_base_to_zed_base" type="fixed">
-        <origin xyz=" ${calib['box_base_to_zed_base']['x']}
-                  ${calib['box_base_to_zed_base']['y']}
-                  ${calib['box_base_to_zed_base']['z']}"
-                rpy=" ${calib['box_base_to_zed_base']['roll']}
-                  ${calib['box_base_to_zed_base']['pitch']}
-                  ${calib['box_base_to_zed_base']['yaw']}"/>
-        <parent link="box_base"/>
-        <child link="zed_base_link"/>
-    </joint>
-    <link name="zed2i_base_link"/>
-    <joint name="zed2i_base_helper_joint" type="fixed">
-        <origin xyz=" ${calib['zed2i_base_helper_joint']['x']}
-                  ${calib['zed2i_base_helper_joint']['y']}
-                  ${calib['zed2i_base_helper_joint']['z']}"
-                rpy=" ${calib['zed2i_base_helper_joint']['roll']}
-                  ${calib['zed2i_base_helper_joint']['pitch']}
-                  ${calib['zed2i_base_helper_joint']['yaw']}"/>
-        <parent link="zed_base_link"/>
-        <child link="zed2i_base_link"/>
-    </joint>
-    <link name="zed2i_camera_center"/>
-    <joint name="zed2i_base_to_camera_center" type="fixed">
-        <origin xyz=" ${calib['zed2i_base_to_camera_center']['x']}
-                  ${calib['zed2i_base_to_camera_center']['y']}
-                  ${calib['zed2i_base_to_camera_center']['z']}"
-                rpy=" ${calib['zed2i_base_to_camera_center']['roll']}
-                  ${calib['zed2i_base_to_camera_center']['pitch']}
-                  ${calib['zed2i_base_to_camera_center']['yaw']}"/>
-        <parent link="zed2i_base_link"/>
-        <child link="zed2i_camera_center"/>
-    </joint>
-    <link name="zed2i_left_camera_frame"/>
-    <joint name="zed_camera_center_to_zed_left" type="fixed">
-        <origin xyz=" ${calib['zed_camera_center_to_zed_left']['x']}
-                  ${calib['zed_camera_center_to_zed_left']['y']}
-                  ${calib['zed_camera_center_to_zed_left']['z']}"
-                rpy=" ${calib['zed_camera_center_to_zed_left']['roll']}
-                  ${calib['zed_camera_center_to_zed_left']['pitch']}
-                  ${calib['zed_camera_center_to_zed_left']['yaw']}"/>
-        <parent link="zed2i_camera_center"/>
-        <child link="zed2i_left_camera_frame"/>
-    </joint>
-    <link name="zed2i_left_camera_optical_frame"/>
-    <joint name="zed_left_to_optical" type="fixed">
-        <origin xyz=" ${calib['zed_left_to_left_optical']['x']}
-                  ${calib['zed_left_to_left_optical']['y']}
-                  ${calib['zed_left_to_left_optical']['z']}"
-                rpy=" ${calib['zed_left_to_left_optical']['roll']}
-                  ${calib['zed_left_to_left_optical']['pitch']}
-                  ${calib['zed_left_to_left_optical']['yaw']}"/>
-        <parent link="zed2i_left_camera_frame"/>
-        <child link="zed2i_left_camera_optical_frame"/>
-    </joint>
-    <link name="zed2i_imu_link"/>
-    <joint name="zed_left_camera_frame_to_zed_imu_joint" type="fixed">
-        <origin xyz=" ${calib['zed_left_camera_frame_to_zed_imu']['x']}
-                  ${calib['zed_left_camera_frame_to_zed_imu']['y']}
-                  ${calib['zed_left_camera_frame_to_zed_imu']['z']}"
-                rpy=" ${calib['zed_left_camera_frame_to_zed_imu']['roll']}
-                  ${calib['zed_left_camera_frame_to_zed_imu']['pitch']}
-                  ${calib['zed_left_camera_frame_to_zed_imu']['yaw']}"/>
-        <parent link="zed2i_left_camera_frame"/>
-        <child link="zed2i_imu_link"/>
-    </joint>
-    <link name="zed2i_right_camera_optical_frame"/>
-    <joint name="zed_left_optical_to_zed_right_optical" type="fixed">
-        <origin xyz=" ${calib['zed_left_optical_to_zed_right_optical']['x']}
-                  ${calib['zed_left_optical_to_zed_right_optical']['y']}
-                  ${calib['zed_left_optical_to_zed_right_optical']['z']}"
-                rpy=" ${calib['zed_left_optical_to_zed_right_optical']['roll']}
-                  ${calib['zed_left_optical_to_zed_right_optical']['pitch']}
-                  ${calib['zed_left_optical_to_zed_right_optical']['yaw']}"/>
-        <parent link="zed2i_left_camera_optical_frame"/>
-        <child link="zed2i_right_camera_optical_frame"/>
-    </joint>
-    <link name="zed2i_right_camera_frame"/>
-    <joint name="zed_camera_center_to_zed_right" type="fixed">
-        <origin xyz=" ${calib['zed_right_to_right_optical']['x']}
-                  ${calib['zed_right_to_right_optical']['y']}
-                  ${calib['zed_right_to_right_optical']['z']}"
-                rpy=" ${calib['zed_right_to_right_optical']['roll']}
-                  ${calib['zed_right_to_right_optical']['pitch']}
-                  ${calib['zed_right_to_right_optical']['yaw']}"/>
-        <parent link="zed2i_right_camera_optical_frame"/>
-        <child link="zed2i_right_camera_frame"/>
-    </joint>
+    <!-- when enable_visualizable_model_prop is true, it results to. -->
+    <!-- Visualization suppoted model enabled. zed2i_base->zed2i_left, zed2i_right, zed2i_imu -->
+    <xacro:unless value="${enable_visualizable_model_prop}">
+      <!-- ZED Base -->
+      <link name="zed_base_link"/>
+      <joint name="box_base_to_zed_base" type="fixed">
+          <origin xyz=" ${calib['box_base_to_zed_base']['x']}
+                    ${calib['box_base_to_zed_base']['y']}
+                    ${calib['box_base_to_zed_base']['z']}"
+                  rpy=" ${calib['box_base_to_zed_base']['roll']}
+                    ${calib['box_base_to_zed_base']['pitch']}
+                    ${calib['box_base_to_zed_base']['yaw']}"/>
+          <parent link="box_base"/>
+          <child link="zed_base_link"/>
+      </joint>
+      <link name="zed2i_base_link"/>
+      <joint name="zed2i_base_helper_joint" type="fixed">
+          <origin xyz=" ${calib['zed2i_base_helper_joint']['x']}
+                    ${calib['zed2i_base_helper_joint']['y']}
+                    ${calib['zed2i_base_helper_joint']['z']}"
+                  rpy=" ${calib['zed2i_base_helper_joint']['roll']}
+                    ${calib['zed2i_base_helper_joint']['pitch']}
+                    ${calib['zed2i_base_helper_joint']['yaw']}"/>
+          <parent link="zed_base_link"/>
+          <child link="zed2i_base_link"/>
+      </joint>
+      <link name="zed2i_camera_center"/>
+      <joint name="zed2i_base_to_camera_center" type="fixed">
+          <origin xyz=" ${calib['zed2i_base_to_camera_center']['x']}
+                    ${calib['zed2i_base_to_camera_center']['y']}
+                    ${calib['zed2i_base_to_camera_center']['z']}"
+                  rpy=" ${calib['zed2i_base_to_camera_center']['roll']}
+                    ${calib['zed2i_base_to_camera_center']['pitch']}
+                    ${calib['zed2i_base_to_camera_center']['yaw']}"/>
+          <parent link="zed2i_base_link"/>
+          <child link="zed2i_camera_center"/>
+      </joint>
+      <link name="zed2i_left_camera_frame"/>
+      <joint name="zed_camera_center_to_zed_left" type="fixed">
+          <origin xyz=" ${calib['zed_camera_center_to_zed_left']['x']}
+                    ${calib['zed_camera_center_to_zed_left']['y']}
+                    ${calib['zed_camera_center_to_zed_left']['z']}"
+                  rpy=" ${calib['zed_camera_center_to_zed_left']['roll']}
+                    ${calib['zed_camera_center_to_zed_left']['pitch']}
+                    ${calib['zed_camera_center_to_zed_left']['yaw']}"/>
+          <parent link="zed2i_camera_center"/>
+          <child link="zed2i_left_camera_frame"/>
+      </joint>
+      <link name="zed2i_left_camera_optical_frame"/>
+      <joint name="zed_left_to_optical" type="fixed">
+          <origin xyz=" ${calib['zed_left_to_left_optical']['x']}
+                    ${calib['zed_left_to_left_optical']['y']}
+                    ${calib['zed_left_to_left_optical']['z']}"
+                  rpy=" ${calib['zed_left_to_left_optical']['roll']}
+                    ${calib['zed_left_to_left_optical']['pitch']}
+                    ${calib['zed_left_to_left_optical']['yaw']}"/>
+          <parent link="zed2i_left_camera_frame"/>
+          <child link="zed2i_left_camera_optical_frame"/>
+      </joint>
+      <link name="zed2i_imu_link"/>
+      <joint name="zed_left_camera_frame_to_zed_imu_joint" type="fixed">
+          <origin xyz=" ${calib['zed_left_camera_frame_to_zed_imu']['x']}
+                    ${calib['zed_left_camera_frame_to_zed_imu']['y']}
+                    ${calib['zed_left_camera_frame_to_zed_imu']['z']}"
+                  rpy=" ${calib['zed_left_camera_frame_to_zed_imu']['roll']}
+                    ${calib['zed_left_camera_frame_to_zed_imu']['pitch']}
+                    ${calib['zed_left_camera_frame_to_zed_imu']['yaw']}"/>
+          <parent link="zed2i_left_camera_frame"/>
+          <child link="zed2i_imu_link"/>
+      </joint>
+      <link name="zed2i_right_camera_optical_frame"/>
+      <joint name="zed_left_optical_to_zed_right_optical" type="fixed">
+          <origin xyz=" ${calib['zed_left_optical_to_zed_right_optical']['x']}
+                    ${calib['zed_left_optical_to_zed_right_optical']['y']}
+                    ${calib['zed_left_optical_to_zed_right_optical']['z']}"
+                  rpy=" ${calib['zed_left_optical_to_zed_right_optical']['roll']}
+                    ${calib['zed_left_optical_to_zed_right_optical']['pitch']}
+                    ${calib['zed_left_optical_to_zed_right_optical']['yaw']}"/>
+          <parent link="zed2i_left_camera_optical_frame"/>
+          <child link="zed2i_right_camera_optical_frame"/>
+      </joint>
+      <link name="zed2i_right_camera_frame"/>
+      <joint name="zed_camera_center_to_zed_right" type="fixed">
+          <origin xyz=" ${calib['zed_right_to_right_optical']['x']}
+                    ${calib['zed_right_to_right_optical']['y']}
+                    ${calib['zed_right_to_right_optical']['z']}"
+                  rpy=" ${calib['zed_right_to_right_optical']['roll']}
+                    ${calib['zed_right_to_right_optical']['pitch']}
+                    ${calib['zed_right_to_right_optical']['yaw']}"/>
+          <parent link="zed2i_right_camera_optical_frame"/>
+          <child link="zed2i_right_camera_frame"/>
+      </joint>
+    </xacro:unless>
 </robot>

File: box_model/box_model/urdf/imus/imus.urdf.xacro (robot description, xacro)
@@ -1,4 +1,6 @@
 <?xml version="1.0" ?>
 <robot name="imus" xmlns:xacro="http://www.ros.org/wiki/xacro">
+  <xacro:macro name="viz_param_imus" params="enable_visualizable_model"/>
+  <xacro:property name="enable_visualizable_model_prop" value="$(arg enable_visualizable_model)" />
   <link name="cpt7_imu"/>
   <!-- CPT7 Coordinate System -->
@@ -13,4 +15,5 @@
     <child link="cpt7_imu" />
   </joint>
+  <xacro:unless value="${enable_visualizable_model_prop}">
   <link name="cpt7_antenna_front"/>
   <!-- CPT7 Coordinate System -->
@@ -37,4 +40,5 @@
     <child link="cpt7_antenna_back" />
   </joint>
+  </xacro:unless>
   <link name="ap20_imu"/>
   <!-- Basilisk IMU Frame -->
@@ -73,15 +77,31 @@
     <child link="adis16475_imu" />
   </joint>
-  <!-- IMU alphasesnse -->
-  <link name="imu_sensor_frame" />
-  <joint name="box_base_to_imu_alphasense" type="fixed">
-    <origin xyz=" ${calib['box_base_to_imu_alphasense']['x']}
-                  ${calib['box_base_to_imu_alphasense']['y']}
-                  ${calib['box_base_to_imu_alphasense']['z']}"
-            rpy=" ${calib['box_base_to_imu_alphasense']['roll']}
-                  ${calib['box_base_to_imu_alphasense']['pitch']}
-                  ${calib['box_base_to_imu_alphasense']['yaw']}" />
-    <parent link="box_base" />
-    <child link="imu_sensor_frame" />
-  </joint>
+  <xacro:if value="${enable_visualizable_model_prop}">
+  <!-- Visualization supported model enabled. imu_sensor_frame->alphasense_imu -->
+    <!-- IMU Alphasense -->
+    <link name="alphasense_imu" />
+    <joint name="box_base_to_imu_alphasense" type="fixed">
+      <origin xyz=" ${calib['box_base_to_imu_alphasense']['x']}
+                    ${calib['box_base_to_imu_alphasense']['y']}
+                    ${calib['box_base_to_imu_alphasense']['z']}"
+              rpy=" ${calib['box_base_to_imu_alphasense']['roll']}
+                    ${calib['box_base_to_imu_alphasense']['pitch']}
+                    ${calib['box_base_to_imu_alphasense']['yaw']}" />
+      <parent link="box_base" />
+      <child link="alphasense_imu" />
+    </joint>
+  </xacro:if>
+  <xacro:unless value="${enable_visualizable_model_prop}">
+    <link name="imu_sensor_frame" />
+    <joint name="box_base_to_imu_alphasense" type="fixed">
+      <origin xyz=" ${calib['box_base_to_imu_alphasense']['x']}
+                    ${calib['box_base_to_imu_alphasense']['y']}
+                    ${calib['box_base_to_imu_alphasense']['z']}"
+              rpy=" ${calib['box_base_to_imu_alphasense']['roll']}
+                    ${calib['box_base_to_imu_alphasense']['pitch']}
+                    ${calib['box_base_to_imu_alphasense']['yaw']}" />
+      <parent link="box_base" />
+      <child link="imu_sensor_frame" />
+    </joint>
+  </xacro:unless>
 </robot>

File: box_model/box_model/urdf/lidars/lidars.urdf.xacro (robot description, xacro)
@@ -1,4 +1,6 @@
 <?xml version="1.0" ?>
 <robot name="lidars" xmlns:xacro="http://www.ros.org/wiki/xacro">
+  <xacro:macro name="viz_param_lidars" params="enable_visualizable_model"/>
+  <xacro:property name="enable_visualizable_model_prop" value="$(arg enable_visualizable_model)" />
   <!-- hesai_lidar -->
   <link name="hesai_lidar" />
@@ -13,21 +15,19 @@
     <child link="hesai_lidar" />
   </joint>
-  <!-- <link name="hesai_model">
-    <visual>
-      <geometry>
-        <mesh filename="package://box_model/urdf/box/mesh/hesai_lidar.dae" />
-      </geometry>
-    </visual>
-  </link> -->
-  <!-- <joint name="hesai_lidar_to_hesai_model" type="fixed">
-    <origin xyz=" ${calib['hesai_lidar_to_hesai_model']['x']}
-                  ${calib['hesai_lidar_to_hesai_model']['y']}
-                  ${calib['hesai_lidar_to_hesai_model']['z']}"
-            rpy=" ${calib['hesai_lidar_to_hesai_model']['roll']}
-                  ${calib['hesai_lidar_to_hesai_model']['pitch']}
-                  ${calib['hesai_lidar_to_hesai_model']['yaw']}" />
-    <parent link="hesai_lidar" />
-    <child link="hesai_model" />
-  </joint> -->
+  <!-- If enable_visualizable_model_prop is false block will execute -->
+  <xacro:unless value="${enable_visualizable_model_prop}">
+    <!-- hesai_model -->
+    <link name="hesai_model" />
+    <joint name="hesai_lidar_to_hesai_model" type="fixed">
+      <origin xyz=" ${calib['hesai_lidar_to_hesai_model']['x']}
+                    ${calib['hesai_lidar_to_hesai_model']['y']}
+                    ${calib['hesai_lidar_to_hesai_model']['z']}"
+              rpy=" ${calib['hesai_lidar_to_hesai_model']['roll']}
+                    ${calib['hesai_lidar_to_hesai_model']['pitch']}
+                    ${calib['hesai_lidar_to_hesai_model']['yaw']}" />
+      <parent link="hesai_lidar" />
+      <child link="hesai_model" />
+    </joint>
+  </xacro:unless>
   <!-- Livox -->
   <link name="livox_lidar" />
@@ -42,21 +42,17 @@
     <child link="livox_lidar" />
   </joint>
-  <!-- <link name="livox_model">
-    <visual>
-      <geometry>
-        <mesh filename="package://box_model/urdf/box/mesh/livox_mid360_lidar.dae" />
-      </geometry>
-    </visual>
-  </link> -->
-  <!-- <joint name="livox_lidar_to_livox_model" type="fixed">
-    <origin xyz=" ${calib['livox_lidar_to_livox_model']['x']}
-                  ${calib['livox_lidar_to_livox_model']['y']}
-                  ${calib['livox_lidar_to_livox_model']['z']}"
-            rpy=" ${calib['livox_lidar_to_livox_model']['roll']}
-                  ${calib['livox_lidar_to_livox_model']['pitch']}
-                  ${calib['livox_lidar_to_livox_model']['yaw']}" />
-    <parent link="livox_lidar" />
-    <child link="livox_model" />
-  </joint> -->
+  <xacro:unless value="${enable_visualizable_model_prop}">
+    <link name="livox_model" />
+    <joint name="livox_lidar_to_livox_model" type="fixed">
+      <origin xyz=" ${calib['livox_lidar_to_livox_model']['x']}
+                    ${calib['livox_lidar_to_livox_model']['y']}
+                    ${calib['livox_lidar_to_livox_model']['z']}"
+              rpy=" ${calib['livox_lidar_to_livox_model']['roll']}
+                    ${calib['livox_lidar_to_livox_model']['pitch']}
+                    ${calib['livox_lidar_to_livox_model']['yaw']}" />
+      <parent link="livox_lidar" />
+      <child link="livox_model" />
+    </joint>
+  </xacro:unless>
   <link name="livox_imu"/>
   <!-- From page 15 https://terra-1-g.djicdn.com/851d20f7b9f64838a34cd02351370894/Livox/Livox_Mid-360_User_Manual_EN.pdf -->

Commit message: Add new model daes

File: box_model/box_model/urdf/box/box.urdf.xacro (robot description, xacro)
@@ -34,4 +34,10 @@
         <child link="box_base_model"/>
   </joint>
+  <!-- Spider model -->
+  <joint name="box_base_to_spider" type="fixed">
+        <origin xyz="0.0 0.0 0.0" rpy="0.0 0.0 0.0"/>
+        <parent link="box_base"/>
+        <child link="spider"/>
+  </joint>
   <!-- Prism model -->
   <joint name="box_base_to_prism_model" type="fixed">
@@ -46,4 +52,12 @@
         <child link="cpt7_antenna_back_model"/>
   </joint>
+  <!-- Spider -->
+  <link name="spider">
+    <visual>
+      <geometry>
+        <mesh filename="package://box_model/urdf/box/mesh/spider.dae" scale="1 1 1" />
+      </geometry>
+    </visual>
+  </link>
   <!-- Back antenna mesh -->
   <link name="cpt7_antenna_back_model">
