Commit message: Add Livox IMU frame to URDF

File: box_model/box_model/urdf/lidars/lidars.urdf.xacro (robot description, xacro)
@@ -49,3 +49,10 @@
     <child link="livox_model" />
   </joint>
+  <link name="livox_frame">
+  <!-- From page 15 https://terra-1-g.djicdn.com/851d20f7b9f64838a34cd02351370894/Livox/Livox_Mid-360_User_Manual_EN.pdf -->
+  <joint name="livox_to_livox_imu_frame" type="fixed">
+    <origin xyz="0.011 0.02329 -0.04412" rpy="0.0 0.0 0.0" />
+    <parent link="livox" />
+    <child link="livox_frame" />
+  </joint>
 </robot>

Commit message: Update hesai model name

File: box_model/box_model/urdf/lidars/lidars.urdf.xacro (robot description, xacro)
@@ -13,5 +13,5 @@
     <child link="hesaiXT32" />
   </joint>
-  <link name="hesaiXT32_model">
+  <link name="hesai_model">
     <visual>
       <geometry>
@@ -20,8 +20,8 @@
     </visual>
   </link>
-  <joint name="hesaiXT32_to_hesaiXT32_model" type="fixed">
+  <joint name="hesaiXT32_to_hesai_model" type="fixed">
     <origin xyz="0.0 0.0 0.0" rpy="0.0 0.0 0.0" />
     <parent link="hesaiXT32" />
-    <child link="hesaiXT32_model" />
+    <child link="hesai_model" />
   </joint>
   <!-- Livox -->

Commit message: Update hesai lidar reference frame ID in lidar driver and URDF

File: box_model/box_model/urdf/lidars/lidars.urdf.xacro (robot description, xacro)
@@ -1,6 +1,6 @@
 <?xml version="1.0" ?>
 <robot name="lidars" xmlns:xacro="http://www.ros.org/wiki/xacro">
-  <!-- hesaiXT32 -->
-  <link name="hesaiXT32" />
+  <!-- hesai_lidar -->
+  <link name="hesai_lidar" />
   <joint name="box_base_to_hesai" type="fixed">
     <origin xyz=" ${calib['box_base_to_hesai']['x']}
@@ -11,5 +11,5 @@
                   ${calib['box_base_to_hesai']['yaw']}" />
     <parent link="box_base" />
-    <child link="hesaiXT32" />
+    <child link="hesai_lidar" />
   </joint>
   <link name="hesai_model">
@@ -20,7 +20,7 @@
     </visual>
   </link>
-  <joint name="hesaiXT32_to_hesai_model" type="fixed">
+  <joint name="hesai_lidar_to_hesai_model" type="fixed">
     <origin xyz="0.0 0.0 0.0" rpy="0.0 0.0 0.0" />
-    <parent link="hesaiXT32" />
+    <parent link="hesai_lidar" />
     <child link="hesai_model" />
   </joint>

Commit message: Update livox lidar frame names

File: box_model/box_model/urdf/lidars/lidars.urdf.xacro (robot description, xacro)
@@ -26,5 +26,5 @@
   </joint>
   <!-- Livox -->
-  <link name="livox" />
+  <link name="livox_lidar" />
   <joint name="box_base_to_livox" type="fixed">
     <origin xyz=" ${calib['box_base_to_livox']['x']}
@@ -35,5 +35,5 @@
                   ${calib['box_base_to_livox']['yaw']}" />
     <parent link="box_base" />
-    <child link="livox" />
+    <child link="livox_lidar" />
   </joint>
   <link name="livox_model">
@@ -46,5 +46,5 @@
   <joint name="livox_to_livox_model" type="fixed">
     <origin xyz="0.0 0.0 0.0" rpy="0.0 0.0 0.0" />
-    <parent link="livox" />
+    <parent link="livox_lidar" />
     <child link="livox_model" />
   </joint>
@@ -53,5 +53,5 @@
   <joint name="livox_to_livox_imu_frame" type="fixed">
     <origin xyz="0.011 0.02329 -0.04412" rpy="0.0 0.0 0.0" />
-    <parent link="livox" />
+    <parent link="livox_lidar" />
     <child link="livox_frame" />
   </joint>

Commit message: Update livox imu frame in urdf

File: box_model/box_model/urdf/lidars/lidars.urdf.xacro (robot description, xacro)
@@ -49,10 +49,10 @@
     <child link="livox_model" />
   </joint>
-  <link name="livox_frame"/>
+  <link name="livox_imu"/>
   <!-- From page 15 https://terra-1-g.djicdn.com/851d20f7b9f64838a34cd02351370894/Livox/Livox_Mid-360_User_Manual_EN.pdf -->
   <joint name="livox_to_livox_imu_frame" type="fixed">
     <origin xyz="0.011 0.02329 -0.04412" rpy="0.0 0.0 0.0" />
     <parent link="livox_lidar" />
-    <child link="livox_frame" />
+    <child link="livox_imu" />
   </joint>
 </robot>
