Commit message: add alphasense imu

File: box_model/box_model/urdf/imus/imus.urdf.xacro (robot description, xacro)
@@ -25,3 +25,15 @@
     <child link="imu_adis16475" />
   </joint>
+  <!-- IMU alphasesnse -->
+  <link name="imu_alphasense" />
+  <joint name="alphasense_front_left_to_imu_alphasense" type="fixed">
+    <origin xyz=" ${calib['alphasense_front_left_to_imu_alphasense']['x']}
+                  ${calib['alphasense_front_left_to_imu_alphasense']['y']}
+                  ${calib['alphasense_front_left_to_imu_alphasense']['z']}"
+            rpy=" ${calib['alphasense_front_left_to_imu_alphasense']['roll']}
+                  ${calib['alphasense_front_left_to_imu_alphasense']['pitch']}
+                  ${calib['alphasense_front_left_to_imu_alphasense']['yaw']}" />
+    <parent link="alphasense_front_left" />
+    <child link="imu_alphasense" />
+  </joint>
 </robot>

Commit message: Update Alphasense IMU frame name

File: box_model/box_model/urdf/imus/imus.urdf.xacro (robot description, xacro)
@@ -26,5 +26,5 @@
   </joint>
   <!-- IMU alphasesnse -->
-  <link name="imu_alphasense" />
+  <link name="imu_sensor_frame" />
   <joint name="box_base_to_imu_alphasense" type="fixed">
     <origin xyz=" ${calib['box_base_to_imu_alphasense']['x']}
@@ -35,5 +35,5 @@
                   ${calib['box_base_to_imu_alphasense']['yaw']}" />
     <parent link="box_base" />
-    <child link="imu_alphasense" />
+    <child link="imu_sensor_frame" />
   </joint>
 </robot>

Commit message: Also change stim320 frame name in URDF

File: box_model/box_model/urdf/imus/imus.urdf.xacro (robot description, xacro)
@@ -2,5 +2,5 @@
 <robot name="imus" xmlns:xacro="http://www.ros.org/wiki/xacro">
   <!-- IMU STIM320 -->
-  <link name="imu_stim320" />
+  <link name="stim320_imu" />
   <joint name="box_base_to_imu_stim320" type="fixed">
     <origin xyz=" ${calib['box_base_to_imu_stim320']['x']}
@@ -11,5 +11,5 @@
                   ${calib['box_base_to_imu_stim320']['yaw']}" />
     <parent link="box_base" />
-    <child link="imu_stim320" />
+    <child link="stim320_imu" />
   </joint>
   <!-- IMU ADIS16475 -->
