Commit message: Adding calibration import library and script

File: box_model/box_model/urdf/cameras/cameras.urdf.xacro (robot description, xacro)
@@ -16,11 +16,11 @@
   <!-- Alphasense Cam0/ front left (should be identity)-->
   <link name="alphasense_front_left" />
-  <joint name="alphasesnse_base_to_alphasense_front_left" type="fixed">
-    <origin xyz=" ${calib['alphasesnse_base_to_alphasense_front_left']['x']}
-                  ${calib['alphasesnse_base_to_alphasense_front_left']['y']}
-                  ${calib['alphasesnse_base_to_alphasense_front_left']['z']}"
-            rpy=" ${calib['alphasesnse_base_to_alphasense_front_left']['roll']}
-                  ${calib['alphasesnse_base_to_alphasense_front_left']['pitch']}
-                  ${calib['alphasesnse_base_to_alphasense_front_left']['yaw']}" />
+  <joint name="alphasense_base_to_alphasense_front_left" type="fixed">
+    <origin xyz=" ${calib['alphasense_base_to_alphasense_front_left']['x']}
+                  ${calib['alphasense_base_to_alphasense_front_left']['y']}
+                  ${calib['alphasense_base_to_alphasense_front_left']['z']}"
+            rpy=" ${calib['alphasense_base_to_alphasense_front_left']['roll']}
+                  ${calib['alphasense_base_to_alphasense_front_left']['pitch']}
+                  ${calib['alphasense_base_to_alphasense_front_left']['yaw']}" />
     <parent link="alphasense_base" />
     <child link="alphasense_front_left" />
@@ -28,11 +28,11 @@
   <!-- Alphasense Cam1/ front right -->
   <link name="alphasense_front_right" />
-  <joint name="alphasesnse_base_to_alphasense_front_right" type="fixed">
-    <origin xyz=" ${calib['alphasesnse_base_to_alphasense_front_right']['x']}
-                  ${calib['alphasesnse_base_to_alphasense_front_right']['y']}
-                  ${calib['alphasesnse_base_to_alphasense_front_right']['z']}"
-            rpy=" ${calib['alphasesnse_base_to_alphasense_front_right']['roll']}
-                  ${calib['alphasesnse_base_to_alphasense_front_right']['pitch']}
-                  ${calib['alphasesnse_base_to_alphasense_front_right']['yaw']}" />
+  <joint name="alphasense_base_to_alphasense_front_right" type="fixed">
+    <origin xyz=" ${calib['alphasense_base_to_alphasense_front_right']['x']}
+                  ${calib['alphasense_base_to_alphasense_front_right']['y']}
+                  ${calib['alphasense_base_to_alphasense_front_right']['z']}"
+            rpy=" ${calib['alphasense_base_to_alphasense_front_right']['roll']}
+                  ${calib['alphasense_base_to_alphasense_front_right']['pitch']}
+                  ${calib['alphasense_base_to_alphasense_front_right']['yaw']}" />
     <parent link="alphasense_base" />
     <child link="alphasense_front_right" />
@@ -40,11 +40,11 @@
   <!-- Alphasense Cam2/ front middle -->
   <link name="alphasense_front_middle" />
-  <joint name="alphasesnse_base_to_alphasense_front_middle" type="fixed">
-    <origin xyz=" ${calib['alphasesnse_base_to_alphasense_front_middle']['x']}
-                  ${calib['alphasesnse_base_to_alphasense_front_middle']['y']}
-                  ${calib['alphasesnse_base_to_alphasense_front_middle']['z']}"
-            rpy=" ${calib['alphasesnse_base_to_alphasense_front_middle']['roll']}
-                  ${calib['alphasesnse_base_to_alphasense_front_middle']['pitch']}
-                  ${calib['alphasesnse_base_to_alphasense_front_middle']['yaw']}" />
+  <joint name="alphasense_base_to_alphasense_front_middle" type="fixed">
+    <origin xyz=" ${calib['alphasense_base_to_alphasense_front_middle']['x']}
+                  ${calib['alphasense_base_to_alphasense_front_middle']['y']}
+                  ${calib['alphasense_base_to_alphasense_front_middle']['z']}"
+            rpy=" ${calib['alphasense_base_to_alphasense_front_middle']['roll']}
+                  ${calib['alphasense_base_to_alphasense_front_middle']['pitch']}
+                  ${calib['alphasense_base_to_alphasense_front_middle']['yaw']}" />
     <parent link="alphasense_base" />
     <child link="alphasense_front_middle" />
@@ -52,11 +52,11 @@
   <!-- Alphasense Cam3/ left -->
   <link name="alphasense_left" />
-  <joint name="alphasesnse_base_to_alphasense_left" type="fixed">
-    <origin xyz=" ${calib['alphasesnse_base_to_alphasense_left']['x']}
-                  ${calib['alphasesnse_base_to_alphasense_left']['y']}
-                  ${calib['alphasesnse_base_to_alphasense_left']['z']}"
-            rpy=" ${calib['alphasesnse_base_to_alphasense_left']['roll']}
-                  ${calib['alphasesnse_base_to_alphasense_left']['pitch']}
-                  ${calib['alphasesnse_base_to_alphasense_left']['yaw']}" />
+  <joint name="alphasense_base_to_alphasense_left" type="fixed">
+    <origin xyz=" ${calib['alphasense_base_to_alphasense_left']['x']}
+                  ${calib['alphasense_base_to_alphasense_left']['y']}
+                  ${calib['alphasense_base_to_alphasense_left']['z']}"
+            rpy=" ${calib['alphasense_base_to_alphasense_left']['roll']}
+                  ${calib['alphasense_base_to_alphasense_left']['pitch']}
+                  ${calib['alphasense_base_to_alphasense_left']['yaw']}" />
     <parent link="alphasense_base" />
     <child link="alphasense_left" />
@@ -64,11 +64,11 @@
   <!-- Alphasense Cam4/ right -->
   <link name="alphasense_right" />
-  <joint name="alphasesnse_base_to_alphasense_right" type="fixed">
-    <origin xyz=" ${calib['alphasesnse_base_to_alphasense_right']['x']}
-                  ${calib['alphasesnse_base_to_alphasense_right']['y']}
-                  ${calib['alphasesnse_base_to_alphasense_right']['z']}"
-            rpy=" ${calib['alphasesnse_base_to_alphasense_right']['roll']}
-                  ${calib['alphasesnse_base_to_alphasense_right']['pitch']}
-                  ${calib['alphasesnse_base_to_alphasense_right']['yaw']}" />
+  <joint name="alphasense_base_to_alphasense_right" type="fixed">
+    <origin xyz=" ${calib['alphasense_base_to_alphasense_right']['x']}
+                  ${calib['alphasense_base_to_alphasense_right']['y']}
+                  ${calib['alphasense_base_to_alphasense_right']['z']}"
+            rpy=" ${calib['alphasense_base_to_alphasense_right']['roll']}
+                  ${calib['alphasense_base_to_alphasense_right']['pitch']}
+                  ${calib['alphasense_base_to_alphasense_right']['yaw']}" />
     <parent link="alphasense_base" />
     <child link="alphasense_right" />
@@ -160,2 +160,3 @@
     <child link="zed_left" />
   </joint>
+</robot>

Commit message: Update the URDF description of the alphasense cameras such that they match the corresponding frame IDs of each camera.

File: box_model/box_model/urdf/cameras/cameras.urdf.xacro (robot description, xacro)
@@ -14,6 +14,6 @@
     <child link="alphasense_base" />
   </joint>
-  <!-- Alphasense Cam0/ front left (should be identity)-->
-  <link name="alphasense_front_left" />
+  <!-- Alphasense Cam1/ front left (should be identity)-->
+  <link name="cam1_sensor_frame" />
   <joint name="alphasense_base_to_alphasense_front_left" type="fixed">
     <origin xyz=" ${calib['alphasense_base_to_alphasense_front_left']['x']}
@@ -24,8 +24,8 @@
                   ${calib['alphasense_base_to_alphasense_front_left']['yaw']}" />
     <parent link="alphasense_base" />
-    <child link="alphasense_front_left" />
+    <child link="cam1_sensor_frame" />
   </joint>
-  <!-- Alphasense Cam1/ front right -->
-  <link name="alphasense_front_right" />
+  <!-- Alphasense Cam2/ front right -->
+  <link name="cam2_sensor_frame" />
   <joint name="alphasense_base_to_alphasense_front_right" type="fixed">
     <origin xyz=" ${calib['alphasense_base_to_alphasense_front_right']['x']}
@@ -36,8 +36,8 @@
                   ${calib['alphasense_base_to_alphasense_front_right']['yaw']}" />
     <parent link="alphasense_base" />
-    <child link="alphasense_front_right" />
+    <child link="cam2_sensor_frame" />
   </joint>
-  <!-- Alphasense Cam2/ front middle -->
-  <link name="alphasense_front_middle" />
+  <!-- Alphasense Cam3/ front middle -->
+  <link name="cam3_sensor_frame" />
   <joint name="alphasense_base_to_alphasense_front_middle" type="fixed">
     <origin xyz=" ${calib['alphasense_base_to_alphasense_front_middle']['x']}
@@ -48,8 +48,8 @@
                   ${calib['alphasense_base_to_alphasense_front_middle']['yaw']}" />
     <parent link="alphasense_base" />
-    <child link="alphasense_front_middle" />
+    <child link="cam3_sensor_frame" />
   </joint>
-  <!-- Alphasense Cam3/ left -->
-  <link name="alphasense_left" />
+  <!-- Alphasense Cam4/ left -->
+  <link name="cam4_sensor_frame" />
   <joint name="alphasense_base_to_alphasense_left" type="fixed">
     <origin xyz=" ${calib['alphasense_base_to_alphasense_left']['x']}
@@ -60,8 +60,8 @@
                   ${calib['alphasense_base_to_alphasense_left']['yaw']}" />
     <parent link="alphasense_base" />
-    <child link="alphasense_left" />
+    <child link="cam4_sensor_frame" />
   </joint>
-  <!-- Alphasense Cam4/ right -->
-  <link name="alphasense_right" />
+  <!-- Alphasense Cam5/ right -->
+  <link name="cam5_sensor_frame" />
   <joint name="alphasense_base_to_alphasense_right" type="fixed">
     <origin xyz=" ${calib['alphasense_base_to_alphasense_right']['x']}
@@ -72,5 +72,5 @@
                   ${calib['alphasense_base_to_alphasense_right']['yaw']}" />
     <parent link="alphasense_base" />
-    <child link="alphasense_right" />
+    <child link="cam5_sensor_frame" />
   </joint>
   <!-- ////////// HDR ////////// -->

Commit message: Add zed2i pinned constraints such that the left ZED cameras defines the relationship to camera center ... and transitively the relationship to the box base Frank Fu 9 minutes ago

File: box_model/box_model/urdf/cameras/cameras.urdf.xacro (robot description, xacro)
@@ -127,10 +127,10 @@
     <link name="zed_base_link"/>
     <joint name="box_base_to_zed_base" type="fixed">
-        <origin xyz=" ${calib['box_base_to_zed_base']['x']}
-                  ${calib['box_base_to_zed_base']['y']}
-                  ${calib['box_base_to_zed_base']['z']}"
-                rpy=" ${calib['box_base_to_zed_base']['roll']}
-                  ${calib['box_base_to_zed_base']['pitch']}
-                  ${calib['box_base_to_zed_base']['yaw']}"/>
+        <origin xyz=" ${pinned_constraints['box_base_to_zed_base']['x']}
+                  ${pinned_constraints['box_base_to_zed_base']['y']}
+                  ${pinned_constraints['box_base_to_zed_base']['z']}"
+                rpy=" ${pinned_constraints['box_base_to_zed_base']['roll']}
+                  ${pinned_constraints['box_base_to_zed_base']['pitch']}
+                  ${pinned_constraints['box_base_to_zed_base']['yaw']}"/>
         <parent link="box_base"/>
         <child link="zed_base_link"/>
@@ -155,10 +155,10 @@
     <link name="zed2i_left_camera_frame"/>
     <joint name="zed_camera_center_to_zed_left" type="fixed">
-        <origin xyz=" ${calib['zed_camera_center_to_zed_left']['x']}
-                  ${calib['zed_camera_center_to_zed_left']['y']}
-                  ${calib['zed_camera_center_to_zed_left']['z']}"
-                rpy=" ${calib['zed_camera_center_to_zed_left']['roll']}
-                  ${calib['zed_camera_center_to_zed_left']['pitch']}
-                  ${calib['zed_camera_center_to_zed_left']['yaw']}"/>
+        <origin xyz=" ${pinned_constraints['zed_camera_center_to_zed_left']['x']}
+                  ${pinned_constraints['zed_camera_center_to_zed_left']['y']}
+                  ${pinned_constraints['zed_camera_center_to_zed_left']['z']}"
+                rpy=" ${pinned_constraints['zed_camera_center_to_zed_left']['roll']}
+                  ${pinned_constraints['zed_camera_center_to_zed_left']['pitch']}
+                  ${pinned_constraints['zed_camera_center_to_zed_left']['yaw']}"/>
         <parent link="zed2i_camera_center"/>
         <child link="zed2i_left_camera_frame"/>
@@ -188,11 +188,11 @@
     <link name="zed2i_right_camera_frame"/>
     <joint name="zed_camera_center_to_zed_right" type="fixed">
-        <origin xyz=" ${calib['zed_camera_center_to_zed_right']['x']}
-                  ${calib['zed_camera_center_to_zed_right']['y']}
-                  ${calib['zed_camera_center_to_zed_right']['z']}"
-                rpy=" ${calib['zed_camera_center_to_zed_right']['roll']}
-                  ${calib['zed_camera_center_to_zed_right']['pitch']}
-                  ${calib['zed_camera_center_to_zed_right']['yaw']}"/>
-        <parent link="zed2i_camera_center"/>
+        <origin xyz=" ${pinned_constraints['zed2i_optical_to_zed2i_camera']['x']}
+                  ${pinned_constraints['zed2i_optical_to_zed2i_camera']['y']}
+                  ${pinned_constraints['zed2i_optical_to_zed2i_camera']['z']}"
+                rpy=" ${pinned_constraints['zed2i_optical_to_zed2i_camera']['roll']}
+                  ${pinned_constraints['zed2i_optical_to_zed2i_camera']['pitch']}
+                  ${pinned_constraints['zed2i_optical_to_zed2i_camera']['yaw']}"/>
+        <parent link="zed2i_right_camera_optical_frame"/>
         <child link="zed2i_right_camera_frame"/>
     </joint>

Commit message: Add right zed camera relative to left zed camera

File: box_model/box_model/urdf/cameras/cameras.urdf.xacro (robot description, xacro)
@@ -186,4 +186,15 @@
         <child link="zed2i_imu_link"/>
     </joint>
+    <link name="zed2i_right_camera_optical_frame"/>
+    <joint name="zed_left_optical_to_zed_right_optical" type="fixed">
+        <origin xyz=" ${calib['zed_left_optical_to_zed_right_optical']['x']}
+                  ${calib['zed_left_optical_to_zed_right_optical']['y']}
+                  ${calib['zed_left_optical_to_zed_right_optical']['z']}"
+                rpy=" ${calib['zed_left_optical_to_zed_right_optical']['roll']}
+                  ${calib['zed_left_optical_to_zed_right_optical']['pitch']}
+                  ${calib['zed_left_optical_to_zed_right_optical']['yaw']}"/>
+        <parent link="zed2i_left_camera_optical_frame"/>
+        <child link="zed2i_right_camera_optical_frame"/>
+    </joint>
     <link name="zed2i_right_camera_frame"/>
     <joint name="zed_camera_center_to_zed_right" type="fixed">
@@ -197,14 +208,3 @@
         <child link="zed2i_right_camera_frame"/>
     </joint>
-    <link name="zed2i_right_camera_optical_frame"/>
-    <joint name="zed_right_to_optical" type="fixed">
-        <origin xyz=" ${pinned_constraints['zed2i_camera_to_zed2i_optical']['x']}
-                  ${pinned_constraints['zed2i_camera_to_zed2i_optical']['y']}
-                  ${pinned_constraints['zed2i_camera_to_zed2i_optical']['z']}"
-                rpy=" ${pinned_constraints['zed2i_camera_to_zed2i_optical']['roll']}
-                  ${pinned_constraints['zed2i_camera_to_zed2i_optical']['pitch']}
-                  ${pinned_constraints['zed2i_camera_to_zed2i_optical']['yaw']}"/>
-        <parent link="zed2i_right_camera_frame"/>
-        <child link="zed2i_right_camera_optical_frame"/>
-    </joint>
 </robot>

Commit message: Add alphasense helper frame ids

File: box_model/box_model/urdf/cameras/cameras.urdf.xacro (robot description, xacro)
@@ -2,5 +2,5 @@
 <robot name="cameras" xmlns:xacro="http://www.ros.org/wiki/xacro">
     <!-- ////////// Alphasense ////////// -->
-    <!-- Alphasense base (coincides with alphasense Cam0/ front left) -->
+    <!-- Alphasense base (coincides with alphasense Cam1/ front center) -->
     <link name="alphasense_base"/>
     <joint name="box_base_to_alphasense_base" type="fixed">
@@ -14,15 +14,27 @@
         <child link="alphasense_base"/>
     </joint>
-    <!-- Alphasense Cam1/ front left (should be identity)-->
+    <link name="alphasense_front_center"/>
+    <joint name="alphasense_front_center_identity" type="fixed">
+        <origin xyz="0 0 0" rpy="0 0 0"/>
+        <parent link="cam1_sensor_frame"/>
+        <child link="alphasense_front_center"/>
+    </joint>
+    <!-- Alphasense Cam1/ front center (should be identity)-->
     <link name="cam1_sensor_frame"/>
-    <joint name="alphasense_base_to_alphasense_front_left" type="fixed">
-        <origin xyz=" ${pinned_constraints['alphasense_base_to_alphasense_front_left']['x']}
-                  ${pinned_constraints['alphasense_base_to_alphasense_front_left']['y']}
-                  ${pinned_constraints['alphasense_base_to_alphasense_front_left']['z']}"
-                rpy=" ${pinned_constraints['alphasense_base_to_alphasense_front_left']['roll']}
-                  ${pinned_constraints['alphasense_base_to_alphasense_front_left']['pitch']}
-                  ${pinned_constraints['alphasense_base_to_alphasense_front_left']['yaw']}"/>
+    <joint name="alphasense_base_to_alphasense_front_middle" type="fixed">
+        <origin xyz=" ${pinned_constraints['alphasense_base_to_alphasense_front_middle']['x']}
+                  ${pinned_constraints['alphasense_base_to_alphasense_front_middle']['y']}
+                  ${pinned_constraints['alphasense_base_to_alphasense_front_middle']['z']}"
+                rpy=" ${pinned_constraints['alphasense_base_to_alphasense_front_middle']['roll']}
+                  ${pinned_constraints['alphasense_base_to_alphasense_front_middle']['pitch']}
+                  ${pinned_constraints['alphasense_base_to_alphasense_front_middle']['yaw']}"/>
         <parent link="alphasense_base"/>
         <child link="cam1_sensor_frame"/>
+    </joint>
+    <link name="alphasense_front_right"/>
+    <joint name="alphasense_front_right_identity" type="fixed">
+        <origin xyz="0 0 0" rpy="0 0 0"/>
+        <parent link="cam2_sensor_frame"/>
+        <child link="alphasense_front_center"/>
     </joint>
     <!-- Alphasense Cam2/ front right -->
@@ -38,15 +50,27 @@
         <child link="cam2_sensor_frame"/>
     </joint>
-    <!-- Alphasense Cam3/ front middle -->
+    <link name="alphasense_front_left"/>
+    <joint name="alphasense_front_left_identity" type="fixed">
+        <origin xyz="0 0 0" rpy="0 0 0"/>
+        <parent link="cam3_sensor_frame"/>
+        <child link="alphasense_front_left"/>
+    </joint>
+    <!-- Alphasense Cam3/ front left -->
     <link name="cam3_sensor_frame"/>
-    <joint name="alphasense_base_to_alphasense_front_middle" type="fixed">
-        <origin xyz=" ${calib['alphasense_base_to_alphasense_front_middle']['x']}
-                  ${calib['alphasense_base_to_alphasense_front_middle']['y']}
-                  ${calib['alphasense_base_to_alphasense_front_middle']['z']}"
-                rpy=" ${calib['alphasense_base_to_alphasense_front_middle']['roll']}
-                  ${calib['alphasense_base_to_alphasense_front_middle']['pitch']}
-                  ${calib['alphasense_base_to_alphasense_front_middle']['yaw']}"/>
+    <joint name="alphasense_base_to_alphasense_front_left" type="fixed">
+        <origin xyz=" ${calib['alphasense_base_to_alphasense_front_left']['x']}
+                  ${calib['alphasense_base_to_alphasense_front_left']['y']}
+                  ${calib['alphasense_base_to_alphasense_front_left']['z']}"
+                rpy=" ${calib['alphasense_base_to_alphasense_front_left']['roll']}
+                  ${calib['alphasense_base_to_alphasense_front_left']['pitch']}
+                  ${calib['alphasense_base_to_alphasense_front_left']['yaw']}"/>
         <parent link="alphasense_base"/>
         <child link="cam3_sensor_frame"/>
+    </joint>
+    <link name="alphasense_left"/>
+    <joint name="alphasense_left_identity" type="fixed">
+        <origin xyz="0 0 0" rpy="0 0 0"/>
+        <parent link="cam4_sensor_frame"/>
+        <child link="alphasense_left"/>
     </joint>
     <!-- Alphasense Cam4/ left -->
@@ -61,4 +85,10 @@
         <parent link="alphasense_base"/>
         <child link="cam4_sensor_frame"/>
+    </joint>
+    <link name="alphasense_right"/>
+    <joint name="alphasense_right_identity" type="fixed">
+        <origin xyz="0 0 0" rpy="0 0 0"/>
+        <parent link="cam5_sensor_frame"/>
+        <child link="alphasense_right"/>
     </joint>
     <!-- Alphasense Cam5/ right -->

Commit message: Fix camera frames

File: box_model/box_model/urdf/cameras/cameras.urdf.xacro (robot description, xacro)
@@ -23,10 +23,10 @@
     <link name="cam1_sensor_frame"/>
     <joint name="alphasense_base_to_alphasense_front_middle" type="fixed">
-        <origin xyz=" ${pinned_constraints['alphasense_base_to_alphasense_front_middle']['x']}
-                  ${pinned_constraints['alphasense_base_to_alphasense_front_middle']['y']}
-                  ${pinned_constraints['alphasense_base_to_alphasense_front_middle']['z']}"
-                rpy=" ${pinned_constraints['alphasense_base_to_alphasense_front_middle']['roll']}
-                  ${pinned_constraints['alphasense_base_to_alphasense_front_middle']['pitch']}
-                  ${pinned_constraints['alphasense_base_to_alphasense_front_middle']['yaw']}"/>
+        <origin xyz=" ${calib['alphasense_base_to_alphasense_front_middle']['x']}
+                  ${calib['alphasense_base_to_alphasense_front_middle']['y']}
+                  ${calib['alphasense_base_to_alphasense_front_middle']['z']}"
+                rpy=" ${calib['alphasense_base_to_alphasense_front_middle']['roll']}
+                  ${calib['alphasense_base_to_alphasense_front_middle']['pitch']}
+                  ${calib['alphasense_base_to_alphasense_front_middle']['yaw']}"/>
         <parent link="alphasense_base"/>
         <child link="cam1_sensor_frame"/>
@@ -36,5 +36,5 @@
         <origin xyz="0 0 0" rpy="0 0 0"/>
         <parent link="cam2_sensor_frame"/>
-        <child link="alphasense_front_center"/>
+        <child link="alphasense_front_right"/>
     </joint>
     <!-- Alphasense Cam2/ front right -->
@@ -59,10 +59,10 @@
     <link name="cam3_sensor_frame"/>
     <joint name="alphasense_base_to_alphasense_front_left" type="fixed">
-        <origin xyz=" ${calib['alphasense_base_to_alphasense_front_left']['x']}
-                  ${calib['alphasense_base_to_alphasense_front_left']['y']}
-                  ${calib['alphasense_base_to_alphasense_front_left']['z']}"
-                rpy=" ${calib['alphasense_base_to_alphasense_front_left']['roll']}
-                  ${calib['alphasense_base_to_alphasense_front_left']['pitch']}
-                  ${calib['alphasense_base_to_alphasense_front_left']['yaw']}"/>
+        <origin xyz=" ${pinned_constraints['alphasense_base_to_alphasense_front_left']['x']}
+                  ${pinned_constraints['alphasense_base_to_alphasense_front_left']['y']}
+                  ${pinned_constraints['alphasense_base_to_alphasense_front_left']['z']}"
+                rpy=" ${pinned_constraints['alphasense_base_to_alphasense_front_left']['roll']}
+                  ${pinned_constraints['alphasense_base_to_alphasense_front_left']['pitch']}
+                  ${pinned_constraints['alphasense_base_to_alphasense_front_left']['yaw']}"/>
         <parent link="alphasense_base"/>
         <child link="cam3_sensor_frame"/>
